File: Hardware/dsp-amplifier-x4.kicad_pcb (KiCad board)
At the start: 2 copper layers, 104 parts, among them J1 Raspberry_Pi_2_3, J2 USB_B, J3 USBi, Q1 STD2805, U1 ADAU1452, U2 24LC1025, U3 SI53365, U5 TPS54308, U6 TPS54308, U7 AMS1117-3.3, U8 USBLC6-2SC6, U9 PCM2707, Y1 12 MHz

Commit message: various fixes
Parts:
- removed C36, C37: 4.7u, Capacitor_SMD:C_0805_2012Metric_Pad1.18x1.45mm_HandSolder
- added C42: 10n, Capacitor_SMD:C_0805_2012Metric_Pad1.18x1.45mm_HandSolder, F.Cu at (54.4, 138.2)
- added C43: 10n, Capacitor_SMD:C_0805_2012Metric_Pad1.18x1.45mm_HandSolder, F.Cu at (54.4, 135.2)
- added C44: 10n, Capacitor_SMD:C_0805_2012Metric_Pad1.18x1.45mm_HandSolder, F.Cu at (78.9, 118.2)
- added C45: 100n, Capacitor_SMD:C_0805_2012Metric_Pad1.18x1.45mm_HandSolder, F.Cu at (83.7, 118.8)
- added C46: 100n, Capacitor_SMD:C_0805_2012Metric_Pad1.18x1.45mm_HandSolder, F.Cu at (88.5, 118.8)
- added C47: 100n, Capacitor_SMD:C_0805_2012Metric_Pad1.18x1.45mm_HandSolder, F.Cu at (59.2, 141.2)
- added C48: 10n, Capacitor_SMD:C_0805_2012Metric_Pad1.18x1.45mm_HandSolder, F.Cu at (54.4, 150.2)
- added C49: 10n, Capacitor_SMD:C_0805_2012Metric_Pad1.18x1.45mm_HandSolder, F.Cu at (78.9, 127.2)
- added C50: 10n, Capacitor_SMD:C_0805_2012Metric_Pad1.18x1.45mm_HandSolder, F.Cu at (59.2, 144.2)
- added C51: 100n, Capacitor_SMD:C_0805_2012Metric_Pad1.18x1.45mm_HandSolder, F.Cu at (78.9, 124.2)
- added C52: 100n, Capacitor_SMD:C_0805_2012Metric_Pad1.18x1.45mm_HandSolder, F.Cu at (93.4, 118.0)
- added C53: 100n, Capacitor_SMD:C_0805_2012Metric_Pad1.18x1.45mm_HandSolder, F.Cu at (78.9, 121.2)
- added C55: 10n, Capacitor_SMD:C_0805_2012Metric_Pad1.18x1.45mm_HandSolder, F.Cu at (54.4, 147.2)
- added C57: 10n, Capacitor_SMD:C_0805_2012Metric_Pad1.18x1.45mm_HandSolder, F.Cu at (54.4, 144.2)
- added C58: 100n, Capacitor_SMD:C_0805_2012Metric_Pad1.18x1.45mm_HandSolder, F.Cu at (64.0, 138.5)
- added C59: 100n, Capacitor_SMD:C_0805_2012Metric_Pad1.18x1.45mm_HandSolder, F.Cu at (52.1, 156.9)
- added C60: 10n, Capacitor_SMD:C_0805_2012Metric_Pad1.18x1.45mm_HandSolder, F.Cu at (83.7, 121.9)
- added C61: 10n, Capacitor_SMD:C_0805_2012Metric_Pad1.18x1.45mm_HandSolder, F.Cu at (59.2, 147.2)
- added C62: 100n, Capacitor_SMD:C_0805_2012Metric_Pad1.18x1.45mm_HandSolder, F.Cu at (64.0, 141.5)
- added C63: 100n, Capacitor_SMD:C_0805_2012Metric_Pad1.18x1.45mm_HandSolder, F.Cu at (68.8, 138.5)
- added J4: Screw_Terminal_01x02, TerminalBlock:TerminalBlock_Altech_AK300-2_P5.00mm, F.Cu at (55.3, 123.6)
- added J5: Screw_Terminal_01x02, TerminalBlock:TerminalBlock_Altech_AK300-2_P5.00mm, F.Cu at (94.3, 109.5)
- added R38: 33, Resistor_SMD:R_0603_1608Metric_Pad0.98x0.95mm_HandSolder, F.Cu at (59.0, 149.9)
- added R39: 33, Resistor_SMD:R_0603_1608Metric_Pad0.98x0.95mm_HandSolder, F.Cu at (105.4, 103.8)
- added R40: 33, Resistor_SMD:R_0603_1608Metric_Pad0.98x0.95mm_HandSolder, F.Cu at (78.5, 130.2)
- added R41: 4.3k, Resistor_SMD:R_0603_1608Metric_Pad0.98x0.95mm_HandSolder, F.Cu at (63.8, 144.3)
- added R42: DNP, Resistor_SMD:R_0603_1608Metric_Pad0.98x0.95mm_HandSolder, F.Cu at (83.5, 124.6)
- added R43: DNP, Resistor_SMD:R_0603_1608Metric_Pad0.98x0.95mm_HandSolder, F.Cu at (54.1, 153.0)
- added R44: 4.3k, Resistor_SMD:R_0603_1608Metric_Pad0.98x0.95mm_HandSolder, F.Cu at (93.1, 120.8)
- added RV1: R_POT, Potentiometer_THT:Potentiometer_Vishay_248GJ-249GJ_Single_Vertical, F.Cu at (69.5, 112.1)
- added RV2: R_POT, Potentiometer_THT:Potentiometer_Vishay_248GJ-249GJ_Single_Vertical, F.Cu at (53.6, 112.1)
- added U?1: TAS5760MDCAR, Package_SO:HTSSOP-32-1EP_6.1x11mm_P0.65mm_EP5.2x11mm_Mask4.11x4.36mm_ThermalVias, F.Cu at (174.2, 46.6)
- C25: value 1u -> 100n
- C32: value 100n -> 470u; footprint Capacitor_SMD:C_0603_1608Metric_Pad1.08x0.95mm_HandSolder -> Capacitor_THT:CP_Radial_D14.0mm_P5.00mm
- moved FB1 225.3 mm to (47.2, 156.8)
- moved R30 223.6 mm to (59.0, 152.5)
- moved R23 214.1 mm to (68.1, 144.3)
- moved C22 211.4 mm to (54.4, 141.2)
- moved R25 207.4 mm to (56.6, 158.0)
- moved R27 206.6 mm to (68.1, 146.8)
- moved R16 201.2 mm to (56.6, 155.5)
- moved R33 196.6 mm to (73.4, 140.8)
- moved C21 196.1 mm to (59.2, 132.1)
- moved C20 195.6 mm to (63.3, 149.9)
- moved R28 190.3 mm to (82.9, 132.4)
- moved R15 189.7 mm to (83.5, 127.1)
- moved R21 189.3 mm to (68.6, 141.2)
- moved R32 187.7 mm to (78.5, 137.7)
- moved R34 187.0 mm to (82.9, 129.9)
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Connections:
- C25 pad 1: +3V3 -> +24V
- C26 pad 2: (no net) -> Net-(C26-Pad2)
- C27 pad 2: (no net) -> Net-(C27-Pad2)
- C29 pad 2: (no net) -> Net-(C29-Pad2)
- C30 pad 1: (no net) -> Net-(C30-Pad1)
- C33 pad 2: (no net) -> Net-(C33-Pad2)
- C34 pad 2: (no net) -> Net-(C34-Pad2)
- Q1 pad 1: Net-(Q1-Pad1) -> /VDRIVE
- R1 pad 2: Net-(Q1-Pad1) -> /VDRIVE
- R22 pad 1: (no net) -> /AMP1_LRCLK
- R23 pad 1: (no net) -> /AMP1_BCLK
- R24 pad 1: (no net) -> /AMP1_SDIN
- U1 pad 26: (no net) -> /AMP1_NSPK_SD
- U1 pad 27: (no net) -> /AMP1_SPK_SLEEP
- U1 pad 3: (no net) -> /VDRIVE
- U1 pad 42: (no net) -> Net-(R38-Pad2)
- U1 pad 43: (no net) -> Net-(R39-Pad2)
- U1 pad 44: (no net) -> Net-(R40-Pad2)
- U1 pad 66: (no net) -> /EXT_O_LRCLK
- U1 pad 8: (no net) -> /VPOT0
- U1 pad 9: (no net) -> /VPOT1
- U3 pad 16: (no net) -> /AMP1_CLOCK

Commit message: started routing
Parts:
- removed FB2, FB3, FB4: 600/100M, Inductor_SMD:L_0805_2012Metric_Pad1.05x1.20mm_HandSolder
- removed U?1: TAS5760MDCAR, Package_SO:HTSSOP-32-1EP_6.1x11mm_P0.65mm_EP5.2x11mm_Mask4.11x4.36mm_ThermalVias
- added C36: 10u, Capacitor_SMD:C_1206_3216Metric_Pad1.33x1.80mm_HandSolder, F.Cu at (92.5, -28.0)
- added C37: 10u, Capacitor_SMD:C_1206_3216Metric_Pad1.33x1.80mm_HandSolder, F.Cu at (61.8, -30.8)
- added C64: 1u, Capacitor_SMD:C_0805_2012Metric_Pad1.18x1.45mm_HandSolder, F.Cu at (177.2, -29.2)
- added C65: 100n, Capacitor_SMD:C_0603_1608Metric_Pad1.08x0.95mm_HandSolder, F.Cu at (197.5, -31.5)
- added C66: 100n, Capacitor_SMD:C_0603_1608Metric_Pad1.08x0.95mm_HandSolder, F.Cu at (197.5, -22.2)
- added C67: 470u, Capacitor_THT:CP_Radial_D16.0mm_P7.50mm, F.Cu at (196.2, -44.0)
- added C68: 220n, Capacitor_SMD:C_0603_1608Metric_Pad1.08x0.95mm_HandSolder, F.Cu at (195.2, -33.8)
- added C69: 220n, Capacitor_SMD:C_0603_1608Metric_Pad1.08x0.95mm_HandSolder, F.Cu at (198.0, -27.8)
- added C70: 220n, Capacitor_SMD:C_0603_1608Metric_Pad1.08x0.95mm_HandSolder, F.Cu at (195.2, -20.0)
- added C71: 220n, Capacitor_SMD:C_0603_1608Metric_Pad1.08x0.95mm_HandSolder, F.Cu at (198.0, -26.0)
- added C72: 680n, Capacitor_SMD:C_0603_1608Metric_Pad1.08x0.95mm_HandSolder, F.Cu at (212.2, -36.2)
- added C73: 680n, Capacitor_SMD:C_0603_1608Metric_Pad1.08x0.95mm_HandSolder, F.Cu at (212.2, -32.8)
- added C74: 680n, Capacitor_SMD:C_0603_1608Metric_Pad1.08x0.95mm_HandSolder, F.Cu at (212.2, -17.5)
- added C75: 680n, Capacitor_SMD:C_0603_1608Metric_Pad1.08x0.95mm_HandSolder, F.Cu at (212.2, -21.0)
- added C76: 33p, Capacitor_SMD:C_0603_1608Metric_Pad1.08x0.95mm_HandSolder, F.Cu at (230.2, 97.0)
- added C77: 33p, Capacitor_SMD:C_0603_1608Metric_Pad1.08x0.95mm_HandSolder, F.Cu at (236.8, 97.0)
- added C78: 100n, Capacitor_SMD:C_0603_1608Metric_Pad1.08x0.95mm_HandSolder, F.Cu at (231.2, 81.8)
- added C79: 10n, Capacitor_SMD:C_0603_1608Metric_Pad1.08x0.95mm_HandSolder, F.Cu at (322.0, 49.5)
- added C80: 10n, Capacitor_SMD:C_0603_1608Metric_Pad1.08x0.95mm_HandSolder, F.Cu at (278.5, 45.8)
- added F1: Fuse, Fuse:Fuseholder_Cylinder-5x20mm_Stelvio-Kontek_PTF78_Horizontal_Open, F.Cu at (25.8, 31.8)
- added J10: Conn_Coaxial, connectors_audio:cui_rcj_02x, F.Cu at (301.5, 45.8)
- added J6: Screw_Terminal_01x02, TerminalBlock:TerminalBlock_Wuerth_691311400102_P7.62mm, F.Cu at (218.5, -39.2)
- added J7: Screw_Terminal_01x02, TerminalBlock:TerminalBlock_Wuerth_691311400102_P7.62mm, F.Cu at (218.5, -22.2)
- added J8: USB_B, Connector_USB:USB_B_TE_5787834_Vertical, F.Cu at (255.8, 88.8)
- added J9: Conn_Coaxial, connectors_audio:cui_rcj_02x, F.Cu at (314.0, 45.5)
- added L10: 10u, Inductor_SMD:L_Abracon_ASPI-0630LR, F.Cu at (206.8, -23.0)
- added L7: 10u, Inductor_SMD:L_Abracon_ASPI-0630LR, F.Cu at (206.8, -38.2)
- added L8: 10u, Inductor_SMD:L_Abracon_ASPI-0630LR, F.Cu at (206.8, -30.8)
- added L9: 10u, Inductor_SMD:L_Abracon_ASPI-0630LR, F.Cu at (206.8, -15.5)
- added R45: 75, Resistor_SMD:R_0603_1608Metric_Pad0.98x0.95mm_HandSolder, F.Cu at (320.0, 49.5)
- added R46: 243, Resistor_SMD:R_0603_1608Metric_Pad0.98x0.95mm_HandSolder, F.Cu at (274.8, 45.8)
- added R47: 107, Resistor_SMD:R_0603_1608Metric_Pad0.98x0.95mm_HandSolder, F.Cu at (277.8, 48.5)
- added T1: DA100J, da100j:SOIC-6, F.Cu at (287.8, 48.2)
- added U10: 24LC1025, Package_SO:SO-8_5.3x6.2mm_P1.27mm, F.Cu at (105.0, 155.0)
- added U4: AMS1117-3.3, Package_TO_SOT_SMD:SOT-223-3_TabPin2, F.Cu at (68.0, -11.8)
- added X1: ASV-24.576MHz-EJ-T, Oscillator:Oscillator_SMD_Abracon_ASV-4Pin_7.0x5.1mm, F.Cu at (215.5, 126.0)
- C1: footprint Capacitor_SMD:C_0805_2012Metric_Pad1.18x1.45mm_HandSolder -> Capacitor_SMD:C_1206_3216Metric_Pad1.33x1.80mm_HandSolder
- C10, C11, C16: value 100n -> 10n
- C12: value 22u -> 100n
- C13, C8: value 10u -> 100n; footprint Capacitor_SMD:C_0805_2012Metric_Pad1.18x1.45mm_HandSolder -> Capacitor_SMD:C_0603_1608Metric_Pad1.08x0.95mm_HandSolder
- C14, C3, C4: value 1u -> 10n
- C15: value 22u -> 10n; footprint Capacitor_SMD:C_0805_2012Metric_Pad1.18x1.45mm_HandSolder -> Capacitor_SMD:C_0603_1608Metric_Pad1.08x0.95mm_HandSolder
- C17, C18: value 22u -> 100n; footprint Capacitor_SMD:C_0805_2012Metric_Pad1.18x1.45mm_HandSolder -> Capacitor_SMD:C_0603_1608Metric_Pad1.08x0.95mm_HandSolder
- C19: value 150p -> 100n
- C2: value 33p -> 150p
- C20: value 5.6n -> 10n
- C21: value 4.7u -> 10n; footprint Capacitor_SMD:C_0805_2012Metric_Pad1.18x1.45mm_HandSolder -> Capacitor_SMD:C_0603_1608Metric_Pad1.08x0.95mm_HandSolder
- C22: value 4.7u -> 10u; footprint Capacitor_SMD:C_0805_2012Metric_Pad1.18x1.45mm_HandSolder -> Capacitor_SMD:C_1206_3216Metric_Pad1.33x1.80mm_HandSolder
- C23, C24, C28: value 4.7u -> 100n; footprint Capacitor_SMD:C_0805_2012Metric_Pad1.18x1.45mm_HandSolder -> Capacitor_SMD:C_0603_1608Metric_Pad1.08x0.95mm_HandSolder
- C25, C31: value 100n -> 10u; footprint Capacitor_SMD:C_0603_1608Metric_Pad1.08x0.95mm_HandSolder -> Capacitor_SMD:C_1206_3216Metric_Pad1.33x1.80mm_HandSolder
- C26, C27, C30: value 1u -> 10u; footprint Capacitor_SMD:C_0603_1608Metric_Pad1.08x0.95mm_HandSolder -> Capacitor_SMD:C_1206_3216Metric_Pad1.33x1.80mm_HandSolder
- C29, C33: value 220n -> 100n
- C32: value 470u -> 100n; footprint Capacitor_THT:CP_Radial_D14.0mm_P5.00mm -> Capacitor_SMD:C_0603_1608Metric_Pad1.08x0.95mm_HandSolder
- C34, C35: value 220n -> 10u; footprint Capacitor_SMD:C_0603_1608Metric_Pad1.08x0.95mm_HandSolder -> Capacitor_SMD:C_1206_3216Metric_Pad1.33x1.80mm_HandSolder
- C38, C39, C40, C41: value 680n -> 10u; footprint Capacitor_SMD:C_0603_1608Metric_Pad1.08x0.95mm_HandSolder -> Capacitor_SMD:C_1206_3216Metric_Pad1.33x1.80mm_HandSolder
- C42: value 10n -> 10u; footprint Capacitor_SMD:C_0805_2012Metric_Pad1.18x1.45mm_HandSolder -> Capacitor_SMD:C_1206_3216Metric_Pad1.33x1.80mm_HandSolder
- C43, C44, C48, C49, C50: value 10n -> 1u
- C45, C62, C63: value 100n -> 1u
- C46, C51, C52: footprint Capacitor_SMD:C_0805_2012Metric_Pad1.18x1.45mm_HandSolder -> Capacitor_SMD:C_0603_1608Metric_Pad1.08x0.95mm_HandSolder
- C47: value 100n -> 10n; footprint Capacitor_SMD:C_0805_2012Metric_Pad1.18x1.45mm_HandSolder -> Capacitor_SMD:C_0603_1608Metric_Pad1.08x0.95mm_HandSolder
- C5: value 4.7u -> 10n
- C53: value 100n -> 470u; footprint Capacitor_SMD:C_0805_2012Metric_Pad1.18x1.45mm_HandSolder -> Capacitor_THT:CP_Radial_D16.0mm_P7.50mm
- C54, C56: value 100n -> 220n
- C55, C57: value 10n -> 220n; footprint Capacitor_SMD:C_0805_2012Metric_Pad1.18x1.45mm_HandSolder -> Capacitor_SMD:C_0603_1608Metric_Pad1.08x0.95mm_HandSolder
- C58, C59: value 100n -> 680n; footprint Capacitor_SMD:C_0805_2012Metric_Pad1.18x1.45mm_HandSolder -> Capacitor_SMD:C_0603_1608Metric_Pad1.08x0.95mm_HandSolder
- C6: value 100n -> 5.6n
- C60, C61: value 10n -> 680n; footprint Capacitor_SMD:C_0805_2012Metric_Pad1.18x1.45mm_HandSolder -> Capacitor_SMD:C_0603_1608Metric_Pad1.08x0.95mm_HandSolder
- C7: value 33p -> 100n
- FB1: footprint Inductor_SMD:L_0805_2012Metric_Pad1.05x1.20mm_HandSolder -> Inductor_SMD:L_0603_1608Metric_Pad1.05x0.95mm_HandSolder
- J1: value Raspberry_Pi_2_3 -> USBi; footprint Connector_PinHeader_2.54mm:PinHeader_2x20_P2.54mm_Vertical -> Connector_PinHeader_2.54mm:PinHeader_2x05_P2.54mm_Vertical
- J2: value USB_B -> EXT; footprint Connector_USB:USB_B_TE_5787834_Vertical -> Connector_PinHeader_2.54mm:PinHeader_2x08_P2.54mm_Vertical
- J3: value USBi -> Raspberry_Pi_2_3; footprint Connector_PinHeader_2.54mm:PinHeader_2x05_P2.54mm_Vertical -> Connector_PinHeader_2.54mm:PinHeader_2x20_P2.54mm_Vertical
- J4, J5: footprint TerminalBlock:TerminalBlock_Altech_AK300-2_P5.00mm -> TerminalBlock:TerminalBlock_Wuerth_691311400102_P7.62mm
- L1, L2, L3, L4, L5, L6: footprint Capacitor_SMD:C_0805_2012Metric_Pad1.18x1.45mm_HandSolder -> Inductor_SMD:L_Abracon_ASPI-0630LR
- R10, R5, R6: value 100k -> 33
- R12, R7: value 13.5k -> 33
- R13: value 33 -> 0.47
- R16, R18, R27, R30: value 33 -> 4.3k
- R17: value 4.3k -> 4.3k DNP
- R19: value 33 -> 4.3k DNP
- R2, R4: value 511k -> 4.3k
- R28: value 4.3k -> DNP
- R29: value 33 -> DNP
- R3: value 100k -> 4.3k
- R31: value 33 -> 511k
- R32, R35: value 4.3k -> 100k
- R33: value 4.3k -> 511k
- R34: value 4.3k DNP -> 100k
- R36: value 4.3k DNP -> 13.5k
- R37: value 33 -> 100k
- R38: value 33 -> 13.5k
- R41, R44: value 4.3k -> 33
- R42, R43: value DNP -> 33
- R9: value 0.47 -> 33
- U2: value 24LC1025 -> TPS54308; footprint Package_SO:SO-8_5.3x6.2mm_P1.27mm -> Package_TO_SOT_SMD:SOT-23-6
- U3: value SI53365 -> TPS54308; footprint Package_SO:TSSOP-16_4.4x5mm_P0.65mm -> Package_TO_SOT_SMD:SOT-23-6
- U5: value TPS54308 -> SI53365; footprint Package_TO_SOT_SMD:SOT-23-6 -> Package_SO:TSSOP-16_4.4x5mm_P0.65mm
- U6: value TPS54308 -> TAS5760MDCAR; footprint Package_TO_SOT_SMD:SOT-23-6 -> Package_SO:HTSSOP-32-1EP_6.1x11mm_P0.65mm_EP5.2x11mm_Mask4.11x4.36mm_ThermalVias
- U7: value AMS1117-3.3 -> TAS5760MDCAR; footprint Package_TO_SOT_SMD:SOT-223-3_TabPin2 -> Package_SO:HTSSOP-32-1EP_6.1x11mm_P0.65mm_EP5.2x11mm_Mask4.11x4.36mm_ThermalVias
- moved C62 206.2 mm to (179.5, -29.2), turned to 90 degrees
- moved C63 202.2 mm to (181.8, -29.2), turned to 90 degrees
- moved C55 200.5 mm to (210.5, 21.4)
- moved C61 200.1 mm to (210.5, 16.4)
- moved J4 197.5 mm to (224.7, 22.1)
- moved R43 197.5 mm to (241.5, 90.5), turned to 180 degrees
- moved R38 192.3 mm to (74.2, -41.8), turned to 180 degrees
- moved C50 185.4 mm to (190.2, 13.0)
- moved R30 180.2 mm to (162.2, 4.75)
- moved R37 179.9 mm to (74.2, -43.5)
- moved U5 179.4 mm to (224.2, 126.0)
- moved R33 178.0 mm to (77.2, -37.2), turned to 90 degrees
- moved R25 176.4 mm to (230.2, 127.0)
- moved C59 173.5 mm to (177.3, 36.9)
- moved R41 171.4 mm to (226.0, 89.0)
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Connections:
- C1 pad 1: Net-(C1-Pad1) -> +3V3
- C10 pad 1: Net-(C10-Pad1) -> /DVDD
- C10 pad 2: Net-(C10-Pad2) -> GND
- C11 pad 1: +24V -> +3V3
- C12 pad 1: +5VD -> /DVDD
- C13 pad 1: +24V -> +3V3
- C14 pad 1: +3V3 -> /DVDD
- C15 pad 1: +5VD -> +3V3
- C16 pad 1: Net-(C16-Pad1) -> +3.3VA
- C16 pad 2: Net-(C16-Pad2) -> GND
- C17 pad 1: +5VA -> /DVDD
- C18 pad 1: +5VA -> +3V3
- C19 pad 2: Net-(C19-Pad2) -> GND
- C2 pad 1: Net-(C2-Pad1) -> +3.3VA
- C2 pad 2: GND -> Net-(C2-Pad2)
- C20 pad 1: +3.3VA -> /DVDD
- C20 pad 2: Net-(C20-Pad2) -> GND
- C22 pad 1: /DVDD -> +3V3
- C22 pad 2: Net-(C22-Pad2) -> GND
- C23 pad 1: +3V3 -> /DVDD
- C24 pad 1: +3.3VA -> +3V3
- C25 pad 1: +24V -> +3.3VA
- C26 pad 1: Net-(C26-Pad1) -> +3.3VA
- C26 pad 2: Net-(C26-Pad2) -> GND
- C27 pad 1: Net-(C26-Pad1) -> /DVDD
- C28 pad 1: +3.3VA -> +24V
- C29 pad 1: Net-(C29-Pad1) -> +24V
- C29 pad 2: Net-(C29-Pad2) -> GND
- C3 pad 1: +3V3 -> /DVDD
- C30 pad 1: Net-(C30-Pad1) -> +24V
- C32 pad 1: +24V -> Net-(C32-Pad1)
- C32 pad 2: GND -> Net-(C32-Pad2)
- C34 pad 1: Net-(C34-Pad1) -> +5VD
- C34 pad 2: Net-(C34-Pad2) -> GND
- C35 pad 1: Net-(C35-Pad1) -> +5VA
- C35 pad 2: (no net) -> GND
- C38 pad 1: /I2S-AMP-2CH/SKP_OUTA+ -> +5VD
- C39 pad 1: /I2S-AMP-2CH/SKP_OUTA- -> +5VA
- C40 pad 1: /I2S-AMP-2CH/SKP_OUTB- -> +5VD
- C41 pad 1: /I2S-AMP-2CH/SKP_OUTB+ -> +5VA
- C42 pad 1: /DVDD -> +3.3VA
- C44 pad 1: +3.3VA -> +3V3
- C45 pad 1: /DVDD -> +3V3
- C47 pad 1: +3.3VA -> +3V3
- C48 pad 1: /DVDD -> Net-(C48-Pad1)
- C48 pad 2: GND -> Net-(C48-Pad2)
- C49 pad 1: +3V3 -> Net-(C48-Pad1)
- C49 pad 2: GND -> Net-(C49-Pad2)
- C50 pad 1: +3.3VA -> Net-(C50-Pad1)
- C51 pad 1: /DVDD -> +24V
- C52 pad 1: +3V3 -> +24V
- C53 pad 1: +3.3VA -> +24V
- C54 pad 2: GND -> Net-(C54-Pad2)
- C55 pad 1: /DVDD -> Net-(C55-Pad1)
- C55 pad 2: GND -> Net-(C55-Pad2)
- C56 pad 2: GND -> Net-(C56-Pad2)
- C57 pad 1: +3V3 -> Net-(C57-Pad1)
- C57 pad 2: GND -> Net-(C57-Pad2)
- C58 pad 1: /DVDD -> GND
- C58 pad 2: GND -> /I2S-AMP-2CH-A/SKP_OUTA+
- C59 pad 1: +3V3 -> GND
- C59 pad 2: GND -> /I2S-AMP-2CH-A/SKP_OUTA-
- C6 pad 1: +24V -> +3.3VA
- C6 pad 2: GND -> Net-(C6-Pad2)
- C60 pad 1: /DVDD -> GND
- C60 pad 2: GND -> /I2S-AMP-2CH-A/SKP_OUTB+
- C61 pad 1: +3V3 -> GND
- C61 pad 2: GND -> /I2S-AMP-2CH-A/SKP_OUTB-
- C62 pad 1: /DVDD -> Net-(C62-Pad1)
- C62 pad 2: GND -> Net-(C62-Pad2)
- C63 pad 1: +3V3 -> Net-(C62-Pad1)
- C63 pad 2: GND -> Net-(C63-Pad2)
- C7 pad 1: Net-(C7-Pad1) -> /DVDD
- C8 pad 1: +24V -> +3V3
- C9 pad 1: Net-(C9-Pad1) -> +3.3VA
- J1 pad 1: (no net) -> /SCL
- J1 pad 10: (no net) -> GND
- J1 pad 2: +5VD -> (no net)
- J1 pad 3: /PI_SDA -> /SDA
- J1 pad 4: +5VD -> (no net)
- J1 pad 5: /PI_SCL -> (no net)
- J1 pad 6: GND -> /DSP_NRESET
- J1 pad 9: GND -> (no net)
- J2 pad 1: VBUS -> +24V
- J2 pad 2: Net-(J2-Pad2) -> GND
- J2 pad 3: Net-(J2-Pad3) -> /EXT_MDI
- J2 pad 5: GND -> /EXT_MDO
- J3 pad 1: /PI_SCL -> (no net)
- J3 pad 10: GND -> (no net)
- J3 pad 2: (no net) -> +5VD
- J3 pad 3: /PI_SDA -> (no net)
- J3 pad 4: (no net) -> +5VD
- J3 pad 6: /DSP_NRESET -> GND
- J3 pad 9: (no net) -> GND
- J4 pad 1: /I2S-AMP-2CH/SKP_OUTA+ -> /I2S-AMP-2CH-A/SKP_OUTA+
- J4 pad 2: /I2S-AMP-2CH/SKP_OUTA- -> /I2S-AMP-2CH-A/SKP_OUTA-
- J5 pad 1: /I2S-AMP-2CH/SKP_OUTB+ -> /I2S-AMP-2CH-A/SKP_OUTB-
- J5 pad 2: /I2S-AMP-2CH/SKP_OUTB- -> /I2S-AMP-2CH-A/SKP_OUTB+
- L1 pad 1: Net-(C33-Pad1) -> +5VD
- L1 pad 2: /I2S-AMP-2CH/SKP_OUTA+ -> Net-(C32-Pad1)
- L2 pad 1: Net-(C29-Pad1) -> +5VA
- L2 pad 2: /I2S-AMP-2CH/SKP_OUTA- -> Net-(C33-Pad1)
- L3 pad 1: Net-(C35-Pad1) -> Net-(C54-Pad2)
- L3 pad 2: /I2S-AMP-2CH/SKP_OUTB- -> /I2S-AMP-2CH-A/SKP_OUTA+
- L4 pad 1: Net-(C34-Pad1) -> Net-(C55-Pad2)
- L4 pad 2: /I2S-AMP-2CH/SKP_OUTB+ -> /I2S-AMP-2CH-A/SKP_OUTA-
- L5 pad 1: +5VA -> Net-(C56-Pad2)
- L5 pad 2: Net-(C16-Pad1) -> /I2S-AMP-2CH-A/SKP_OUTB+
- L6 pad 1: +5VD -> Net-(C57-Pad2)
- L6 pad 2: Net-(C10-Pad1) -> /I2S-AMP-2CH-A/SKP_OUTB-
- PS1 pad 1: (no net) -> /Power/AC_L
- R1 pad 1: +3.3VA -> /DSP_NRESET
- R1 pad 2: /VDRIVE -> +3V3
- R10 pad 1: +5VD -> /AMP2_LRCLK
- R10 pad 2: /Power/FB_5V0 -> Net-(R10-Pad2)
- R11 pad 1: Net-(R11-Pad1) -> /AMP2_BCLK
- R11 pad 2: /USB I2S/USB-DP -> Net-(R11-Pad2)
- R12 pad 1: /Power/FB_5V0 -> /AMP2_SDIN
- R12 pad 2: GND -> Net-(R12-Pad2)
- R13 pad 1: Net-(R13-Pad1) -> GND
- R13 pad 2: /USB I2S/USB-DM -> Net-(C27-Pad2)
- R14 pad 1: /DSP_NRESET -> /EEPROM_SCL
- R15 pad 1: /DSP_SELFBOOT -> /EEPROM_SDA
- R16 pad 1: /DSP_CLOCK -> /SDA
- R16 pad 2: Net-(R16-Pad2) -> +3V3
- R17 pad 1: Net-(C19-Pad2) -> GND
- R17 pad 2: Net-(C20-Pad2) -> /DSP_ADDR0
- R18 pad 1: /USB_LRCLK -> /SCL
- R18 pad 2: Net-(R18-Pad2) -> +3V3
- R19 pad 1: /USB_BCLK -> GND
- R19 pad 2: Net-(R19-Pad2) -> /DSP_ADDR1
- R2 pad 1: +24V -> /DSP_SELFBOOT
- R2 pad 2: Net-(R2-Pad2) -> +3V3
- R20 pad 1: (no net) -> Net-(J3-Pad35)
- R20 pad 2: Net-(R20-Pad2) -> /PI_LRCLK
- R21 pad 1: /PI_SDATA_I -> Net-(J3-Pad38)
- R21 pad 2: Net-(R21-Pad2) -> /PI_SDATA_I
- R22 pad 1: /AMP1_LRCLK -> Net-(J3-Pad40)
- R22 pad 2: Net-(R22-Pad2) -> /PI_SDATA_O
- R23 pad 1: /AMP1_BCLK -> /Clock/CLK1
- R23 pad 2: Net-(R23-Pad2) -> /AMP1_CLOCK
- R24 pad 1: /AMP1_SDIN -> /Clock/CLK3
- R24 pad 2: Net-(R24-Pad2) -> /AMP2_CLOCK
- R25 pad 1: (no net) -> /Clock/CLK5
- R25 pad 2: Net-(R25-Pad2) -> /DSP_CLOCK
- R26 pad 1: (no net) -> /Clock/CLK7
- R26 pad 2: Net-(R26-Pad2) -> /EXT_MCLK
- R27 pad 1: (no net) -> /GAIN1
- R27 pad 2: Net-(R27-Pad2) -> +3V3
- R28 pad 1: /EEPROM_SCL -> GND
- R28 pad 2: +3V3 -> /GAIN1
- R29 pad 1: Net-(J1-Pad35) -> /GAIN0
- R29 pad 2: /PI_LRCLK -> +3V3
- R3 pad 1: Net-(R2-Pad2) -> Net-(C2-Pad2)
- R3 pad 2: GND -> Net-(C6-Pad2)
- R30 pad 1: Net-(J1-Pad38) -> GND
- R30 pad 2: /PI_SDATA_I -> /GAIN0
- R31 pad 1: Net-(J1-Pad40) -> +24V
- R31 pad 2: /PI_SDATA_O -> Net-(R31-Pad2)
- R32 pad 1: /EEPROM_SDA -> Net-(R31-Pad2)
- R32 pad 2: +3V3 -> GND
- R33 pad 1: /PI_SDA -> +24V
- R33 pad 2: +3V3 -> Net-(R33-Pad2)
- R34 pad 1: GND -> Net-(R33-Pad2)
- R34 pad 2: /DSP_ADDR0 -> GND
- R35 pad 1: /PI_SCL -> +5VD
- R35 pad 2: +3V3 -> /Power/FB_5V0
- R36 pad 1: GND -> /Power/FB_5V0
- R36 pad 2: /DSP_ADDR1 -> GND
- R37 pad 1: /USB_SDATA -> +5VA
- R37 pad 2: Net-(R37-Pad2) -> /Power/FB_5V0_SEC
- R38 pad 1: /EXT_O_LRCLK -> /Power/FB_5V0_SEC
- R38 pad 2: Net-(R38-Pad2) -> GND
- R39 pad 1: (no net) -> Net-(R39-Pad1)
- R39 pad 2: Net-(R39-Pad2) -> /USB I2S/USB-DM
- R4 pad 1: +24V -> +3.3VA
- R4 pad 2: Net-(R4-Pad2) -> /VDRIVE
- R40 pad 1: (no net) -> Net-(R40-Pad1)
- R40 pad 2: Net-(R40-Pad2) -> /USB I2S/USB-DP
- R41 pad 1: /GAIN1 -> /USB_LRCLK
- R41 pad 2: +3V3 -> Net-(R41-Pad2)
- R42 pad 1: GND -> /USB_BCLK
- R42 pad 2: /GAIN1 -> Net-(R42-Pad2)
- R43 pad 1: /GAIN0 -> (no net)
- R43 pad 2: +3V3 -> Net-(R43-Pad2)
- R44 pad 1: GND -> /USB_SDATA
- R44 pad 2: /GAIN0 -> Net-(R44-Pad2)
- R5 pad 1: Net-(R4-Pad2) -> /PI_SDATA_I
- R5 pad 2: GND -> Net-(R5-Pad2)
- R6 pad 1: +5VA -> /EXT_MDO
- R6 pad 2: /Power/FB_5V0_SEC -> Net-(R6-Pad2)
- R7 pad 1: /Power/FB_5V0_SEC -> /AMP1_LRCLK
- R7 pad 2: GND -> Net-(R7-Pad2)
- R8 pad 1: /SPDIF_IN -> /AMP1_BCLK
- R8 pad 2: (no net) -> Net-(R8-Pad2)
- R9 pad 1: GND -> /AMP1_SDIN
- R9 pad 2: Net-(C22-Pad2) -> Net-(R9-Pad2)
- U1 pad 16: Net-(C19-Pad2) -> Net-(C2-Pad2)
- U1 pad 21: Net-(R16-Pad2) -> /DSP_CLOCK
- U1 pad 30: /PI_SDA -> /SDA
- U1 pad 31: /PI_SCL -> /SCL
- U1 pad 41: Net-(R21-Pad2) -> Net-(R5-Pad2)
- U1 pad 42: Net-(R38-Pad2) -> (no net)
- U1 pad 43: Net-(R39-Pad2) -> (no net)
- U1 pad 44: Net-(R40-Pad2) -> Net-(R6-Pad2)
- U1 pad 45: (no net) -> /AMP2_NSPK_SD
- U1 pad 46: (no net) -> /AMP2_SPK_SLEEP
- U1 pad 47: Net-(R22-Pad2) -> Net-(R7-Pad2)
- U1 pad 48: Net-(R23-Pad2) -> Net-(R8-Pad2)
- U1 pad 49: Net-(R24-Pad2) -> Net-(R9-Pad2)
- U1 pad 5: (no net) -> /SPDIF_OUT
- U1 pad 50: Net-(R25-Pad2) -> Net-(R10-Pad2)
- U1 pad 51: Net-(R26-Pad2) -> Net-(R11-Pad2)
- U1 pad 52: Net-(R27-Pad2) -> Net-(R12-Pad2)
- U1 pad 60: /USB_BCLK -> /EXT_BCLK
- U1 pad 61: /USB_LRCLK -> /EXT_LRCLK
- U1 pad 62: /USB_SDATA -> /EXT_MDI
- U1 pad 65: (no net) -> /USB_BCLK
- U1 pad 66: /EXT_O_LRCLK -> /USB_LRCLK
- U1 pad 67: (no net) -> /USB_SDATA
- U2 pad 1: +3V3 -> GND
- U2 pad 2: +3V3 -> Net-(C32-Pad1)
- U2 pad 3: +3V3 -> +24V
- U2 pad 4: GND -> /Power/FB_5V0
- U2 pad 5: /EEPROM_SDA -> Net-(R31-Pad2)
- U2 pad 6: /EEPROM_SCL -> Net-(C32-Pad2)
- U3 pad 1: (no net) -> GND
- U3 pad 2: +3V3 -> Net-(C33-Pad1)
- U3 pad 3: /DSP_CLOCK -> +24V
- U3 pad 4: GND -> /Power/FB_5V0_SEC
- U3 pad 5: +3V3 -> Net-(R33-Pad2)
- U3 pad 6: (no net) -> Net-(C33-Pad2)
- U5 pad 1: GND -> Net-(U5-Pad1)
- U5 pad 2: Net-(C16-Pad1) -> +3V3
- U5 pad 3: +24V -> (no net)
- U5 pad 4: /Power/FB_5V0_SEC -> GND
- U5 pad 5: Net-(R2-Pad2) -> +3V3
- U5 pad 6: Net-(C16-Pad2) -> (no net)
- U6 pad 1: GND -> +24V
- U6 pad 2: Net-(C10-Pad1) -> Net-(C50-Pad1)
- U6 pad 3: +24V -> Net-(C48-Pad2)
- U6 pad 4: /Power/FB_5V0 -> Net-(C49-Pad2)
- U6 pad 5: Net-(R4-Pad2) -> Net-(C48-Pad1)
- U6 pad 6: Net-(C10-Pad2) -> (no net)
- U7 pad 1: GND -> +24V
- U7 pad 2: +3.3VA -> Net-(C64-Pad1)
- U7 pad 3: +5VA -> Net-(C62-Pad2)
- U8 pad 1: Net-(J2-Pad3) -> Net-(J8-Pad2)
- U8 pad 3: Net-(J2-Pad2) -> Net-(J8-Pad3)
- U8 pad 4: Net-(R13-Pad1) -> Net-(R40-Pad1)
- U8 pad 6: Net-(R11-Pad1) -> Net-(R39-Pad1)
- U9 pad 12: Net-(C2-Pad1) -> Net-(C76-Pad1)
- U9 pad 13: Net-(C7-Pad1) -> Net-(C77-Pad1)
- U9 pad 17: Net-(R37-Pad2) -> Net-(R44-Pad2)
- U9 pad 18: Net-(R20-Pad2) -> Net-(R43-Pad2)
- U9 pad 19: Net-(R19-Pad2) -> Net-(R42-Pad2)
- U9 pad 32: Net-(C9-Pad1) -> Net-(C78-Pad1)
- U9 pad 5: Net-(R18-Pad2) -> Net-(R41-Pad2)
- Y1 pad 1: Net-(C2-Pad1) -> Net-(C76-Pad1)
- Y1 pad 2: Net-(C7-Pad1) -> GND
- Y1 pad 3: (no net) -> Net-(C77-Pad1)
- Y1 pad 4: (no net) -> GND
Routing:
- net GND: track 0.00 -> 72.2 mm, vias 0 -> 17
- net +3V3: track 0.00 -> 33.1 mm, vias 0 -> 18
- net VBUS: track 0.00 -> 29.8 mm, vias 0 -> 2
- net +5VD: track 0.00 -> 26.6 mm
- net +5VA: track 0.00 -> 26.6 mm
- net +24V: track 0.00 -> 19.1 mm, vias 0 -> 7
- net Net-(J10-Pad1): track 0.00 -> 9.62 mm
- net Net-(C76-Pad1): track 0.00 -> 8.30 mm
- net Net-(C33-Pad1): track 0.00 -> 8.22 mm, vias 0 -> 9
- net Net-(C32-Pad1): track 0.00 -> 8.22 mm, vias 0 -> 9
- net Net-(J10-Pad2): track 0.00 -> 8.05 mm
- net Net-(C62-Pad2): track 0.00 -> 7.21 mm
- net Net-(R33-Pad2): track 0.00 -> 5.97 mm
- net Net-(R31-Pad2): track 0.00 -> 5.96 mm
- net Net-(C77-Pad1): track 0.00 -> 5.81 mm
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- added copper zone on B.Cu, net +24V
- added copper zone on F.Cu, net +24V
- added copper zone on F.Cu, net +3.3VA
- added copper zone on F.Cu, net +5VA
- added copper zone on F.Cu, net +5VD
- added copper zone on F.Cu, net /I2S-AMP-2CH-B/SKP_OUTA+
- added copper zone on F.Cu, net /I2S-AMP-2CH-B/SKP_OUTA-
- added copper zone on F.Cu, net /I2S-AMP-2CH-B/SKP_OUTB+
- added copper zone on F.Cu, net /I2S-AMP-2CH-B/SKP_OUTB-
- added copper zone on B.Cu, net GND
- added copper zone on F.Cu, net GND
- added copper zone on B.Cu, net Net-(C32-Pad1)
- added copper zone on F.Cu, net Net-(C32-Pad1)
- added copper zone on B.Cu, net Net-(C33-Pad1)
- added copper zone on F.Cu, net Net-(C33-Pad1)
- added copper zone on F.Cu, net Net-(C68-Pad2)
- added copper zone on F.Cu, net Net-(C69-Pad2)
- added copper zone on F.Cu, net Net-(C70-Pad2)
- added copper zone on F.Cu, net Net-(C71-Pad2)
Other:
- net class +3V3 removed
- net class ADAU removed
- net class Default: clearance 0.2 -> 0.25
- net class Default AMP removed
- net class VCC removed
- rule trace_clearance: 0.2 -> 0.25
- rule via_min_drill: 0.3 -> 0.2

Commit message: routing progress
Parts:
- removed R21: 33, Resistor_SMD:R_0603_1608Metric_Pad0.98x0.95mm_HandSolder
- PS1: moved to B.Cu
- moved R45 301.5 mm to (29.2, 129.2), turned to 180 degrees
- moved C79 299.8 mm to (33.0, 129.2), turned to 0 degrees
- moved J10 295.7 mm to (15.8, 121.8), turned to 0 degrees
- moved J9 292.9 mm to (31.2, 121.8), turned to 0 degrees
- moved T1 282.5 mm to (18.2, 133.0), turned to 90 degrees
- moved C80 266.6 mm to (27.5, 135.5), turned to 180 degrees
- moved R47 263.3 mm to (28.2, 132.8), turned to 90 degrees
- moved R46 259.5 mm to (31.2, 135.5), turned to 180 degrees
- moved PS1 207.8 mm to (168.5, 193.2), turned to 90 degrees
- moved F1 206.8 mm to (179.8, 169.8)
- moved C50 198.9 mm to (73.8, 174.2), turned to 270 degrees
- moved C37 198.5 mm to (146.0, 149.0), turned to 180 degrees
- moved C62 198.4 mm to (76.0, 140.0)
- moved C63 198.4 mm to (78.2, 140.0)
- moved C64 198.4 mm to (73.8, 140.0)
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Connections:
- J3 pad 38: Net-(J3-Pad38) -> /PI_SDATA_I
Routing:
- net +24V: track 19.1 -> 166.9 mm, vias 7 -> 14
- net +3.3VA: track 1.94 -> 139.0 mm
- net +5VD: track 26.6 -> 102.9 mm
- net GND: track 72.2 -> 142.7 mm, vias 17 -> 34
- net /DVDD: track 0.00 -> 32.5 mm
- net +3V3: track 33.1 -> 58.1 mm, vias 18 -> 20
- net /AMP2_SDIN: track 0.00 -> 19.0 mm
- net Net-(J8-Pad2): track 0.00 -> 18.4 mm
- net /AMP2_BCLK: track 0.00 -> 13.9 mm
- net Net-(J8-Pad3): track 0.00 -> 11.9 mm
- net Net-(C79-Pad1): track 0.00 -> 11.4 mm
- net Net-(J10-Pad1): track 9.62 -> 17.7 mm
- net /VDRIVE: track 0.00 -> 8.04 mm
- net Net-(R7-Pad2): track 0.00 -> 7.67 mm
- net Net-(R11-Pad2): track 0.00 -> 7.46 mm
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- added copper zone on F.Cu, net /I2S-AMP-2CH-A/SKP_OUTA+
- added copper zone on F.Cu, net /I2S-AMP-2CH-A/SKP_OUTA-
- added copper zone on F.Cu, net /I2S-AMP-2CH-A/SKP_OUTB+
- added copper zone on F.Cu, net /I2S-AMP-2CH-A/SKP_OUTB-
- added copper zone on F.Cu, net Net-(C54-Pad2)
- added copper zone on F.Cu, net Net-(C55-Pad2)
- added copper zone on F.Cu, net Net-(C56-Pad2)
- added copper zone on F.Cu, net Net-(C57-Pad2)

Commit message: routing, added 4 layers
Parts:
- removed R43: 33, Resistor_SMD:R_0603_1608Metric_Pad0.98x0.95mm_HandSolder
- J1, J2: moved to B.Cu
- J3: footprint Connector_PinHeader_2.54mm:PinHeader_2x20_P2.54mm_Vertical -> rpi_socket:PinSocket_2x20_P2.54mm_Vertical; moved to B.Cu
- moved J1 144.4 mm to (132.8, 119.2)
- moved R18 141.3 mm to (81.8, 63.8)
- moved R16 134.6 mm to (77.2, 63.8), turned to 180 degrees
- moved R1 126.0 mm to (118.0, 124.0)
- moved C22 117.2 mm to (100.5, 83.2), turned to 180 degrees
- moved FB1 114.0 mm to (102.2, 88.5)
- moved C1 112.3 mm to (100.5, 86.2), turned to 180 degrees
- moved J3 100.5 mm to (92.8, 137.8), turned to 90 degrees
- moved R20 87.9 mm to (73.8, 132.8), turned to 90 degrees
- moved R19 80.2 mm to (126.5, 108.5), turned to 270 degrees
- moved J8 78.8 mm to (128.2, 75.5), turned to 0 degrees
- moved R17 77.7 mm to (124.8, 108.5), turned to 270 degrees
- moved R22 77.4 mm to (70.0, 132.8), turned to 90 degrees
- moved J2 75.9 mm to (65.5, 66.5), turned to 270 degrees
- moved R2 75.2 mm to (123.0, 108.5), turned to 90 degrees
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Connections:
- R23 pad 2: /AMP1_CLOCK -> /DSP_CLOCK
- R25 pad 2: /DSP_CLOCK -> /AMP1_CLOCK
- U9 pad 18: Net-(R43-Pad2) -> (no net)
Routing:
- net /SCL: track 0.00 -> 135.7 mm, vias 0 -> 2
- net /SDA: track 0.00 -> 135.1 mm, vias 0 -> 2
- net +24V: track 166.9 -> 38.1 mm
- net /EXT_MCLK: track 0.00 -> 88.2 mm
- net GND: track 142.7 -> 226.0 mm, vias 34 -> 93
- net /PI_SDATA_I: track 0.00 -> 80.9 mm, vias 0 -> 1
- net +5VD: track 102.9 -> 26.6 mm
- net /EXT_MDO: track 0.00 -> 76.3 mm, vias 0 -> 1
- net /DSP_NRESET: track 0.00 -> 75.9 mm, vias 0 -> 2
- net /PI_SDATA_O: track 0.00 -> 74.8 mm, vias 0 -> 2
- net /PI_LRCLK: track 0.00 -> 67.3 mm, vias 0 -> 2
- net /EXT_MDI: track 0.00 -> 65.9 mm, vias 0 -> 1
- net /DSP_SELFBOOT: track 0.00 -> 61.7 mm, vias 0 -> 2
- net /EXT_BCLK: track 0.00 -> 58.0 mm, vias 0 -> 1
- net /AMP1_LRCLK: track 0.00 -> 56.7 mm
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- added copper zone on In1.Cu, net +3.3VA
- added copper zone on In1.Cu, net +3V3
- added copper zone on In1.Cu, net /DVDD
- added copper zone on In2.Cu, net GND
Other:
- board outline added: 182.5 x 95 mm
- copper layers 2 -> 4

Commit message: complete
Parts:
- C53, C67, F1, J4, J5, J6, J7: moved to B.Cu
- moved R29 16.0 mm to (133.5, 140.2), turned to 90 degrees
- moved R27 15.8 mm to (135.2, 140.2), turned to 90 degrees
- moved R30 12.6 mm to (133.5, 143.9), turned to 90 degrees
- moved F1 12.5 mm to (236.5, 137.5), turned to 90 degrees
- moved R28 12.4 mm to (135.2, 143.9), turned to 90 degrees
- moved J2 6.00 mm to (71.5, 66.5)
- moved R16 6.00 mm to (83.2, 63.8)
- moved R18 6.00 mm to (87.8, 63.8)
- moved J1 4.03 mm to (128.8, 118.8)
- moved R41 1.25 mm to (110.8, 67.5), turned to 270 degrees
- moved C48 1.00 mm to (132.0, 129.5)
- moved C49 1.00 mm to (134.2, 129.5)
- moved C50 1.00 mm to (129.8, 129.5)
- moved C62 1.00 mm to (132.0, 95.2)
- moved C63 1.00 mm to (134.2, 95.2)
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Routing:
- net +3.3VA: track 154.2 -> 29.4 mm, vias 5 -> 11
- net +24V: track 38.1 -> 126.6 mm
- net /GAIN0: track 2.93 -> 52.6 mm, vias 1 -> 3
- net /GAIN1: track 2.93 -> 49.9 mm, vias 1 -> 3
- net /VPOT0: track 1.77 -> 34.7 mm
- net Net-(C64-Pad1): track 0.00 -> 24.6 mm
- net Net-(C50-Pad1): track 0.00 -> 24.2 mm
- net /Power/AC_L: track 0.00 -> 19.2 mm
- net /VPOT1: track 1.19 -> 17.9 mm
- net /SCL: track 135.7 -> 126.4 mm
- net /EXT_MCLK: track 88.2 -> 95.3 mm
- net /SDA: track 135.1 -> 128.0 mm
- net /AMP1_SDIN: track 48.2 -> 54.2 mm
- net /AMP1_LRCLK: track 56.7 -> 62.7 mm
- net /AMP1_BCLK: track 52.2 -> 58.2 mm
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- added copper zone on In1.Cu, net +5VD
Other:
- board text added: "+ A -"
- board text added: "+ C -"
- board text added: "- B +"
- board text added: "- D +"
- board text added: "0"
- board text added: "1"
- board text added: "GAIN0"
- board text added: "GAIN1"
- board text added: "IN"
- board text added: "OUT"
- board text added: "af 2021"
- board text added: "soundi v0.1"

Commit message: bugfixes, made smaller
Parts:
- removed C78: 100n, Capacitor_SMD:C_0603_1608Metric_Pad1.08x0.95mm_HandSolder
- added C81: 10n, Capacitor_SMD:C_0603_1608Metric_Pad1.08x0.95mm_HandSolder, F.Cu at (104.8, 128.5)
- added C82: 100n, Capacitor_SMD:C_0603_1608Metric_Pad1.08x0.95mm_HandSolder, F.Cu at (106.5, 128.5)
- added C83: 10u, Capacitor_SMD:C_1206_3216Metric_Pad1.33x1.80mm_HandSolder, F.Cu at (119.2, 69.0)
- added C84: 10u, Capacitor_SMD:C_1206_3216Metric_Pad1.33x1.80mm_HandSolder, F.Cu at (103.7, 81.8)
- added C85: 10u, Capacitor_SMD:C_1206_3216Metric_Pad1.33x1.80mm_HandSolder, F.Cu at (114.8, 66.0)
- added C86: 100n, Capacitor_SMD:C_0603_1608Metric_Pad1.08x0.95mm_HandSolder, F.Cu at (114.8, 68.2)
- added C87: 100n, Capacitor_SMD:C_0603_1608Metric_Pad1.08x0.95mm_HandSolder, F.Cu at (103.8, 79.5)
- added C88: 1u, Capacitor_SMD:C_0805_2012Metric_Pad1.18x1.45mm_HandSolder, F.Cu at (117.8, 73.0)
- added C89: 1u, Capacitor_SMD:C_0805_2012Metric_Pad1.18x1.45mm_HandSolder, F.Cu at (117.8, 77.0)
- moved R16 69.5 mm to (123.8, 120.2), turned to 270 degrees
- moved R18 68.0 mm to (125.5, 120.2), turned to 270 degrees
- moved RV1 15.1 mm to (64.0, 107.0), turned to 0 degrees
- moved PS1 5.59 mm to (226.5, 143.0)
- moved F1 4.28 mm to (237.0, 133.2)
- moved C22 3.26 mm to (97.2, 83.0)
Connections:
- U6 pad 9: +3V3 -> GND
- U7 pad 9: +3V3 -> GND
Routing:
- net GND: track 228.9 -> 248.7 mm, vias 93 -> 121
- net /Power/AC_L: track 19.2 -> 0.00 mm
- net /VPOT0: track 34.7 -> 48.9 mm
- net +3V3: track 105.0 -> 117.1 mm
- net /SDA: track 128.0 -> 134.4 mm
- net /SCL: track 126.4 -> 129.9 mm
- net +24V: track 126.6 -> 124.8 mm
- net Net-(C83-Pad1): track 2.73 -> 3.86 mm
- net /USB_LRCLK: track 33.4 -> 32.3 mm
- net +5VD: vias 10 -> 6
- net +3.3VA: vias 11 -> 17
- added copper zone on In1.Cu, net GND
Other:
- board size 182.5 x 95 mm -> 182.5 x 90 mm
- board text added: "+3.3VA"
- board text added: "+5VA"
- board text added: "+5VD"
- board text added: "+DC-"
- board text added: "AC"
- board text added: "EXT"
- board text added: "POWER"
- board text added: "RPi"
- board text added: "S/PDIF"
- board text added: "USB-I2S"
- board text added: "USBi"
