File: Hardware/SPDIF.sch (KiCad schematic (older format))
At the start: 7 parts, among them P11 FCR684205T, P12 FCR684205R

Commit message: started routing
Parts:
- removed C56: 100n, Capacitor_SMD:C_0603_1608Metric_Pad1.08x0.95mm_HandSolder, symbol dsp-amplifier-x4-rescue:C
- removed FB2, FB4: 600/100M, Inductor_SMD:L_0805_2012Metric_Pad1.05x1.20mm_HandSolder, symbol Device:Ferrite_Bead
- removed P11: FCR684205T, FCR684205:FC684205_R_T, symbol dsp-amplifier-x4-rescue:FCR684205T
- removed P12: FCR684205R, FCR684205:FC684205_R_T, symbol dsp-amplifier-x4-rescue:FCR684205R
- removed R8: 33, Resistor_SMD:R_0603_1608Metric_Pad0.98x0.95mm_HandSolder, symbol Device:R
- added C80: 10n, Capacitor_SMD:C_0603_1608Metric_Pad1.08x0.95mm_HandSolder, symbol Device:C
- added J10, J9: Conn_Coaxial, connectors_audio:cui_rcj_02x, symbol Connector:Conn_Coaxial
- added R45: 75, Resistor_SMD:R_0603_1608Metric_Pad0.98x0.95mm_HandSolder, symbol Device:R
- added R46: 243, Resistor_SMD:R_0603_1608Metric_Pad0.98x0.95mm_HandSolder, symbol Device:R
- added R47: 107, Resistor_SMD:R_0603_1608Metric_Pad0.98x0.95mm_HandSolder, symbol Device:R
- added T1: DA100J, da100j:SOIC-6, symbol transformer_audio:DA100J
- C79: renamed from C54; value 100n -> 10n; symbol dsp-amplifier-x4-rescue:C -> Device:C
Connections:
- net GND: now also J9.2 (Ext), R45.2, R47.2, T1.3 (InRet); no longer C79.2
- net SPDIF_IN: now also C79.2
- net SPDIF_OUT: now also R46.1
- net at C79.1: now also J9.1 (In), R45.1
- new net: C80.2, T1.1 (In)
- new net: J10.2 (Ext), T1.4 (OutRet)
- new net: J10.1 (In), T1.6 (Out)
- new net: C80.1, R46.2, R47.1
Other:
- moved on the sheet: C79

Commit message: hardware bugfixes
Parts:
- renumbered C79 to C85, C80 to C86, R45 to R41, R46 to R42, R47 to R43
Changed lines of the file:
@@
 $EndComp
 $Comp
-L power:GND #PWR0115
+L power:GND #PWR0107
 U 1 1 60DEB8DA
 P 3500 4050
-F 0 "#PWR0115" H 3500 3800 50  0001 C CNN
+F 0 "#PWR0107" H 3500 3800 50  0001 C CNN
 F 1 "GND" H 3500 3900 50  0000 C CNN
 F 2 "" H 3500 4050 60  0000 C CNN
@@
 	3500 4050 3500 4000
 $Comp
-L Device:C C79
+L Device:C C85
 U 1 1 5B17A13D
 P 4200 3500
-F 0 "C79" H 4225 3600 50  0000 L CNN
+F 0 "C85" H 4225 3600 50  0000 L CNN
 F 1 "10n" H 4225 3400 50  0000 L CNN
 F 2 "Capacitor_SMD:C_0603_1608Metric_Pad1.08x0.95mm_HandSolder" H 4238 3350 30  0001 C CNN
@@
 P 3850 3800
 AR Path="/606A5C2E" Ref="R?"  Part="1"
-AR Path="/5AFACEFB/606A5C2E" Ref="R45"  Part="1"
-F 0 "R45" V 3643 3800 50  0000 C CNN
+AR Path="/5AFACEFB/606A5C2E" Ref="R41"  Part="1"
+F 0 "R41" V 3643 3800 50  0000 C CNN
 F 1 "75" V 3734 3800 50  0000 C CNN
 F 2 "Resistor_SMD:R_0603_1608Metric_Pad0.98x0.95mm_HandSolder" V 3780 3800 50  0001 C CNN
@@
 	7750 3700 8000 3700
 $Comp
-L power:GND #PWR0117
+L power:GND #PWR0109
 U 1 1 606B3C38
 P 6700 3750
-F 0 "#PWR0117" H 6700 3500 50  0001 C CNN
+F 0 "#PWR0109" H 6700 3500 50  0001 C CNN
 F 1 "GND" H 6700 3600 50  0000 C CNN
 F 2 "" H 6700 3750 60  0000 C CNN
@@
 	6750 3700 6700 3700
 $Comp
-L Device:C C80
+L Device:C C86
 U 1 1 606B665C
 P 6550 3500
-F 0 "C80" H 6575 3600 50  0000 L CNN
+F 0 "C86" H 6575 3600 50  0000 L CNN
 F 1 "10n" H 6575 3400 50  0000 L CNN
 F 2 "Capacitor_SMD:C_0603_1608Metric_Pad1.08x0.95mm_HandSolder" H 6588 3350 30  0001 C CNN
@@
 P 6350 3700
 AR Path="/606B7B41" Ref="R?"  Part="1"
-AR Path="/5AFACEFB/606B7B41" Ref="R47"  Part="1"
-F 0 "R47" V 6143 3700 50  0000 C CNN
+AR Path="/5AFACEFB/606B7B41" Ref="R43"  Part="1"
+F 0 "R43" V 6143 3700 50  0000 C CNN
 F 1 "107" V 6234 3700 50  0000 C CNN
 F 2 "Resistor_SMD:R_0603_1608Metric_Pad0.98x0.95mm_HandSolder" V 6280 3700 50  0001 C CNN
@@
 P 6350 3300
 AR Path="/606B8671" Ref="R?"  Part="1"
-AR Path="/5AFACEFB/606B8671" Ref="R46"  Part="1"
-F 0 "R46" V 6143 3300 50  0000 C CNN
+AR Path="/5AFACEFB/606B8671" Ref="R42"  Part="1"
+F 0 "R42" V 6143 3300 50  0000 C CNN
 F 1 "243" V 6234 3300 50  0000 C CNN
 F 2 "Resistor_SMD:R_0603_1608Metric_Pad0.98x0.95mm_HandSolder" V 6280 3300 50  0001 C CNN
@@
 	6350 3500 6350 3550
 $Comp
-L power:GND #PWR0116
+L power:GND #PWR0108
 U 1 1 606B988D
 P 6350 3900
-F 0 "#PWR0116" H 6350 3650 50  0001 C CNN
+F 0 "#PWR0108" H 6350 3650 50  0001 C CNN
 F 1 "GND" H 6350 3750 50  0000 C CNN
 F 2 "" H 6350 3900 60  0000 C CNN
