File: Hardware/clock.sch (KiCad schematic (older format))
At the start: 7 parts, among them U3 SI53365, X1 ASV-24.576MHz-EJ-T

Commit message: started routing
Parts:
- removed C1: 10u, Capacitor_SMD:C_0805_2012Metric_Pad1.18x1.45mm_HandSolder, symbol dsp-amplifier-x4-rescue:C
- removed FB3: 600/100M, Inductor_SMD:L_0805_2012Metric_Pad1.05x1.20mm_HandSolder, symbol Device:Ferrite_Bead
- added C46: 100n, Capacitor_SMD:C_0603_1608Metric_Pad1.08x0.95mm_HandSolder, symbol Device:C
- added C47: 10n, Capacitor_SMD:C_0603_1608Metric_Pad1.08x0.95mm_HandSolder, symbol Device:C
- C43: renamed from C3; footprint Capacitor_SMD:C_0603_1608Metric_Pad1.08x0.95mm_HandSolder -> Capacitor_SMD:C_0805_2012Metric_Pad1.18x1.45mm_HandSolder
- C44: renamed from C4; footprint Capacitor_SMD:C_0603_1608Metric_Pad1.08x0.95mm_HandSolder -> Capacitor_SMD:C_0805_2012Metric_Pad1.18x1.45mm_HandSolder
- C45: renamed from C14; footprint Capacitor_SMD:C_0603_1608Metric_Pad1.08x0.95mm_HandSolder -> Capacitor_SMD:C_0805_2012Metric_Pad1.18x1.45mm_HandSolder
- X1: footprint fdsp_crystal-oscillator_new:Oscillator_SMD_Abracon_ASV-4pin_7.0x5.1mm_HandSoldering -> Oscillator:Oscillator_SMD_Abracon_ASV-4Pin_7.0x5.1mm; symbol dsp-amplifier-x4-rescue:Crystal_Oszillator -> Oscillator:ASV-xxxMHz
- renumbered U3 to U5
Connections:
- net +3V3: now also X1.1 (EN), X1.4 (Vdd), C46.1, C47.1
- net GND: now also C46.2, C47.2
Other:
- moved on the sheet: C43, C44, C45

Commit message: hardware bugfixes
Parts:
- renumbered U5 to U6
Changed lines of the file:
@@
 	6550 3200 5500 3200
 $Comp
-L power:GND #PWR071
+L power:GND #PWR066
 U 1 1 6065E986
 P 6900 4200
-F 0 "#PWR071" H 6900 3950 50  0001 C CNN
+F 0 "#PWR066" H 6900 3950 50  0001 C CNN
 F 1 "GND" H 6900 4050 50  0000 C CNN
 F 2 "" H 6900 4200 60  0000 C CNN
@@
 	6900 4150 6900 4200
 $Comp
-L power:GND #PWR068
+L power:GND #PWR063
 U 1 1 6065F931
 P 5200 3750
-F 0 "#PWR068" H 5200 3500 50  0001 C CNN
+F 0 "#PWR063" H 5200 3500 50  0001 C CNN
 F 1 "GND" H 5200 3600 50  0000 C CNN
 F 2 "" H 5200 3750 60  0000 C CNN
@@
 $EndComp
 $Comp
-L power:+3V3 #PWR067
+L power:+3V3 #PWR062
 U 1 1 606634F4
 P 4600 2500
-F 0 "#PWR067" H 4600 2350 50  0001 C CNN
+F 0 "#PWR062" H 4600 2350 50  0001 C CNN
 F 1 "+3V3" H 4600 2640 50  0000 C CNN
 F 2 "" H 4600 2500 60  0000 C CNN
@@
 $EndComp
 $Comp
-L power:+3V3 #PWR070
+L power:+3V3 #PWR065
 U 1 1 60667485
 P 6900 2250
-F 0 "#PWR070" H 6900 2100 50  0001 C CNN
+F 0 "#PWR065" H 6900 2100 50  0001 C CNN
 F 1 "+3V3" H 6900 2390 50  0000 C CNN
 F 2 "" H 6900 2250 60  0000 C CNN
@@
 	7250 3900 7500 3900
 $Comp
-L buffers:SI53365 U5
+L buffers:SI53365 U6
 U 1 1 60656034
 P 6900 3300
-F 0 "U5" H 6900 4253 60  0000 C CNN
+F 0 "U6" H 6900 4253 60  0000 C CNN
 F 1 "SI53365" H 6900 4147 60  0000 C CNN
 F 2 "Package_SO:TSSOP-16_4.4x5mm_P0.65mm" H 6900 3650 60  0001 C CNN
@@
 $EndComp
 $Comp
-L power:+3V3 #PWR069
+L power:+3V3 #PWR064
 U 1 1 6066D5DA
 P 6450 3100
-F 0 "#PWR069" H 6450 2950 50  0001 C CNN
+F 0 "#PWR064" H 6450 2950 50  0001 C CNN
 F 1 "+3V3" H 6450 3240 50  0000 C CNN
 F 2 "" H 6450 3100 60  0000 C CNN
@@
 	6450 3300 6550 3300
 $Comp
-L power:+3V3 #PWR065
+L power:+3V3 #PWR060
 U 1 1 6067464E
 P 4350 1050
-F 0 "#PWR065" H 4350 900 50  0001 C CNN
+F 0 "#PWR060" H 4350 900 50  0001 C CNN
 F 1 "+3V3" H 4350 1190 50  0000 C CNN
 F 2 "" H 4350 1050 60  0000 C CNN
@@
 	5150 1100 5150 1200
 $Comp
-L power:GND #PWR066
+L power:GND #PWR061
 U 1 1 60675B90
 P 4350 1650
-F 0 "#PWR066" H 4350 1400 50  0001 C CNN
+F 0 "#PWR061" H 4350 1400 50  0001 C CNN
 F 1 "GND" H 4350 1500 50  0000 C CNN
 F 2 "" H 4350 1650 60  0000 C CNN
