File: Hardware/i2c_eeprom.sch (KiCad schematic (older format))
At the start: 1 part, among them U2 24LC1025

Commit message: started routing
Parts:
- renumbered U2 to U10
Changed lines of the file:
@@
 $Descr A4 11693 8268
 encoding utf-8
-Sheet 6 7
+Sheet 7 8
 Title ""
 Date ""
@@
 $EndDescr
 $Comp
-L Memory_EEPROM:24LC1025 U2
+L Memory_EEPROM:24LC1025 U10
 U 1 1 619E8E3D
 P 2700 2350
-F 0 "U2" H 2700 2831 50  0000 C CNN
+F 0 "U10" H 2700 2831 50  0000 C CNN
 F 1 "24LC1025" H 2700 2740 50  0000 C CNN
 F 2 "Package_SO:SO-8_5.3x6.2mm_P1.27mm" H 2700 2350 50  0001 C CNN
@@
 $EndComp
 $Comp
-L power:+3.3V #PWR0109
+L power:+3.3V #PWR0112
 U 1 1 619E8E43
 P 2700 1800
-F 0 "#PWR0109" H 2700 1650 50  0001 C CNN
+F 0 "#PWR0112" H 2700 1650 50  0001 C CNN
 F 1 "+3.3V" H 2715 1973 50  0000 C CNN
 F 2 "" H 2700 1800 50  0001 C CNN
@@
 	2700 1800 2700 2050
 $Comp
-L dsp-amplifier-x4-rescue:GND #PWR0111
+L power:GND #PWR0113
 U 1 1 619E8E4A
 P 2700 2700
-F 0 "#PWR0111" H 2700 2450 50  0001 C CNN
+F 0 "#PWR0113" H 2700 2450 50  0001 C CNN
 F 1 "GND" H 2700 2550 50  0000 C CNN
 F 2 "" H 2700 2700 50  0001 C CNN
@@
 	2700 2650 2700 2700
 $Comp
-L power:+3.3V #PWR0127
+L power:+3.3V #PWR0111
 U 1 1 619E8E55
 P 2050 1800
-F 0 "#PWR0127" H 2050 1650 50  0001 C CNN
+F 0 "#PWR0111" H 2050 1650 50  0001 C CNN
 F 1 "+3.3V" H 2065 1973 50  0000 C CNN
 F 2 "" H 2050 1800 50  0001 C CNN
@@
 	2050 2450 2300 2450
 $Comp
-L dsp-amplifier-x4-rescue:GND #PWR0128
+L power:GND #PWR0114
 U 1 1 619E8E5D
 P 3150 2700
-F 0 "#PWR0128" H 3150 2450 50  0001 C CNN
+F 0 "#PWR0114" H 3150 2450 50  0001 C CNN
 F 1 "GND" H 3150 2550 50  0000 C CNN
 F 2 "" H 3150 2700 50  0001 C CNN

Commit message: bugfixes, made smaller
Parts:
- added C81: 10n, Capacitor_SMD:C_0603_1608Metric_Pad1.08x0.95mm_HandSolder, symbol Device:C
- added C82: 100n, Capacitor_SMD:C_0603_1608Metric_Pad1.08x0.95mm_HandSolder, symbol Device:C
Connections:
- net +3V3: now also C81.1, C82.1
- net GND: now also C81.2, C82.2
Changed lines of the file:
@@
 Wire Wire Line
 	3100 2350 3150 2350
+$Comp
+L Device:C C?
+U 1 1 60A729EF
+P 4150 2400
+AR Path="/5AF9FF80/60A729EF" Ref="C?"  Part="1"
+AR Path="/60A729EF" Ref="C?"  Part="1"
+AR Path="/619C0687/60A729EF" Ref="C81"  Part="1"
+F 0 "C81" H 4200 2500 50  0000 L CNN
+F 1 "10n" H 4200 2300 50  0000 L CNN
+F 2 "Capacitor_SMD:C_0603_1608Metric_Pad1.08x0.95mm_HandSolder" V 3850 2540 50  0001 C CNN
+F 3 "~" V 3850 2540 50  0001 C CNN
+F 4 "GRM31CR71H475KA12L" H 4150 2400 60  0001 C CNN "Mfr.Nr."
+	1    4150 2400
+	1    0    0    -1
+$EndComp
+$Comp
+L Device:C C?
+U 1 1 60A729F6
+P 4500 2400
+AR Path="/5AF9FF80/60A729F6" Ref="C?"  Part="1"
+AR Path="/60A729F6" Ref="C?"  Part="1"
+AR Path="/619C0687/60A729F6" Ref="C82"  Part="1"
+F 0 "C82" H 4550 2500 50  0000 L CNN
+F 1 "100n" H 4550 2300 50  0000 L CNN
+F 2 "Capacitor_SMD:C_0603_1608Metric_Pad1.08x0.95mm_HandSolder" V 4200 2540 50  0001 C CNN
+F 3 "~" V 4200 2540 50  0001 C CNN
+F 4 "GRM31CR71H475KA12L" H 4500 2400 60  0001 C CNN "Mfr.Nr."
+	1    4500 2400
+	1    0    0    -1
+$EndComp
+Wire Wire Line
+	4500 2150 4500 2250
+Wire Wire Line
+	4150 2250 4150 2150
+Connection ~ 4150 2150
+Wire Wire Line
+	4150 2150 4500 2150
+$Comp
+L power:GND #PWR?
+U 1 1 60A72A00
+P 4150 2650
+AR Path="/60A72A00" Ref="#PWR?"  Part="1"
+AR Path="/619C0687/60A72A00" Ref="#PWR0118"  Part="1"
+F 0 "#PWR0118" H 4150 2400 50  0001 C CNN
+F 1 "GND" H 4150 2500 50  0000 C CNN
+F 2 "" H 4150 2650 50  0001 C CNN
+F 3 "" H 4150 2650 50  0001 C CNN
+	1    4150 2650
+	1    0    0    -1
+$EndComp
+Wire Wire Line
+	4150 1850 4150 2150
+Wire Wire Line
+	4150 2550 4150 2600
+Wire Wire Line
+	4150 2600 4500 2600
+Wire Wire Line
+	4500 2600 4500 2550
+Connection ~ 4150 2600
+Wire Wire Line
+	4150 2600 4150 2650
+$Comp
+L power:+3.3V #PWR0119
+U 1 1 60A72BB3
+P 4150 1850
+F 0 "#PWR0119" H 4150 1700 50  0001 C CNN
+F 1 "+3.3V" H 4165 2023 50  0000 C CNN
+F 2 "" H 4150 1850 50  0001 C CNN
+F 3 "" H 4150 1850 50  0001 C CNN
+	1    4150 1850
+	1    0    0    -1
+$EndComp
 $EndSCHEMATC

Commit message: style fixes, spi/i2c
Parts:
- removed U10: 24LC1025, Package_SO:SO-8_5.3x6.2mm_P1.27mm, symbol Memory_EEPROM:24LC1025
- added U10: 25LCxxx, Package_SO:SOIC-8_5.275x5.275mm_P1.27mm, symbol Memory_EEPROM:25LCxxx
Connections:
- net +3V3: now also U10.3 (~WP), U10.7 (~HOLD), U10.8 (VCC)
- net GND: now also U10.4 (GND)
- new net EEPROM_MISO: U10.2 (MISO)
- new net EEPROM_MOSI: U10.5 (MOSI)
- new net EEPROM_NCS: U10.1 (~CS)
- new net EEPROM_SCK: U10.6 (SCK)
Changed lines of the file:
@@
 $Descr A4 11693 8268
 encoding utf-8
-Sheet 7 8
+Sheet 8 8
 Title ""
 Date ""
@@
 Comment4 ""
 $EndDescr
-$Comp
-L Memory_EEPROM:24LC1025 U10
-U 1 1 619E8E3D
-P 2700 2350
-F 0 "U10" H 2700 2831 50  0000 C CNN
-F 1 "24LC1025" H 2700 2740 50  0000 C CNN
-F 2 "Package_SO:SO-8_5.3x6.2mm_P1.27mm" H 2700 2350 50  0001 C CNN
-F 3 "http://ww1.microchip.com/downloads/en/DeviceDoc/21941B.pdf" H 2700 2350 50  0001 C CNN
-	1    2700 2350
-	1    0    0    -1
-$EndComp
 $Comp
 L power:+3.3V #PWR0112
@@
 	1    0    0    -1
 $EndComp
-Wire Wire Line
-	2700 1800 2700 2050
 $Comp
 L power:GND #PWR0113
@@
 	1    0    0    -1
 $EndComp
-Wire Wire Line
-	2700 2650 2700 2700
 $Comp
 L power:+3.3V #PWR0111
 U 1 1 619E8E55
-P 2050 1800
-F 0 "#PWR0111" H 2050 1650 50  0001 C CNN
-F 1 "+3.3V" H 2065 1973 50  0000 C CNN
-F 2 "" H 2050 1800 50  0001 C CNN
-F 3 "" H 2050 1800 50  0001 C CNN
-	1    2050 1800
+P 1750 1750
+F 0 "#PWR0111" H 1750 1600 50  0001 C CNN
+F 1 "+3.3V" H 1765 1923 50  0000 C CNN
+F 2 "" H 1750 1750 50  0001 C CNN
+F 3 "" H 1750 1750 50  0001 C CNN
+	1    1750 1750
 	1    0    0    -1
 $EndComp
 Wire Wire Line
-	2050 1800 2050 2250
-Wire Wire Line
-	2050 2450 2300 2450
-$Comp
-L power:GND #PWR0114
-U 1 1 619E8E5D
-P 3150 2700
-F 0 "#PWR0114" H 3150 2450 50  0001 C CNN
-F 1 "GND" H 3150 2550 50  0000 C CNN
-F 2 "" H 3150 2700 50  0001 C CNN
-F 3 "" H 3150 2700 50  0001 C CNN
-	1    3150 2700
-	1    0    0    -1
-$EndComp
-Wire Wire Line
-	3100 2450 3150 2450
-Wire Wire Line
-	3150 2450 3150 2700
-Wire Wire Line
-	2300 2350 2050 2350
-Connection ~ 2050 2350
-Wire Wire Line
-	2050 2350 2050 2450
-Wire Wire Line
-	2050 2250 2300 2250
-Connection ~ 2050 2250
-Wire Wire Line
-	2050 2250 2050 2350
-Text HLabel 3150 2250 2    60   BiDi ~ 0
-EEPROM_SDA
-Text HLabel 3150 2350 2    60   BiDi ~ 0
-EEPROM_SCL
-Wire Wire Line
-	3150 2250 3100 2250
-Wire Wire Line
-	3100 2350 3150 2350
+	1750 1750 1750 2200
+Text HLabel 3150 2200 2    60   Input ~ 0
+EEPROM_SCK
+Text HLabel 3150 2300 2    60   Input ~ 0
+EEPROM_MOSI
 $Comp
 L Device:C C?
@@
 	1    0    0    -1
 $EndComp
+$Comp
+L Memory_EEPROM:25LCxxx U10
+U 1 1 60A473E7
+P 2700 2300
+F 0 "U10" H 2700 2781 50  0000 C CNN
+F 1 "25LCxxx" H 2700 2690 50  0000 C CNN
+F 2 "Package_SO:SOIC-8_5.275x5.275mm_P1.27mm" H 2700 2300 50  0001 C CNN
+F 3 "http://ww1.microchip.com/downloads/en/DeviceDoc/21832H.pdf" H 2700 2300 50  0001 C CNN
+	1    2700 2300
+	1    0    0    -1
+$EndComp
+Wire Wire Line
+	2700 2600 2700 2700
+Wire Wire Line
+	3150 2200 3100 2200
+Text HLabel 3150 2400 2    60   Output ~ 0
+EEPROM_MISO
+Wire Wire Line
+	3150 2300 3100 2300
+Wire Wire Line
+	3100 2400 3150 2400
+Text HLabel 2250 2400 0    60   Input ~ 0
+EEPROM_NCS
+Wire Wire Line
+	2300 2400 2250 2400
+Wire Wire Line
+	1750 2200 2300 2200
+Wire Wire Line
+	2300 2300 1750 2300
+Wire Wire Line
+	1750 2300 1750 2200
+Connection ~ 1750 2200
+Wire Wire Line
+	2700 2000 2700 1800
 $EndSCHEMATC

Commit message: hardware bugfixes
Parts:
- renumbered C81 to C87, C82 to C88, U10 to U11
Changed lines of the file:
@@
 $EndDescr
 $Comp
-L power:+3.3V #PWR0112
+L power:+3.3V #PWR0111
 U 1 1 619E8E43
 P 2700 1800
-F 0 "#PWR0112" H 2700 1650 50  0001 C CNN
+F 0 "#PWR0111" H 2700 1650 50  0001 C CNN
 F 1 "+3.3V" H 2715 1973 50  0000 C CNN
 F 2 "" H 2700 1800 50  0001 C CNN
@@
 $EndComp
 $Comp
-L power:GND #PWR0113
+L power:GND #PWR0112
 U 1 1 619E8E4A
 P 2700 2700
-F 0 "#PWR0113" H 2700 2450 50  0001 C CNN
+F 0 "#PWR0112" H 2700 2450 50  0001 C CNN
 F 1 "GND" H 2700 2550 50  0000 C CNN
 F 2 "" H 2700 2700 50  0001 C CNN
@@
 $EndComp
 $Comp
-L power:+3.3V #PWR0111
+L power:+3.3V #PWR0110
 U 1 1 619E8E55
 P 1750 1750
-F 0 "#PWR0111" H 1750 1600 50  0001 C CNN
+F 0 "#PWR0110" H 1750 1600 50  0001 C CNN
 F 1 "+3.3V" H 1765 1923 50  0000 C CNN
 F 2 "" H 1750 1750 50  0001 C CNN
@@
 AR Path="/5AF9FF80/60A729EF" Ref="C?"  Part="1"
 AR Path="/60A729EF" Ref="C?"  Part="1"
-AR Path="/619C0687/60A729EF" Ref="C81"  Part="1"
-F 0 "C81" H 4200 2500 50  0000 L CNN
+AR Path="/619C0687/60A729EF" Ref="C87"  Part="1"
+F 0 "C87" H 4200 2500 50  0000 L CNN
 F 1 "10n" H 4200 2300 50  0000 L CNN
 F 2 "Capacitor_SMD:C_0603_1608Metric_Pad1.08x0.95mm_HandSolder" V 3850 2540 50  0001 C CNN
@@
 AR Path="/5AF9FF80/60A729F6" Ref="C?"  Part="1"
 AR Path="/60A729F6" Ref="C?"  Part="1"
-AR Path="/619C0687/60A729F6" Ref="C82"  Part="1"
-F 0 "C82" H 4550 2500 50  0000 L CNN
+AR Path="/619C0687/60A729F6" Ref="C88"  Part="1"
+F 0 "C88" H 4550 2500 50  0000 L CNN
 F 1 "100n" H 4550 2300 50  0000 L CNN
 F 2 "Capacitor_SMD:C_0603_1608Metric_Pad1.08x0.95mm_HandSolder" V 4200 2540 50  0001 C CNN
@@
 P 4150 2650
 AR Path="/60A72A00" Ref="#PWR?"  Part="1"
-AR Path="/619C0687/60A72A00" Ref="#PWR0118"  Part="1"
-F 0 "#PWR0118" H 4150 2400 50  0001 C CNN
+AR Path="/619C0687/60A72A00" Ref="#PWR0114"  Part="1"
+F 0 "#PWR0114" H 4150 2400 50  0001 C CNN
 F 1 "GND" H 4150 2500 50  0000 C CNN
 F 2 "" H 4150 2650 50  0001 C CNN
@@
 	4150 2600 4150 2650
 $Comp
-L power:+3.3V #PWR0119
+L power:+3.3V #PWR0113
 U 1 1 60A72BB3
 P 4150 1850
-F 0 "#PWR0119" H 4150 1700 50  0001 C CNN
+F 0 "#PWR0113" H 4150 1700 50  0001 C CNN
 F 1 "+3.3V" H 4165 2023 50  0000 C CNN
 F 2 "" H 4150 1850 50  0001 C CNN
@@
 $EndComp
 $Comp
-L Memory_EEPROM:25LCxxx U10
+L Memory_EEPROM:25LCxxx U11
 U 1 1 60A473E7
 P 2700 2300
-F 0 "U10" H 2700 2781 50  0000 C CNN
+F 0 "U11" H 2700 2781 50  0000 C CNN
 F 1 "25LCxxx" H 2700 2690 50  0000 C CNN
 F 2 "Package_SO:SOIC-8_5.275x5.275mm_P1.27mm" H 2700 2300 50  0001 C CNN
