File: Hardware/dsp-amplifier-x4.sch (KiCad schematic (older format))
At the start: 65 parts, among them J1 USBi, J2 EXT, J3 Raspberry_Pi_2_3, J4 Screw_Terminal_01x02, J5 Screw_Terminal_01x02, J6 Screw_Terminal_01x02, J7 Screw_Terminal_01x02, P1 Conn_WallPlug, Q1 STD2805, U1 ADAU1452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

Commit message: smallify
Connections:
- net +5VD is gone; now on net +5VA: J3.2 (5V), J3.4 (5V)
Changed lines of the file:
@@
 F2 "VOUT_3V3" O R 11150 1050 60
 F3 "VOUT_5V0" O R 11150 1150 60
-F4 "VOUT_5V0_SEC" O R 11150 1250 60
-F5 "VOUT_24V0" O R 11150 950 60
-F6 "AC_L" I L 9950 1000 60
-F7 "AC_N" I L 9950 1100 60
+F4 "VOUT_24V0" O R 11150 950 60
+F5 "AC_L" I L 9950 1000 60
+F6 "AC_N" I L 9950 1100 60
 $EndSheet
 $Sheet
@@
 Wire Wire Line
 	11150 1150 11900 1150
-Wire Wire Line
-	11150 1250 12200 1250
 $Comp
 L power:+24V #PWR028
@@
 	11900 900  11900 1150
 Wire Wire Line
-	12200 900  12200 1250
+	12200 900  12200 1150
 $Comp
 L power:+24V #PWR032
@@
 Wire Wire Line
 	13500 1350 14000 1350
+Wire Wire Line
+	11900 1150 12200 1150
+Connection ~ 11900 1150
 $EndSCHEMATC

Commit message: slight adjustments
Connections:
- net AUX_BCLK: now reaches U1.68 (BCLK_IN3)
- net AUX_MDI: now reaches U1.70 (SDATA_IN3)
- net PI_MUTE: no longer names the net of J3.13 (GPIO27)
- net PI_MUTE: no longer U1.69 (LRCLK_IN3/MP13)
- new net AUX_LRCLK: U1.69 (LRCLK_IN3/MP13)
- no-connect marks 35 -> 34
Other:
- moved on the sheet: J1, J2
Changed lines of the file:
@@
 Text Label 11250 8150 2    60   ~ 0
 PI_SCLK0
-Text Label 8350 8350 0    60   ~ 0
-PI_MUTE
 Text Label 8350 7850 0    60   ~ 0
 DSP_SELFBOOT
@@
 Wire Wire Line
 	8350 7850 9050 7850
-Wire Wire Line
-	8350 8350 9050 8350
 Text Label 5400 4050 2    60   ~ 0
 AMP2_LRCLK
@@
 L Connector_Generic:Conn_02x05_Odd_Even J1
 U 1 1 6119A08E
-P 6300 4850
-F 0 "J1" H 6350 5267 50  0000 C CNN
-F 1 "USBi" H 6350 5176 50  0000 C CNN
-F 2 "Connector_IDC:IDC-Header_2x05_P2.54mm_Vertical" H 6300 4850 50  0001 C CNN
-F 3 "~" H 6300 4850 50  0001 C CNN
-	1    6300 4850
-	1    0    0    -1
-$EndComp
-NoConn ~ 6600 4650
+P 7250 4200
+F 0 "J1" H 7300 4617 50  0000 C CNN
+F 1 "USBi" H 7300 4526 50  0000 C CNN
+F 2 "Connector_IDC:IDC-Header_2x05_P2.54mm_Vertical" H 7250 4200 50  0001 C CNN
+F 3 "~" H 7250 4200 50  0001 C CNN
+	1    7250 4200
+	1    0    0    -1
+$EndComp
+NoConn ~ 7550 4000
 $Comp
 L power:GND #PWR023
 U 1 1 611E8646
-P 6650 5100
-F 0 "#PWR023" H 6650 4850 50  0001 C CNN
-F 1 "GND" H 6650 4950 50  0000 C CNN
-F 2 "" H 6650 5100 50  0001 C CNN
-F 3 "" H 6650 5100 50  0001 C CNN
-	1    6650 5100
-	1    0    0    -1
-$EndComp
-Wire Wire Line
-	6600 5050 6650 5050
-Wire Wire Line
-	6650 5050 6650 5100
-Text Label 7250 4850 2    60   ~ 0
+P 7600 4450
+F 0 "#PWR023" H 7600 4200 50  0001 C CNN
+F 1 "GND" H 7600 4300 50  0000 C CNN
+F 2 "" H 7600 4450 50  0001 C CNN
+F 3 "" H 7600 4450 50  0001 C CNN
+	1    7600 4450
+	1    0    0    -1
+$EndComp
+Wire Wire Line
+	7550 4400 7600 4400
+Wire Wire Line
+	7600 4400 7600 4450
+Text Label 8200 4200 2    60   ~ 0
 DSP_NRESET
-NoConn ~ 6600 4750
-Wire Wire Line
-	6600 4850 7250 4850
+NoConn ~ 7550 4100
+Wire Wire Line
+	7550 4200 8200 4200
 $Comp
 L Device:Ferrite_Bead FB?
@@
 L Connector_Generic:Conn_02x08_Odd_Even J2
 U 1 1 606ED66E
-P 8550 3350
-F 0 "J2" H 8600 3867 50  0000 C CNN
-F 1 "EXT" H 8600 3776 50  0000 C CNN
-F 2 "Connector_IDC:IDC-Header_2x08_P2.54mm_Vertical" H 8550 3350 50  0001 C CNN
-F 3 "~" H 8550 3350 50  0001 C CNN
-	1    8550 3350
-	1    0    0    -1
-$EndComp
-Wire Wire Line
-	8850 3750 8900 3750
-Wire Wire Line
-	8850 3050 8900 3050
-Wire Wire Line
-	8900 3050 8900 3150
-Wire Wire Line
-	8850 3650 8900 3650
-Connection ~ 8900 3650
-Wire Wire Line
-	8900 3650 8900 3750
-Wire Wire Line
-	8850 3550 8900 3550
-Connection ~ 8900 3550
-Wire Wire Line
-	8900 3550 8900 3650
-Wire Wire Line
-	8900 3450 8850 3450
-Connection ~ 8900 3450
-Wire Wire Line
-	8900 3450 8900 3550
-Wire Wire Line
-	8850 3350 8900 3350
-Connection ~ 8900 3350
-Wire Wire Line
-	8900 3350 8900 3450
-Wire Wire Line
-	8850 3250 8900 3250
-Connection ~ 8900 3250
-Wire Wire Line
-	8900 3250 8900 3350
-Wire Wire Line
-	8850 3150 8900 3150
-Connection ~ 8900 3150
-Wire Wire Line
-	8900 3150 8900 3250
-Text Label 7750 3450 0    60   ~ 0
+P 7250 3050
+F 0 "J2" H 7300 3567 50  0000 C CNN
+F 1 "EXT" H 7300 3476 50  0000 C CNN
+F 2 "Connector_IDC:IDC-Header_2x08_P2.54mm_Vertical" H 7250 3050 50  0001 C CNN
+F 3 "~" H 7250 3050 50  0001 C CNN
+	1    7250 3050
+	1    0    0    -1
+$EndComp
+Wire Wire Line
+	7550 3450 7600 3450
+Wire Wire Line
+	7550 2750 7600 2750
+Wire Wire Line
+	7600 2750 7600 2850
+Wire Wire Line
+	7550 3350 7600 3350
+Connection ~ 7600 3350
+Wire Wire Line
+	7600 3350 7600 3450
+Wire Wire Line
+	7550 3250 7600 3250
+Connection ~ 7600 3250
+Wire Wire Line
+	7600 3250 7600 3350
+Wire Wire Line
+	7600 3150 7550 3150
+Connection ~ 7600 3150
+Wire Wire Line
+	7600 3150 7600 3250
+Wire Wire Line
+	7550 3050 7600 3050
+Connection ~ 7600 3050
+Wire Wire Line
+	7600 3050 7600 3150
+Wire Wire Line
+	7550 2950 7600 2950
+Connection ~ 7600 2950
+Wire Wire Line
+	7600 2950 7600 3050
+Wire Wire Line
+	7550 2850 7600 2850
+Connection ~ 7600 2850
+Wire Wire Line
+	7600 2850 7600 2950
+Text Label 6450 3150 0    60   ~ 0
 EXT_LRCLK
-Text Label 7750 3350 0    60   ~ 0
+Text Label 6450 3050 0    60   ~ 0
 EXT_BCLK
-Text Label 7750 3150 0    60   ~ 0
+Text Label 6450 2850 0    60   ~ 0
 EXT_MDI
 Wire Wire Line
-	8350 3150 7750 3150
-Wire Wire Line
-	8350 3450 7750 3450
-Wire Wire Line
-	7750 3350 8350 3350
-Text Label 7750 3250 0    60   ~ 0
+	7050 2850 6450 2850
+Wire Wire Line
+	7050 3150 6450 3150
+Wire Wire Line
+	6450 3050 7050 3050
+Text Label 6450 2950 0    60   ~ 0
 EXT_MDO
 Wire Wire Line
-	8350 3250 7750 3250
-Text Label 7750 3750 0    60   ~ 0
+	7050 2950 6450 2950
+Text Label 6450 3450 0    60   ~ 0
 EXT_MCLK
 Wire Wire Line
-	8350 3750 7750 3750
-Wire Wire Line
-	8300 3000 8300 3050
-Wire Wire Line
-	8300 3050 8350 3050
+	7050 3450 6450 3450
+Wire Wire Line
+	7000 2700 7000 2750
+Wire Wire Line
+	7000 2750 7050 2750
 $Comp
 L power:GND #PWR025
 U 1 1 606EF4D1
-P 8900 3800
-F 0 "#PWR025" H 8900 3550 50  0001 C CNN
-F 1 "GND" H 8900 3650 50  0000 C CNN
-F 2 "" H 8900 3800 50  0001 C CNN
-F 3 "" H 8900 3800 50  0001 C CNN
-	1    8900 3800
-	1    0    0    -1
-$EndComp
-Wire Wire Line
-	8900 3750 8900 3800
-Connection ~ 8900 3750
+P 7600 3500
+F 0 "#PWR025" H 7600 3250 50  0001 C CNN
+F 1 "GND" H 7600 3350 50  0000 C CNN
+F 2 "" H 7600 3500 50  0001 C CNN
+F 3 "" H 7600 3500 50  0001 C CNN
+	1    7600 3500
+	1    0    0    -1
+$EndComp
+Wire Wire Line
+	7600 3450 7600 3500
+Connection ~ 7600 3450
 $Comp
 L Connector:Conn_WallPlug P1
@@
 Wire Wire Line
 	1400 4050 1400 4100
-NoConn ~ 6100 4650
-NoConn ~ 6100 4750
+NoConn ~ 7050 4000
+NoConn ~ 7050 4100
 Wire Wire Line
 	5300 4850 4400 4850
 Wire Wire Line
 	4400 4950 5300 4950
-Text Label 5500 5050 0    60   ~ 0
+Text Label 6450 4400 0    60   ~ 0
 PI_NCE0
-Text Label 7250 4950 2    60   ~ 0
+Text Label 8200 4300 2    60   ~ 0
 PI_MOSI0
-Text Label 5500 4850 0    60   ~ 0
+Text Label 6450 4200 0    60   ~ 0
 PI_MISO0
-Text Label 5500 4950 0    60   ~ 0
+Text Label 6450 4300 0    60   ~ 0
 PI_SCLK0
 Wire Wire Line
-	7250 4950 6600 4950
-Wire Wire Line
-	6100 4950 5500 4950
-Wire Wire Line
-	5500 5050 6100 5050
-Wire Wire Line
-	6100 4850 5500 4850
+	8200 4300 7550 4300
+Wire Wire Line
+	7050 4300 6450 4300
+Wire Wire Line
+	6450 4400 7050 4400
+Wire Wire Line
+	7050 4200 6450 4200
 $Comp
 L Device:R R14
@@
 Wire Wire Line
 	9000 7250 9050 7250
-Text Label 2000 4150 0    60   ~ 0
-PI_MUTE
-Wire Wire Line
-	2000 4150 2600 4150
 Text Label 4050 7050 2    60   ~ 0
 IOVDD
@@
 $EndComp
 NoConn ~ 4400 3350
-NoConn ~ 2600 4050
-NoConn ~ 2600 4250
 NoConn ~ 9050 7050
 NoConn ~ 9050 8050
@@
 L power:+5VA #PWR024
 U 1 1 609E250E
-P 8300 3000
-F 0 "#PWR024" H 8300 2850 50  0001 C CNN
-F 1 "+5VA" H 8315 3173 50  0000 C CNN
-F 2 "" H 8300 3000 50  0001 C CNN
-F 3 "" H 8300 3000 50  0001 C CNN
-	1    8300 3000
+P 7000 2700
+F 0 "#PWR024" H 7000 2550 50  0001 C CNN
+F 1 "+5VA" H 7015 2873 50  0000 C CNN
+F 2 "" H 7000 2700 50  0001 C CNN
+F 3 "" H 7000 2700 50  0001 C CNN
+	1    7000 2700
 	1    0    0    -1
 $EndComp
@@
 Text Label 11250 7150 2    60   ~ 0
 PI_SCL
-Text Label 7750 3550 0    60   ~ 0
+Text Label 6450 3250 0    60   ~ 0
 PI_SDA
-Text Label 7750 3650 0    60   ~ 0
+Text Label 6450 3350 0    60   ~ 0
 PI_SCL
 Wire Wire Line
-	7750 3550 8350 3550
-Wire Wire Line
-	8350 3650 7750 3650
+	6450 3250 7050 3250
+Wire Wire Line
+	7050 3350 6450 3350
 $Comp
 L Device:R R21
@@
 	11900 1150 12200 1150
 Connection ~ 11900 1150
+Text Label 2000 4150 0    60   ~ 0
+AUX_LRCLK
+Text Label 2000 4050 0    60   ~ 0
+AUX_BCLK
+Text Label 2000 4250 0    60   ~ 0
+AUX_MDI
+Wire Wire Line
+	2600 4250 2000 4250
+Wire Wire Line
+	2600 4150 2000 4150
+Wire Wire Line
+	2000 4050 2600 4050
+NoConn ~ 9050 8350
 $EndSCHEMATC

Commit message: mostly ready
Parts:
- removed P1: Conn_WallPlug, terminal_connectors:wuerth_691216410002, symbol Connector:Conn_WallPlug
- added J11: Screw_Terminal_01x02, terminal_connectors:wuerth_691216410002, symbol Connector:Screw_Terminal_01x02
Connections:
- new net Power/24V0_IN: J11.1 (Pin_1)
- new net Power/GND_IN: J11.2 (Pin_2)
Changed lines of the file:
@@
 $EndDescr
-$Sheet
-S 9950 900  1200 400
-U 5AFACF29
-F0 "Power" 60
-F1 "power.sch" 60
-F2 "VOUT_3V3" O R 11150 1050 60
-F3 "VOUT_5V0" O R 11150 1150 60
-F4 "VOUT_24V0" O R 11150 950 60
-F5 "AC_L" I L 9950 1000 60
-F6 "AC_N" I L 9950 1100 60
-$EndSheet
 $Sheet
 S 9950 1600 550  1000
@@
 PI_SDATA_I
 Wire Wire Line
-	9350 1000 9350 950
-Wire Wire Line
-	9350 950  9250 950
-Wire Wire Line
-	9350 1100 9350 1150
-Wire Wire Line
-	9350 1150 9250 1150
-Wire Wire Line
 	11550 2250 10850 2250
 Wire Wire Line
@@
 	7600 3450 7600 3500
 Connection ~ 7600 3450
-$Comp
-L Connector:Conn_WallPlug P1
-U 1 1 60704E3B
-P 9050 1050
-F 0 "P1" H 9067 1375 50  0000 C CNN
-F 1 "Conn_WallPlug" H 9067 1284 50  0000 C CNN
-F 2 "terminal_connectors:wuerth_691216410002" H 9450 1050 50  0001 C CNN
-F 3 "~" H 9450 1050 50  0001 C CNN
-	1    9050 1050
-	1    0    0    -1
-$EndComp
 Text Label 2000 3750 0    60   ~ 0
 USB_LRCLK
@@
 Wire Wire Line
 	9650 6050 9650 6300
-Wire Wire Line
-	9950 1100 9350 1100
 NoConn ~ 10500 1750
 NoConn ~ 10500 1950
@@
 Text Notes 14350 1600 0    60   ~ 0
 GAIN[1:0]\n00: 12.9 V full-scale\n01: 15.1 V full-scale\n10: 25.15 V full-scale\n11: Software-controlled
-Wire Wire Line
-	9350 1000 9950 1000
 Text Label 5300 5150 2    60   ~ 0
 PI_NCE0
@@
 	2000 4050 2600 4050
 NoConn ~ 9050 8350
+$Comp
+L Connector:Screw_Terminal_01x02 J11
+U 1 1 60D6FB76
+P 9750 1000
+F 0 "J11" H 9830 992 50  0000 L CNN
+F 1 "Screw_Terminal_01x02" H 9830 901 50  0000 L CNN
+F 2 "terminal_connectors:wuerth_691216410002" H 9750 1000 50  0001 C CNN
+F 3 "~" H 9750 1000 50  0001 C CNN
+	1    9750 1000
+	-1   0    0    -1
+$EndComp
+$Sheet
+S 9950 900  1200 400
+U 5AFACF29
+F0 "Power" 60
+F1 "power.sch" 60
+F2 "VOUT_3V3" O R 11150 1050 60
+F3 "VOUT_5V0" O R 11150 1150 60
+F4 "VOUT_24V0" O R 11150 950 60
+F5 "24V0_IN" I L 9950 1000 60
+F6 "GND_IN" I L 9950 1100 60
+$EndSheet
 $EndSCHEMATC
