File: Hardware/power.sch (KiCad schematic (older format))
At the start: 25 parts, among them U5 TPS54308, U6 TPS54308, U7 AMS1117-3.3

Commit message: started routing
Parts:
- removed C12: 22u, Capacitor_SMD:C_0603_1608Metric_Pad1.08x0.95mm_HandSolder, symbol Device:C
- removed C15, C17, C18: 22u, Capacitor_SMD:C_0805_2012Metric_Pad1.18x1.45mm_HandSolder, symbol Device:C
- added C34, C35, C36, C37, C38, C39, C40, C41: 10u, Capacitor_SMD:C_1206_3216Metric_Pad1.33x1.80mm_HandSolder, symbol Device:C
- C30: renamed from C8; footprint Capacitor_SMD:C_0805_2012Metric_Pad1.18x1.45mm_HandSolder -> Capacitor_SMD:C_1206_3216Metric_Pad1.33x1.80mm_HandSolder
- C31: renamed from C13; footprint Capacitor_SMD:C_0805_2012Metric_Pad1.18x1.45mm_HandSolder -> Capacitor_SMD:C_1206_3216Metric_Pad1.33x1.80mm_HandSolder
- C42: renamed from C5; value 4.7u -> 10u; footprint Capacitor_SMD:C_0603_1608Metric_Pad1.08x0.95mm_HandSolder -> Capacitor_SMD:C_1206_3216Metric_Pad1.33x1.80mm_HandSolder
- L1: renamed from L6; footprint Capacitor_SMD:C_0805_2012Metric_Pad1.18x1.45mm_HandSolder -> Inductor_SMD:L_Abracon_ASPI-0630LR
- L2: renamed from L5; footprint Capacitor_SMD:C_0805_2012Metric_Pad1.18x1.45mm_HandSolder -> Inductor_SMD:L_Abracon_ASPI-0630LR
- renumbered C6 to C28, C11 to C29, C10 to C32, C16 to C33, R4 to R31, R5 to R32, R2 to R33, R3 to R34, R10 to R35, R12 to R36, R6 to R37, R7 to R38, U6 to U2, U5 to U3, U7 to U4
Connections:
- wire segments 90 -> 102
Other:
- moved on the sheet: C42, R35, R36, R37, R38, U4

Commit message: hardware bugfixes
Parts:
- renumbered R31 to R25, R32 to R26, R33 to R27, R34 to R28, R35 to R29, R36 to R30, R37 to R31, R38 to R32, U2 to U3, U3 to U4, U4 to U5
Changed lines of the file:
@@
 VOUT_3V3
 $Comp
-L Regulator_Switching:TPS54308 U2
+L Regulator_Switching:TPS54308 U3
 U 1 1 60759E86
 P 4200 2850
-F 0 "U2" H 4200 3217 50  0000 C CNN
+F 0 "U3" H 4200 3217 50  0000 C CNN
 F 1 "TPS54308" H 4200 3126 50  0000 C CNN
 F 2 "Package_TO_SOT_SMD:SOT-23-6" H 4250 2500 50  0001 L CNN
@@
 	3550 2750 3550 2050
 $Comp
-L Device:R R31
+L Device:R R25
 U 1 1 60759E8F
 P 3200 2700
-F 0 "R31" H 3270 2746 50  0000 L CNN
+F 0 "R25" H 3270 2746 50  0000 L CNN
 F 1 "511k" H 3270 2655 50  0000 L CNN
 F 2 "Resistor_SMD:R_0603_1608Metric_Pad0.98x0.95mm_HandSolder" V 3130 2700 50  0001 C CNN
@@
 	3200 2050 3550 2050
 $Comp
-L power:GND #PWR049
+L power:GND #PWR044
 U 1 1 60759EA1
 P 3200 3400
-F 0 "#PWR049" H 3200 3150 50  0001 C CNN
+F 0 "#PWR044" H 3200 3150 50  0001 C CNN
 F 1 "GND" H 3205 3227 50  0000 C CNN
 F 2 "" H 3200 3400 50  0001 C CNN
@@
 $EndComp
 $Comp
-L power:GND #PWR051
+L power:GND #PWR046
 U 1 1 60759EA7
 P 4200 3400
-F 0 "#PWR051" H 4200 3150 50  0001 C CNN
+F 0 "#PWR046" H 4200 3150 50  0001 C CNN
 F 1 "GND" H 4205 3227 50  0000 C CNN
 F 2 "" H 4200 3400 50  0001 C CNN
@@
 	2200 2100 2200 2050
 $Comp
-L power:GND #PWR047
+L power:GND #PWR042
 U 1 1 60759EC1
 P 2700 2450
-F 0 "#PWR047" H 2700 2200 50  0001 C CNN
+F 0 "#PWR042" H 2700 2200 50  0001 C CNN
 F 1 "GND" H 2705 2277 50  0000 C CNN
 F 2 "" H 2700 2450 50  0001 C CNN
@@
 $EndComp
 $Comp
-L power:GND #PWR045
+L power:GND #PWR040
 U 1 1 60759EC7
 P 2200 2450
-F 0 "#PWR045" H 2200 2200 50  0001 C CNN
+F 0 "#PWR040" H 2200 2200 50  0001 C CNN
 F 1 "GND" H 2205 2277 50  0000 C CNN
 F 2 "" H 2200 2450 50  0001 C CNN
@@
 Connection ~ 5550 2850
 $Comp
-L Device:R R36
+L Device:R R30
 U 1 1 60759EF6
 P 7500 3450
-F 0 "R36" H 7570 3496 50  0000 L CNN
+F 0 "R30" H 7570 3496 50  0000 L CNN
 F 1 "13.5k" H 7570 3405 50  0000 L CNN
 F 2 "Resistor_SMD:R_0603_1608Metric_Pad0.98x0.95mm_HandSolder" V 7430 3450 50  0001 C CNN
@@
 $EndComp
 $Comp
-L Device:R R35
+L Device:R R29
 U 1 1 60759EFC
 P 7500 3050
-F 0 "R35" H 7570 3096 50  0000 L CNN
+F 0 "R29" H 7570 3096 50  0000 L CNN
 F 1 "100k" H 7570 3005 50  0000 L CNN
 F 2 "Resistor_SMD:R_0603_1608Metric_Pad0.98x0.95mm_HandSolder" V 7430 3050 50  0001 C CNN
@@
 	7500 3200 7500 3250
 $Comp
-L power:GND #PWR053
+L power:GND #PWR048
 U 1 1 60759F06
 P 5550 3300
-F 0 "#PWR053" H 5550 3050 50  0001 C CNN
+F 0 "#PWR048" H 5550 3050 50  0001 C CNN
 F 1 "GND" H 5555 3127 50  0000 C CNN
 F 2 "" H 5550 3300 50  0001 C CNN
@@
 $EndComp
 $Comp
-L power:GND #PWR055
+L power:GND #PWR050
 U 1 1 60759F0C
 P 6050 3300
-F 0 "#PWR055" H 6050 3050 50  0001 C CNN
+F 0 "#PWR050" H 6050 3050 50  0001 C CNN
 F 1 "GND" H 6055 3127 50  0000 C CNN
 F 2 "" H 6050 3300 50  0001 C CNN
@@
 	7500 3600 7500 3650
 $Comp
-L power:GND #PWR061
+L power:GND #PWR056
 U 1 1 60759F15
 P 7500 3650
-F 0 "#PWR061" H 7500 3400 50  0001 C CNN
+F 0 "#PWR056" H 7500 3400 50  0001 C CNN
 F 1 "GND" H 7505 3477 50  0000 C CNN
 F 2 "" H 7500 3650 50  0001 C CNN
@@
 VOUT_5V0
 $Comp
-L Device:R R32
+L Device:R R26
 U 1 1 6075ED5F
 P 3200 3200
-F 0 "R32" H 3270 3246 50  0000 L CNN
+F 0 "R26" H 3270 3246 50  0000 L CNN
 F 1 "100k" H 3270 3155 50  0000 L CNN
 F 2 "Resistor_SMD:R_0603_1608Metric_Pad0.98x0.95mm_HandSolder" V 3130 3200 50  0001 C CNN
@@
 Connection ~ 2200 2050
 $Comp
-L power:GND #PWR063
+L power:GND #PWR058
 U 1 1 6065F737
 P 8450 5150
-F 0 "#PWR063" H 8450 4900 50  0001 C CNN
+F 0 "#PWR058" H 8450 4900 50  0001 C CNN
 F 1 "GND" H 8455 4977 50  0000 C CNN
 F 2 "" H 8450 5150 50  0001 C CNN
@@
 	8850 4700 8750 4700
 $Comp
-L power:GND #PWR064
+L power:GND #PWR059
 U 1 1 60669E4D
 P 8850 5150
-F 0 "#PWR064" H 8850 4900 50  0001 C CNN
+F 0 "#PWR059" H 8850 4900 50  0001 C CNN
 F 1 "GND" H 8855 4977 50  0000 C CNN
 F 2 "" H 8850 5150 50  0001 C CNN
@@
 	8450 5000 8450 5150
 $Comp
-L Regulator_Switching:TPS54308 U3
+L Regulator_Switching:TPS54308 U4
 U 1 1 606B57FE
 P 4200 4700
-F 0 "U3" H 4200 5067 50  0000 C CNN
+F 0 "U4" H 4200 5067 50  0000 C CNN
 F 1 "TPS54308" H 4200 4976 50  0000 C CNN
 F 2 "Package_TO_SOT_SMD:SOT-23-6" H 4250 4350 50  0001 L CNN
@@
 	3550 4600 3550 3900
 $Comp
-L Device:R R33
+L Device:R R27
 U 1 1 606B5806
 P 3200 4550
-F 0 "R33" H 3270 4596 50  0000 L CNN
+F 0 "R27" H 3270 4596 50  0000 L CNN
 F 1 "511k" H 3270 4505 50  0000 L CNN
 F 2 "Resistor_SMD:R_0603_1608Metric_Pad0.98x0.95mm_HandSolder" V 3130 4550 50  0001 C CNN
@@
 	3200 3900 3550 3900
 $Comp
-L power:GND #PWR050
+L power:GND #PWR045
 U 1 1 606B5812
 P 3200 5250
-F 0 "#PWR050" H 3200 5000 50  0001 C CNN
+F 0 "#PWR045" H 3200 5000 50  0001 C CNN
 F 1 "GND" H 3205 5077 50  0000 C CNN
 F 2 "" H 3200 5250 50  0001 C CNN
@@
 $EndComp
 $Comp
-L power:GND #PWR052
+L power:GND #PWR047
 U 1 1 606B5818
 P 4200 5250
-F 0 "#PWR052" H 4200 5000 50  0001 C CNN
+F 0 "#PWR047" H 4200 5000 50  0001 C CNN
 F 1 "GND" H 4205 5077 50  0000 C CNN
 F 2 "" H 4200 5250 50  0001 C CNN
@@
 	2200 3950 2200 3900
 $Comp
-L power:GND #PWR048
+L power:GND #PWR043
 U 1 1 606B5831
 P 2700 4300
-F 0 "#PWR048" H 2700 4050 50  0001 C CNN
+F 0 "#PWR043" H 2700 4050 50  0001 C CNN
 F 1 "GND" H 2705 4127 50  0000 C CNN
 F 2 "" H 2700 4300 50  0001 C CNN
@@
 $EndComp
 $Comp
-L power:GND #PWR046
+L power:GND #PWR041
 U 1 1 606B5837
 P 2200 4300
-F 0 "#PWR046" H 2200 4050 50  0001 C CNN
+F 0 "#PWR041" H 2200 4050 50  0001 C CNN
 F 1 "GND" H 2205 4127 50  0000 C CNN
 F 2 "" H 2200 4300 50  0001 C CNN
@@
 Connection ~ 5550 4700
 $Comp
-L Device:R R38
+L Device:R R32
 U 1 1 606B5865
 P 7500 5300
-F 0 "R38" H 7570 5346 50  0000 L CNN
+F 0 "R32" H 7570 5346 50  0000 L CNN
 F 1 "13.5k" H 7570 5255 50  0000 L CNN
 F 2 "Resistor_SMD:R_0603_1608Metric_Pad0.98x0.95mm_HandSolder" V 7430 5300 50  0001 C CNN
@@
 $EndComp
 $Comp
-L Device:R R37
+L Device:R R31
 U 1 1 606B586B
 P 7500 4900
-F 0 "R37" H 7570 4946 50  0000 L CNN
+F 0 "R31" H 7570 4946 50  0000 L CNN
 F 1 "100k" H 7570 4855 50  0000 L CNN
 F 2 "Resistor_SMD:R_0603_1608Metric_Pad0.98x0.95mm_HandSolder" V 7430 4900 50  0001 C CNN
@@
 	7500 5050 7500 5100
 $Comp
-L power:GND #PWR054
+L power:GND #PWR049
 U 1 1 606B5875
 P 5550 5150
-F 0 "#PWR054" H 5550 4900 50  0001 C CNN
+F 0 "#PWR049" H 5550 4900 50  0001 C CNN
 F 1 "GND" H 5555 4977 50  0000 C CNN
 F 2 "" H 5550 5150 50  0001 C CNN
@@
 $EndComp
 $Comp
-L power:GND #PWR056
+L power:GND #PWR051
 U 1 1 606B587B
 P 6050 5150
-F 0 "#PWR056" H 6050 4900 50  0001 C CNN
+F 0 "#PWR051" H 6050 4900 50  0001 C CNN
 F 1 "GND" H 6055 4977 50  0000 C CNN
 F 2 "" H 6050 5150 50  0001 C CNN
@@
 	7500 5450 7500 5500
 $Comp
-L power:GND #PWR062
+L power:GND #PWR057
 U 1 1 606B5884
 P 7500 5500
-F 0 "#PWR062" H 7500 5250 50  0001 C CNN
+F 0 "#PWR057" H 7500 5250 50  0001 C CNN
 F 1 "GND" H 7505 5327 50  0000 C CNN
 F 2 "" H 7500 5500 50  0001 C CNN
@@
 	7500 5100 7500 5150
 $Comp
-L Device:R R34
+L Device:R R28
 U 1 1 606B5891
 P 3200 5050
-F 0 "R34" H 3270 5096 50  0000 L CNN
+F 0 "R28" H 3270 5096 50  0000 L CNN
 F 1 "100k" H 3270 5005 50  0000 L CNN
 F 2 "Resistor_SMD:R_0603_1608Metric_Pad0.98x0.95mm_HandSolder" V 3130 5050 50  0001 C CNN
@@
 	7500 5100 8150 5100
 $Comp
-L Regulator_Linear:AMS1117-3.3 U4
+L Regulator_Linear:AMS1117-3.3 U5
 U 1 1 606CA892
 P 8450 4700
-F 0 "U4" H 8450 4942 50  0000 C CNN
+F 0 "U5" H 8450 4942 50  0000 C CNN
 F 1 "AMS1117-3.3" H 8450 4851 50  0000 C CNN
 F 2 "Package_TO_SOT_SMD:SOT-223-3_TabPin2" H 8450 4900 50  0001 C CNN
@@
 	1950 2050 2200 2050
 $Comp
-L power:GND #PWR044
+L power:GND #PWR039
 U 1 1 6066C031
 P 1750 2300
-F 0 "#PWR044" H 1750 2050 50  0001 C CNN
+F 0 "#PWR039" H 1750 2050 50  0001 C CNN
 F 1 "GND" H 1755 2127 50  0000 C CNN
 F 2 "" H 1750 2300 50  0001 C CNN
@@
 	7000 5100 7000 5150
 $Comp
-L power:GND #PWR060
+L power:GND #PWR055
 U 1 1 606D9266
 P 7000 5150
-F 0 "#PWR060" H 7000 4900 50  0001 C CNN
+F 0 "#PWR055" H 7000 4900 50  0001 C CNN
 F 1 "GND" H 7005 4977 50  0000 C CNN
 F 2 "" H 7000 5150 50  0001 C CNN
@@
 $EndComp
 $Comp
-L power:GND #PWR058
+L power:GND #PWR053
 U 1 1 606D9260
 P 6500 5150
-F 0 "#PWR058" H 6500 4900 50  0001 C CNN
+F 0 "#PWR053" H 6500 4900 50  0001 C CNN
 F 1 "GND" H 6505 4977 50  0000 C CNN
 F 2 "" H 6500 5150 50  0001 C CNN
@@
 Connection ~ 6500 2850
 $Comp
-L power:GND #PWR057
+L power:GND #PWR052
 U 1 1 606E4252
 P 6500 3300
-F 0 "#PWR057" H 6500 3050 50  0001 C CNN
+F 0 "#PWR052" H 6500 3050 50  0001 C CNN
 F 1 "GND" H 6505 3127 50  0000 C CNN
 F 2 "" H 6500 3300 50  0001 C CNN
@@
 $EndComp
 $Comp
-L power:GND #PWR059
+L power:GND #PWR054
 U 1 1 606E4258
 P 7000 3300
-F 0 "#PWR059" H 7000 3050 50  0001 C CNN
+F 0 "#PWR054" H 7000 3050 50  0001 C CNN
 F 1 "GND" H 7005 3127 50  0000 C CNN
 F 2 "" H 7000 3300 50  0001 C CNN

Commit message: bom
Other:
- note added: "Alternative: TPS54302, TPS54202"
Changed lines of the file:
@@
 	7000 4700 7000 4800
 Connection ~ 7000 4700
+Text Notes 3900 2150 0    60   ~ 0
+Alternative: TPS54302, TPS54202
 $EndSCHEMATC

Commit message: smallify
Parts:
- removed C28, C32: 100n, Capacitor_SMD:C_0603_1608Metric_Pad1.08x0.95mm_HandSolder, symbol Device:C
- removed C30, C34, C36, C38, C40: 10u, Capacitor_SMD:C_1206_3216Metric_Pad1.33x1.80mm_HandSolder, symbol Device:C
- removed L1: 10u, Inductor_SMD:L_Abracon_ASPI-0630LR, symbol Device:L
- removed R25: 511k, Resistor_SMD:R_0603_1608Metric_Pad0.98x0.95mm_HandSolder, symbol Device:R
- removed R26, R29: 100k, Resistor_SMD:R_0603_1608Metric_Pad0.98x0.95mm_HandSolder, symbol Device:R
- removed R30: 13.5k, Resistor_SMD:R_0603_1608Metric_Pad0.98x0.95mm_HandSolder, symbol Device:R
- removed U3: TPS54308, Package_TO_SOT_SMD:SOT-23-6, symbol Regulator_Switching:TPS54308
Connections:
- net labels removed: FB_5V0, VOUT_5V0_SEC
- wire segments 102 -> 59

Commit message: mostly ready
Parts:
- removed PS1: IRM-60-24, Converter_ACDC:Converter_ACDC_MeanWell_IRM-60-xx_THT, symbol Converter_ACDC:IRM-60-24
Connections:
- net labels added: 24V0_IN, GND_IN
- net labels removed: AC_L, AC_N
- wire segments 59 -> 56
Changed lines of the file:
@@
 $Descr A4 11693 8268
 encoding utf-8
-Sheet 2 8
+Sheet 8 8
 Title "Supply"
 Date "2021-04-01"
@@
 	1    0    0    -1
 $EndComp
-$Comp
-L Converter_ACDC:IRM-60-24 PS1
-U 1 1 606647DE
-P 1300 2150
-F 0 "PS1" H 1300 2517 50  0000 C CNN
-F 1 "IRM-60-24" H 1300 2426 50  0000 C CNN
-F 2 "Converter_ACDC:Converter_ACDC_MeanWell_IRM-60-xx_THT" H 1300 1750 50  0001 C CNN
-F 3 "http://www.meanwellusa.com/productPdf.aspx?i=687" H 1300 2150 50  0001 C CNN
-	1    1300 2150
-	1    0    0    -1
-$EndComp
-Wire Wire Line
-	1700 2050 1950 2050
 Wire Wire Line
 	1950 2050 1950 3900
-Connection ~ 1950 2050
 $Comp
 L power:GND #PWR035
@@
 $EndComp
 Wire Wire Line
-	1700 2250 1750 2250
-Wire Wire Line
 	1750 2250 1750 2300
-Text HLabel 2150 1850 2    60   Output ~ 0
+Text HLabel 2350 2050 2    60   Output ~ 0
 VOUT_24V0
-Wire Wire Line
-	2150 1850 1950 1850
-Wire Wire Line
-	1950 1850 1950 2050
-Text HLabel 850  2050 0    60   Input ~ 0
-AC_L
-Text HLabel 850  2250 0    60   Input ~ 0
-AC_N
-Wire Wire Line
-	900  2050 850  2050
-Wire Wire Line
-	900  2250 850  2250
+Text HLabel 1200 2050 0    60   Input ~ 0
+24V0_IN
+Text HLabel 1200 2250 0    60   Input ~ 0
+GND_IN
 $Comp
 L Device:C C35
@@
 Text Notes 3350 3750 0    60   ~ 0
 Alternative: TPS54302, TPS54202
+Wire Wire Line
+	1200 2050 1950 2050
+Wire Wire Line
+	1200 2250 1750 2250
+Wire Wire Line
+	1950 2050 2350 2050
+Connection ~ 1950 2050
 $EndSCHEMATC
