File: Hardware/dsp-amplifier-x4.kicad_sch (KiCad schematic)
At the start: 65 parts, among them J1 USBi, J11 Screw_Terminal_01x02, J2 EXT, J3 Raspberry_Pi_2_3, J4 Screw_Terminal_01x02, J5 Screw_Terminal_01x02, J6 Screw_Terminal_01x02, J7 Screw_Terminal_01x02, Q1 STD2805, U1 ADAU1452, U2 TSOP583xx

Commit message: Updated power supply
Connections:
- net Power/24V0_IN renamed Power-15V/15V0_IN
- net Power/GND_IN renamed Power-15V/GND_IN
Other:
- removed sheet Power
- added sheet Power-15V (power_15v.kicad_sch)

Commit message: Updated clock buffer
Connections:
- net Clock/CLK5 is gone; now on net Clock/CLK1: R19.1
- net Clock/CLK7 is gone; now on net Clock/CLK0: R20.1
- net Clock/CLK1: no longer R17.1
- net Clock/CLK2: now also R18.1
- net Clock/CLK3: now also R17.1; no longer R18.1
- no-connect marks 34 -> 30
Other:
- sheet Clock ports: added none; removed CLK4, CLK5, CLK6, CLK7
- note added: "GAIN[1:0] 00: 12.9 V full-scale 01: 15.1 V full-scale 10: 25.15 V full-scale (not recommended on TAS5760L) 11: Software-controlled"
- note removed: "GAIN[1:0] 00: 12.9 V full-scale 01: 15.1 V full-scale 10: 25.15 V full-scale 11: Software-controlled"

Commit message: feat: updated amplifier IC, finalized design
Parts:
- removed C1: 10u, Capacitor_SMD:C_1206_3216Metric_Pad1.33x1.80mm_HandSolder, symbol Device:C
- removed FB1: BLM18SP601SZ1D (600/100M), Inductor_SMD:L_0603_1608Metric_Pad1.05x0.95mm_HandSolder, symbol Device:Ferrite_Bead
- removed J1: USBi, Connector_IDC:IDC-Header_2x05_P2.54mm_Vertical, symbol Connector_Generic:Conn_02x05_Odd_Even
- removed J11, J4, J5, J6, J7: Screw_Terminal_01x02, terminal_connectors:wuerth_691216410002, symbol Connector:Screw_Terminal_01x02
- removed Q1: STD2805, Package_TO_SOT_SMD:TO-252-3_TabPin2, symbol Device:Q_PNP_BCE
- removed R10, R11, R12, R14, R15, R19, R20, R5, R6, R7, R8, R9: 33, Resistor_SMD:R_0603_1608Metric_Pad0.98x0.95mm_HandSolder, symbol Device:R
- removed R21, R22, R23, R24: 4.3k, Resistor_SMD:R_0603_1608Metric_Pad0.98x0.95mm_HandSolder, symbol Device:R
- removed RV2: PTV09A-1020F-B203, Potentiometer_THT:Potentiometer_Bourns_PTV09A-1_Single_Vertical, symbol Device:R_POT
- added J1: Screw_Terminal_01x02, terminal_connectors:wuerth_691216410002, symbol Connector:Screw_Terminal_01x02
- added Q1: SS8550, Package_TO_SOT_SMD:SOT-23, symbol Device:Q_PNP_BEC
- added RN1, RN2, RN3, RN5: R_Pack04, Resistor_SMD:R_Array_Convex_4x0603, symbol Device:R_Pack04
- C10, C11, C12, C13, C14, C15, C16, C17, C18, C19, C2, C20, C21, C23, C24, C3, C4, C5, C6, C7, C8, C9: footprint Capacitor_SMD:C_0603_1608Metric_Pad1.08x0.95mm_HandSolder -> Capacitor_SMD:C_0402_1005Metric
- C22, C25, C26, C27: footprint Capacitor_SMD:C_1206_3216Metric_Pad1.33x1.80mm_HandSolder -> Capacitor_SMD:C_1206_3216Metric
- R1, R13, R16, R17, R18, R2, R3, R4: footprint Resistor_SMD:R_0603_1608Metric_Pad0.98x0.95mm_HandSolder -> Resistor_SMD:R_0402_1005Metric
Connections:
- net +3V3 is gone; now on net +3.3VA: C11.1, C13.1, C15.1, C18.1, C21.1, C22.1, C24.1, C4.1, C8.1, R1.2, R2.2, R4.1, U1.18 (IOVDD), U1.2 (IOVDD), U1.38 (IOVDD), U1.56 (IOVDD)
- net AMP2_CLOCK is gone; now on net PI_SDATA_O: R18.2
- net +3.3VA: now also Q1.2 (E)
- net AMP1_BCLK: now also RN2.8 (R1.2)
- net AMP1_LRCLK: now also RN2.7 (R2.2)
- net AMP1_SDIN: now also RN3.5 (R4.2)
- net AMP2_BCLK: now also RN3.7 (R2.2)
- net AMP2_LRCLK: now also RN3.6 (R3.2)
- net AMP2_SDIN: now also RN3.8 (R1.2)
- net Clock/CLK0: now also RN1.8 (R1.2)
- net Clock/CLK1: now also RN1.7 (R2.2)
- net Clock/CLK2: now also RN1.6 (R3.2); no longer R18.1
- net Clock/CLK3: now also RN1.5 (R4.2); no longer R17.1
- net DSP_CLOCK: now also RN1.4 (R4.1); no longer R17.2
- net DVDD: now also Q1.3 (C)
- net EXT_MCLK: now also RN1.3 (R3.1)
- net EXT_MDO: now also RN2.6 (R3.2)
- net PI_BCLK: now also R16.2
- net PI_LRCLK: now also R17.2
- net PI_SDATA_I: now also RN2.5 (R4.2)
- net PI_SDATA_O: no longer R16.2
- net Power/15V0_IN: now also J1.2 (Pin_2)
- net Power/GND_IN: now also J1.1 (Pin_1)
- net USB_BCLK: now also RN5.7 (R2.2)
- net USB_LRCLK: now also RN5.6 (R3.2)
- net USB_SDATA: now also RN5.5 (R4.2)
- net VDRIVE: now also Q1.1 (B)
- net VPOT0: now also U1.11 (AUXADC3); no longer U1.8 (AUXADC0)
- net _PI_SDATA_I: now reaches U1.41 (SDATA_OUT0)
- net _PI_SDATA_I: now also RN2.4 (R4.1)
- net _EXT_MDO: now reaches U1.44 (SDATA_OUT1)
- net _EXT_MDO: now also RN2.3 (R3.1)
- net _AMP1_LRCLK: now reaches U1.47 (LRCLK_OUT2/MP8)
- net _AMP1_LRCLK: now also RN2.2 (R2.1)
- net _AMP1_BCLK: now reaches U1.48 (BCLK_OUT2)
- net _AMP1_BCLK: now also RN2.1 (R1.1)
- net _AMP1_SDIN: now reaches U1.49 (SDATA_OUT2)
- net _AMP1_SDIN: now also RN3.4 (R4.1)
- net _AMP2_LRCLK: now reaches U1.50 (LRCLK_OUT3/MP9)
- net _AMP2_LRCLK: now also RN3.3 (R3.1)
- net _AMP2_BCLK: now reaches U1.51 (BCLK_OUT3)
- net _AMP2_BCLK: now also RN3.2 (R2.1)
- net _AMP2_SDIN: now reaches U1.52 (SDATA_OUT3)
- net _AMP2_SDIN: now also RN3.1 (R1.1)
- net _PI_BCLK: now reaches J3.12 (GPIO18/PWM0)
- net _PI_BCLK: now also R16.1
- net _PI_LRCLK: now reaches J3.35 (GPIO19/MISO1)
- net _PI_LRCLK: now also R17.1
- net _PI_SDATA_O: now reaches J3.40 (GPIO21/SCLK1)
- net _PI_SDATA_O: now also R18.1; no longer R16.1
- net AMP_SPK_SLEEP: no longer names the net of U1.46 (MP7)
- net GAIN0_OUT: no longer names the net of U1.39 (LRCLK_OUT0/MP4)
- net GAIN1_OUT: no longer names the net of U1.42 (LRCLK_OUT1/MP5)
- net VPOT1: no longer names the net of U1.9 (AUXADC1)
- new net MCU/I2S3_MCK: RN5.1 (R1.1)
- new net MCU/I2S3_SCK: RN5.2 (R2.1)
- new net MCU/I2S3_SD: RN5.4 (R4.1)
- new net MCU/I2S3_WS: RN5.3 (R3.1)
- new net MCU_CLOCK: RN1.1 (R1.1)
- new net USB_MCLK: RN5.8 (R1.2)
- no-connect marks 30 -> 32
Other:
- sheet Power-15V renamed Power
- removed sheet I2S-AMP-2CH-A
- removed sheet I2S-AMP-2CH-B
- removed sheet USB I2S
- added sheet Amplifiers (amplifiers.kicad_sch)
- added sheet MCU (mcu.kicad_sch)
- sheet Power ports: added VOUT_1V8; removed none
- note removed: "GAIN[1:0] 00: 12.9 V full-scale 01: 15.1 V full-scale 10: 25.15 V full-scale (not recommended on TAS5760L) 11: Software-controlled"
- moved on the sheet: J2, J3, R1, R2, RV1, U2

Commit message: prod. version blus mini a
Parts:
- removed RN1, RN2, RN3, RN5: R_Pack04, Resistor_SMD:R_Array_Convex_4x0603, symbol Device:R_Pack04
- added H1, H2, H3, H4: MountingHole, MountingHole:MountingHole_3.2mm_M3_ISO7380_Pad, symbol Mechanical:MountingHole
- added R16, R17, R18, R19, R20, R21, R22, R27, R29, R30, R33, R38, R39, R40: 33, Resistor_SMD:R_0402_1005Metric, symbol Device:R
- C61: renamed from C25; MPN (none) -> C13585; Mfr.Nr. GRM31CR71H475KA12L -> (none)
- C62: renamed from C26; MPN (none) -> C13585; Mfr.Nr. GRM31CR71H475KA12L -> (none)
- C64: renamed from C7; MPN (none) -> C307331; Mfr.Nr. GRM31CR71H475KA12L -> (none)
- C65: renamed from C13; MPN (none) -> C307331; Mfr.Nr. GRM31CR71H475KA12L -> (none)
- C67: renamed from C3; MPN (none) -> C15195; Mfr.Nr. GRM31CR71H475KA12L -> (none)
- C68: renamed from C11; MPN (none) -> C15195; Mfr.Nr. GRM31CR71H475KA12L -> (none)
- C71: renamed from C8; MPN (none) -> C307331; Mfr.Nr. GRM31CR71H475KA12L -> (none)
- C72: renamed from C4; MPN (none) -> C15195; Mfr.Nr. GRM31CR71H475KA12L -> (none)
- C73: renamed from C10; MPN (none) -> C15195; Mfr.Nr. GRM31CR71H475KA12L -> (none)
- C74: renamed from C12; MPN (none) -> C307331; Mfr.Nr. GRM31CR71H475KA12L -> (none)
- C77: renamed from C17; MPN (none) -> C307331; Mfr.Nr. GRM31CR71H475KA12L -> (none)
- C78: renamed from C14; MPN (none) -> C15195; Mfr.Nr. GRM31CR71H475KA12L -> (none)
- C79: renamed from C20; MPN (none) -> C15195; Mfr.Nr. GRM31CR71H475KA12L -> (none)
- C80: renamed from C23; MPN (none) -> C307331; Mfr.Nr. GRM31CR71H475KA12L -> (none)
- C82: renamed from C5; MPN (none) -> C15195; Mfr.Nr. GRM31CR71H475KA12L -> (none)
- C83: renamed from C16; MPN (none) -> C15195; Mfr.Nr. GRM31CR71H475KA12L -> (none)
- C84: renamed from C21; MPN (none) -> C15195; Mfr.Nr. GRM31CR71H475KA12L -> (none)
- C85: renamed from C15; MPN (none) -> C15195; Mfr.Nr. GRM31CR71H475KA12L -> (none)
- C87: renamed from C9; MPN (none) -> C307331; Mfr.Nr. GRM31CR71H475KA12L -> (none)
- C88: renamed from C19; MPN (none) -> C307331; Mfr.Nr. GRM31CR71H475KA12L -> (none)
- C89: renamed from C24; MPN (none) -> C307331; Mfr.Nr. GRM31CR71H475KA12L -> (none)
- C90: renamed from C18; MPN (none) -> C307331; Mfr.Nr. GRM31CR71H475KA12L -> (none)
- C91: renamed from C22; MPN (none) -> C13585; Mfr.Nr. GRM31CR71H475KA12L -> (none)
- C92: renamed from C27; MPN (none) -> C13585; Mfr.Nr. GRM31CR71H475KA12L -> (none)
- C93: renamed from C2; MPN (none) -> C1527
- C95: renamed from C6; value 5.6n -> 4.7n; MPN (none) -> C1538
- J10: renamed from J2; footprint Connector_IDC:IDC-Header_2x08_P2.54mm_Vertical -> Connector_IDC:IDC-Header_2x08_P2.54mm_Horizontal
- Q1: JLCPCB Rotation Offset (none) -> 180; MPN (none) -> C8542
- R28: renamed from R2; value 4.3k -> 4.7k; MPN (none) -> C25900
- R31: renamed from R1; value 4.3k -> 4.7k; MPN (none) -> C25900
- R34: renamed from R13; value 0.47 -> 1; MPN (none) -> C25086
- R36: renamed from R3; value 4.3k -> 4.7k; MPN (none) -> C25900
- R37: renamed from R4; value 4.3k -> 4.7k; MPN (none) -> C25900
- R41: renamed from R18; MPN (none) -> C25105
- R42: renamed from R17; MPN (none) -> C25105
- R43: renamed from R16; MPN (none) -> C25105
- RV1: value PTV09A-1020F-B203 -> R_Potentiometer; symbol Device:R_POT -> Device:R_Potentiometer
- renumbered J3 to J11, J1 to J9, U1 to U11, U2 to U13
Connections:
- net Power/GND_IN is gone; now on net GND: J9.1 (Pin_1)
- net AMP1_BCLK: now also R20.1
- net AMP1_LRCLK: now also R21.1
- net AMP1_SDIN: now also R19.1
- net AMP2_BCLK: now also R17.1
- net AMP2_LRCLK: now also R18.1
- net AMP2_SDIN: now also R16.1
- net Clock/CLK0: now also R38.2
- net Clock/CLK1: now also R39.2
- net Clock/CLK2: now also R40.2
- net DSP_CLOCK: now also R40.1
- net EXT_MCLK: now also R39.1
- net EXT_MDO: now also R22.1
- net MCU/I2S3_SCK: now also R29.2
- net MCU/I2S3_SD: now also R33.2
- net MCU/I2S3_WS: now also R30.2
- net MCU_CLOCK: now also R38.1
- net PI_SDATA_I: now also R27.1
- net USB_BCLK: now also R29.1
- net USB_LRCLK: now also R30.1
- net USB_SDATA: now also R33.1
- net _AMP1_BCLK: now also R20.2
- net _AMP1_LRCLK: now also R21.2
- net _AMP1_SDIN: now also R19.2
- net _AMP2_BCLK: now also R17.2
- net _AMP2_LRCLK: now also R18.2
- net _AMP2_SDIN: now also R16.2
- net _EXT_MDO: now also R22.2
- net _PI_SDATA_I: now also R27.2
- net +3.3VA renamed +3.3V
- net +5VA renamed +5V
- net AUX_BCLK: no longer names the net of U11.68 (BCLK_IN3)
- net AUX_LRCLK: no longer names the net of U11.69 (LRCLK_IN3/MP13)
- net AUX_MDI: no longer names the net of U11.70 (SDATA_IN3)
- net Power/15V0_IN renamed VPP
- no-connect marks 32 -> 36
Other:
- sheet Power ports: added none; removed 15V0_IN, GND_IN, VOUT_15V0
- note added: "Adjusted filter component values, for availability"
- moved on the sheet: J9, R41, R42
