File: Hardware/dsp-amplifier-x4.kicad_sch (KiCad schematic)
At the start: 59 parts, among them J10 EXT, J11 Raspberry_Pi_2_3, J9 Screw_Terminal_01x02, Q1 SS8550, U11 ADAU1452, U13 TSOP583xx

Commit message: feat!: wip, version b
Parts:
- removed J10: EXT, Connector_IDC:IDC-Header_2x08_P2.54mm_Horizontal, symbol Connector_Generic:Conn_02x08_Odd_Even
- removed R16, R17, R18: 33, Resistor_SMD:R_0402_1005Metric, symbol Device:R
- added J10: Conn_01x10_Female, Connector_Debug:WR-WST REDFIT IDC 10, symbol Connector:Conn_01x10_Female
- added R46, R47: 4.7k, Resistor_SMD:R_0402_1005Metric, symbol Device:R
- J11: footprint rpi_socket:PinSocket_2x20_P2.54mm_Vertical -> Connector_Rpi:PinSocket_2x20_P2.54mm_Vertical; Mfr.Nr. (none) -> DK
- J9: footprint terminal_connectors:wuerth_691216410002 -> Connector_Terminal:wuerth_691216410002; Mfr.Nr. (none) -> DK
- RV1, U11: Mfr.Nr. (none) -> M
- U13: Mfr.Nr. (none) -> DK
Connections:
- net +3.3V: now also J10.7 (Pin_7), R46.2, R47.2
- net +5V: now also J10.1 (Pin_1)
- net EXT_BCLK: now also J10.4 (Pin_4)
- net EXT_LRCLK: now also J10.5 (Pin_5)
- net EXT_MDI: now also J10.2 (Pin_2)
- net EXT_MDO: now also J10.3 (Pin_3)
- net GND: now also J10.10 (Pin_10)
- net PI_SCL: now also J10.9 (Pin_9), R46.1
- net PI_SDA: now also J10.8 (Pin_8), R47.1
- net VPOT0: no longer U11.11 (AUXADC3)
- net AMP_NSPK_SD renamed DSP_STATUS
- net EXT_MCLK renamed EXT_CLOCK
- net EXT_CLOCK: now also J10.6 (Pin_6)
- net _AMP2_BCLK: no longer names the net of U11.51 (BCLK_OUT3)
- net _AMP2_LRCLK: no longer names the net of U11.50 (LRCLK_OUT3/MP9)
- net _AMP2_SDIN: no longer names the net of U11.52 (SDATA_OUT3)
- no-connect marks 36 -> 40
Other:
- sheet Amplifiers ports: added none; removed LRCKB, SCLKB, SDINB
- sheet MCU ports: added ADC1_IN9, DSP_STATUS, NSPK_SD; removed none
- note added: "IC2 for DSP?"
- moved on the sheet: R19, RV1

Commit message: fix: issues with rev a
Parts:
- removed J10: Conn_01x10_Female, Connector_Debug:WR-WST REDFIT IDC 10, symbol Connector:Conn_01x10_Female
- removed R27: 33, Resistor_SMD:R_0402_1005Metric, symbol Device:R
- added J10: Conn_01x16_Female, Connector_Debug:WR-WST REDFIT IDC 16, symbol Connector:Conn_01x16_Female
- added R16, R17: 33, Resistor_SMD:R_0402_1005Metric, symbol Device:R
Connections:
- net +3.3V: now also J10.1 (Pin_1)
- net +5V: now also J10.2 (Pin_2)
- net EXT_CLOCK: now also J10.12 (Pin_12)
- net EXT_MDI: now also J10.10 (Pin_10)
- net EXT_MDO: now also J10.4 (Pin_4)
- net GND: now also J10.11 (Pin_11), J10.13 (Pin_13), J10.16 (Pin_16), J10.3 (Pin_3), J10.7 (Pin_7)
- net PI_SCL: now also J10.15 (Pin_15)
- net PI_SDA: now also J10.14 (Pin_14)
- net VPOT0: now also U11.8 (AUXADC0)
- net _EXT_BCLKO: now reaches U11.42 (LRCLK_OUT1/MP5)
- net _EXT_BCLKO: now also R16.2
- net _EXT_LRCLKO: now reaches U11.43 (BCLK_OUT1)
- net _EXT_LRCLKO: now also R17.2
- net EXT_BCLK renamed EXT_BCLKI
- net EXT_BCLKI: now also J10.8 (Pin_8)
- net EXT_LRCLK renamed EXT_LRCLKI
- net EXT_LRCLKI: now also J10.9 (Pin_9)
- net _PI_SDATA_I: no longer names the net of U11.41 (SDATA_OUT0)
- new net EXT_BCLKO: J10.6 (Pin_6), R16.1
- new net EXT_LRCLKO: J10.5 (Pin_5), R17.1
- no-connect marks 40 -> 38
Other:
- note removed: "IC2 for DSP?"
- moved on the sheet: R19, R20, R21, R22, U13

Commit message: chore: cleanup
Other:
- sheet EEPROM: file i2c_eeprom.kicad_sch -> spi_eeprom.kicad_sch
- sheet Power: file power_15v.kicad_sch -> power.kicad_sch
- sheet SPDIF: file SPDIF.kicad_sch -> spdif.kicad_sch
