File: Hardware/I2S-AMP-2CH.kicad_sch (KiCad schematic)
At the start: 19 parts, among them U8 TAS5760MDCAR

Commit message: Updated power supply
Parts:
- renumbered C62 to C48, C63 to C49, C64 to C50, C65 to C51, C66 to C52, C67 to C53, C68 to C54, C69 to C55, C70 to C56, C71 to C57, C72 to C58, C73 to C59, C74 to C60, C75 to C61, L7 to L3, L8 to L4, L9 to L5, L10 to L6, U8 to U7
Other:
- note added: "Alternative: TAS5760L (max. 15 V)"
Changed lines of the file:
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@@
+    (effects (font (size 1.524 1.524)) (justify left bottom))
+  )
+  (text "Alternative: TAS5760L (max. 15 V)" (at 93.98 33.02 0)
     (effects (font (size 1.524 1.524)) (justify left bottom))
   )
@@
   (symbol (lib_id "Device:C") (at 74.93 41.91 0)
     (in_bom yes) (on_board yes)
-    (property "Reference" "C64" (id 0) (at 76.2 39.37 0)
+    (property "Reference" "C50" (id 0) (at 76.2 39.37 0)
       (effects (font (size 1.27 1.27)) (justify left))
     )
@@
   (symbol (lib_id "Device:C") (at 114.3 149.86 0)
     (in_bom yes) (on_board yes)
-    (property "Reference" "C66" (id 0) (at 115.57 147.32 0)
+    (property "Reference" "C52" (id 0) (at 115.57 147.32 0)
       (effects (font (size 1.27 1.27)) (justify left))
     )
@@
   (symbol (lib_id "Device:C") (at 59.69 64.77 180)
     (in_bom yes) (on_board yes)
-    (property "Reference" "C63" (id 0) (at 58.42 67.31 0)
+    (property "Reference" "C49" (id 0) (at 58.42 67.31 0)
       (effects (font (size 1.27 1.27)) (justify left))
     )
@@
   (symbol (lib_id "Device:C") (at 46.99 64.77 180)
     (in_bom yes) (on_board yes)
-    (property "Reference" "C62" (id 0) (at 45.72 67.31 0)
+    (property "Reference" "C48" (id 0) (at 45.72 67.31 0)
       (effects (font (size 1.27 1.27)) (justify left))
     )
@@
   (symbol (lib_id "power:GND") (at 114.3 156.21 0)
     (in_bom yes) (on_board yes)
-    (property "Reference" "#PWR080" (id 0) (at 114.3 162.56 0)
+    (property "Reference" "#PWR068" (id 0) (at 114.3 162.56 0)
       (effects (font (size 1.27 1.27)) hide)
     )
@@
   (symbol (lib_id "power:GND") (at 74.93 46.99 0)
     (in_bom yes) (on_board yes)
-    (property "Reference" "#PWR075" (id 0) (at 74.93 53.34 0)
+    (property "Reference" "#PWR063" (id 0) (at 74.93 53.34 0)
       (effects (font (size 1.27 1.27)) hide)
     )
@@
   (symbol (lib_id "Device:C") (at 143.51 97.79 90)
     (in_bom yes) (on_board yes)
-    (property "Reference" "C71" (id 0) (at 140.97 96.52 90)
+    (property "Reference" "C57" (id 0) (at 140.97 96.52 90)
       (effects (font (size 1.27 1.27)) (justify left))
     )
@@
   (symbol (lib_id "Device:C") (at 143.51 71.12 90)
     (in_bom yes) (on_board yes)
-    (property "Reference" "C69" (id 0) (at 140.97 69.85 90)
+    (property "Reference" "C55" (id 0) (at 140.97 69.85 90)
       (effects (font (size 1.27 1.27)) (justify left))
     )
@@
   (symbol (lib_id "Device:C") (at 143.51 62.23 90)
     (in_bom yes) (on_board yes)
-    (property "Reference" "C68" (id 0) (at 140.97 60.96 90)
+    (property "Reference" "C54" (id 0) (at 140.97 60.96 90)
       (effects (font (size 1.27 1.27)) (justify left))
     )
@@
   (symbol (lib_id "Device:L") (at 166.37 59.69 90)
     (in_bom yes) (on_board yes)
-    (property "Reference" "L7" (id 0) (at 166.37 57.15 90))
+    (property "Reference" "L3" (id 0) (at 166.37 57.15 90))
     (property "Value" "10u" (id 1) (at 166.37 62.23 90))
     (property "Footprint" "Inductor_SMD:L_Abracon_ASPI-0630LR" (id 2) (at 166.37 59.69 0)
@@
   (symbol (lib_id "Device:C") (at 179.07 63.5 270)
     (in_bom yes) (on_board yes)
-    (property "Reference" "C72" (id 0) (at 181.61 64.77 0)
+    (property "Reference" "C58" (id 0) (at 181.61 64.77 0)
       (effects (font (size 1.27 1.27)) (justify left))
     )
@@
   (symbol (lib_id "power:VAA") (at 114.3 142.24 0)
     (in_bom yes) (on_board yes)
-    (property "Reference" "#PWR079" (id 0) (at 114.3 146.05 0)
+    (property "Reference" "#PWR067" (id 0) (at 114.3 146.05 0)
       (effects (font (size 1.27 1.27)) hide)
     )
@@
   (symbol (lib_id "tas5760:TAS5760MDCAR") (at 111.76 81.28 0)
     (in_bom yes) (on_board yes)
-    (property "Reference" "U8" (id 0) (at 111.76 31.75 0)
+    (property "Reference" "U7" (id 0) (at 111.76 31.75 0)
       (effects (font (size 1.524 1.524)) (justify top) hide)
     )
-    (property "Value" "TAS5760MDCAR" (id 1) (at 111.76 43.2562 0)
+    (property "Value" "TAS5760MDCAR" (id 1) (at 101.6 48.26 0)
       (effects (font (size 1.524 1.524)))
     )
@@
   (symbol (lib_id "power:+3.3V") (at 118.11 40.64 0)
     (in_bom yes) (on_board yes)
-    (property "Reference" "#PWR081" (id 0) (at 118.11 44.45 0)
+    (property "Reference" "#PWR069" (id 0) (at 118.11 44.45 0)
       (effects (font (size 1.27 1.27)) hide)
     )
@@
   (symbol (lib_id "power:VAA") (at 125.73 40.64 0)
     (in_bom yes) (on_board yes)
-    (property "Reference" "#PWR082" (id 0) (at 125.73 44.45 0)
+    (property "Reference" "#PWR070" (id 0) (at 125.73 44.45 0)
       (effects (font (size 1.27 1.27)) hide)
     )
@@
   (symbol (lib_id "power:VAA") (at 113.03 40.64 0)
     (in_bom yes) (on_board yes)
-    (property "Reference" "#PWR078" (id 0) (at 113.03 44.45 0)
+    (property "Reference" "#PWR066" (id 0) (at 113.03 44.45 0)
       (effects (font (size 1.27 1.27)) hide)
     )
@@
   (symbol (lib_id "power:GND") (at 106.68 119.38 0)
     (in_bom yes) (on_board yes)
-    (property "Reference" "#PWR077" (id 0) (at 106.68 125.73 0)
+    (property "Reference" "#PWR065" (id 0) (at 106.68 125.73 0)
       (effects (font (size 1.27 1.27)) hide)
     )
@@
   (symbol (lib_id "Device:CP") (at 124.46 149.86 0)
     (in_bom yes) (on_board yes)
-    (property "Reference" "C67" (id 0) (at 127.4572 148.6916 0)
+    (property "Reference" "C53" (id 0) (at 127.4572 148.6916 0)
       (effects (font (size 1.27 1.27)) (justify left))
     )
@@
   (symbol (lib_id "Device:C") (at 104.14 149.86 0)
     (in_bom yes) (on_board yes)
-    (property "Reference" "C65" (id 0) (at 105.41 147.32 0)
+    (property "Reference" "C51" (id 0) (at 105.41 147.32 0)
       (effects (font (size 1.27 1.27)) (justify left))
     )
@@
   (symbol (lib_id "power:GND") (at 77.47 80.01 270)
     (in_bom yes) (on_board yes)
-    (property "Reference" "#PWR076" (id 0) (at 71.12 80.01 0)
+    (property "Reference" "#PWR064" (id 0) (at 71.12 80.01 0)
       (effects (font (size 1.27 1.27)) hide)
     )
@@
   (symbol (lib_id "Device:C") (at 143.51 88.9 90)
     (in_bom yes) (on_board yes)
-    (property "Reference" "C70" (id 0) (at 140.97 87.63 90)
+    (property "Reference" "C56" (id 0) (at 140.97 87.63 90)
       (effects (font (size 1.27 1.27)) (justify left))
     )
@@
   (symbol (lib_id "Device:L") (at 166.37 73.66 90)
     (in_bom yes) (on_board yes)
-    (property "Reference" "L8" (id 0) (at 166.37 71.12 90))
+    (property "Reference" "L4" (id 0) (at 166.37 71.12 90))
     (property "Value" "10u" (id 1) (at 166.37 76.2 90))
     (property "Footprint" "Inductor_SMD:L_Abracon_ASPI-0630LR" (id 2) (at 166.37 73.66 0)
@@
   (symbol (lib_id "Device:L") (at 166.37 86.36 90)
     (in_bom yes) (on_board yes)
-    (property "Reference" "L9" (id 0) (at 166.37 83.82 90))
+    (property "Reference" "L5" (id 0) (at 166.37 83.82 90))
     (property "Value" "10u" (id 1) (at 166.37 88.9 90))
     (property "Footprint" "Inductor_SMD:L_Abracon_ASPI-0630LR" (id 2) (at 166.37 86.36 0)
@@
   (symbol (lib_id "Device:L") (at 166.37 100.33 90)
     (in_bom yes) (on_board yes)
-    (property "Reference" "L10" (id 0) (at 166.37 97.79 90))
+    (property "Reference" "L6" (id 0) (at 166.37 97.79 90))
     (property "Value" "10u" (id 1) (at 166.37 102.87 90))
     (property "Footprint" "Inductor_SMD:L_Abracon_ASPI-0630LR" (id 2) (at 166.37 100.33 0)
@@
   (symbol (lib_id "Device:C") (at 179.07 77.47 270)
     (in_bom yes) (on_board yes)
-    (property "Reference" "C73" (id 0) (at 181.61 78.74 0)
+    (property "Reference" "C59" (id 0) (at 181.61 78.74 0)
       (effects (font (size 1.27 1.27)) (justify left))
     )
@@
   (symbol (lib_id "Device:C") (at 179.07 90.17 270)
     (in_bom yes) (on_board yes)
-    (property "Reference" "C74" (id 0) (at 181.61 91.44 0)
+    (property "Reference" "C60" (id 0) (at 181.61 91.44 0)
       (effects (font (size 1.27 1.27)) (justify left))
     )
@@
   (symbol (lib_id "Device:C") (at 179.07 104.14 270)
     (in_bom yes) (on_board yes)
-    (property "Reference" "C75" (id 0) (at 181.61 105.41 0)
+    (property "Reference" "C61" (id 0) (at 181.61 105.41 0)
       (effects (font (size 1.27 1.27)) (justify left))
     )
@@
   (symbol (lib_id "power:GND") (at 185.42 66.04 0)
     (in_bom yes) (on_board yes)
-    (property "Reference" "#PWR083" (id 0) (at 185.42 72.39 0)
+    (property "Reference" "#PWR071" (id 0) (at 185.42 72.39 0)
       (effects (font (size 1.27 1.27)) hide)
     )
@@
   (symbol (lib_id "power:GND") (at 185.42 80.01 0)
     (in_bom yes) (on_board yes)
-    (property "Reference" "#PWR084" (id 0) (at 185.42 86.36 0)
+    (property "Reference" "#PWR072" (id 0) (at 185.42 86.36 0)
       (effects (font (size 1.27 1.27)) hide)
     )
@@
   (symbol (lib_id "power:GND") (at 185.42 92.71 0)
     (in_bom yes) (on_board yes)
-    (property "Reference" "#PWR085" (id 0) (at 185.42 99.06 0)
+    (property "Reference" "#PWR073" (id 0) (at 185.42 99.06 0)
       (effects (font (size 1.27 1.27)) hide)
     )
@@
   (symbol (lib_id "power:GND") (at 185.42 106.68 0)
     (in_bom yes) (on_board yes)
-    (property "Reference" "#PWR086" (id 0) (at 185.42 113.03 0)
-      (effects (font (size 1.27 1.27)) hide)
-    )
+    (property "Reference" "#PWR074" (id 0) (at 185.42 113.03 0)
+      (effects (font (size 1.27 1.27)) hide)
+    )
