File: Hardware/SPDIF.kicad_sch (KiCad schematic)
At the start: 8 parts, among them J10 Conn_Coaxial, J9 Conn_Coaxial, T1 DA100J

Commit message: Updated power supply
Changed lines of the file:
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@@
     (pin "2")
   )
-  (symbol (lib_id "Device:R") (at 97.79 96.52 0)
+  (symbol (lib_id "Device:R") (at 97.79 96.52 0) (unit 1)
     (in_bom yes) (on_board yes)
     (property "Reference" "R41" (id 0) (at 92.5322 96.52 90))
@@
     (pin "2")
   )
-  (symbol (lib_id "Device:R") (at 161.29 93.98 0)
+  (symbol (lib_id "Device:R") (at 161.29 93.98 0) (unit 1)
     (in_bom yes) (on_board yes)
     (property "Reference" "R43" (id 0) (at 156.0322 93.98 90))
@@
     (pin "2")
   )
-  (symbol (lib_id "Device:R") (at 161.29 83.82 0)
+  (symbol (lib_id "Device:R") (at 161.29 83.82 0) (unit 1)
     (in_bom yes) (on_board yes)
     (property "Reference" "R42" (id 0) (at 156.0322 83.82 90))

Commit message: feat: updated amplifier IC, finalized design
Parts:
- C85, C86: footprint Capacitor_SMD:C_0603_1608Metric_Pad1.08x0.95mm_HandSolder -> Capacitor_SMD:C_0402_1005Metric
- R41, R42, R43: footprint Resistor_SMD:R_0603_1608Metric_Pad0.98x0.95mm_HandSolder -> Resistor_SMD:R_0402_1005Metric
Changed lines of the file:
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@@
       (effects (font (size 1.27 1.27)) (justify left))
     )
-    (property "Footprint" "Capacitor_SMD:C_0603_1608Metric_Pad1.08x0.95mm_HandSolder" (id 2) (at 110.49 89.8652 0)
+    (property "Footprint" "Capacitor_SMD:C_0402_1005Metric" (id 2) (at 110.49 89.8652 0)
       (effects (font (size 0.762 0.762)) hide)
     )
-    (property "Datasheet" "" (id 3) (at 106.68 88.9 0)
+    (property "Datasheet" "~" (id 3) (at 106.68 88.9 0)
       (effects (font (size 1.524 1.524)))
     )
@@
     (property "Reference" "R41" (id 0) (at 92.5322 96.52 90))
     (property "Value" "75" (id 1) (at 94.8436 96.52 90))
-    (property "Footprint" "Resistor_SMD:R_0603_1608Metric_Pad0.98x0.95mm_HandSolder" (id 2) (at 96.012 96.52 90)
+    (property "Footprint" "Resistor_SMD:R_0402_1005Metric" (id 2) (at 96.012 96.52 90)
       (effects (font (size 1.27 1.27)) hide)
     )
@@
       (effects (font (size 1.27 1.27)) (justify left))
     )
-    (property "Footprint" "Capacitor_SMD:C_0603_1608Metric_Pad1.08x0.95mm_HandSolder" (id 2) (at 170.18 89.8652 0)
+    (property "Footprint" "Capacitor_SMD:C_0402_1005Metric" (id 2) (at 170.18 89.8652 0)
       (effects (font (size 0.762 0.762)) hide)
     )
-    (property "Datasheet" "" (id 3) (at 166.37 88.9 0)
+    (property "Datasheet" "~" (id 3) (at 166.37 88.9 0)
       (effects (font (size 1.524 1.524)))
     )
@@
     (property "Reference" "R43" (id 0) (at 156.0322 93.98 90))
     (property "Value" "107" (id 1) (at 158.3436 93.98 90))
-    (property "Footprint" "Resistor_SMD:R_0603_1608Metric_Pad0.98x0.95mm_HandSolder" (id 2) (at 159.512 93.98 90)
+    (property "Footprint" "Resistor_SMD:R_0402_1005Metric" (id 2) (at 159.512 93.98 90)
       (effects (font (size 1.27 1.27)) hide)
     )
@@
     (property "Reference" "R42" (id 0) (at 156.0322 83.82 90))
     (property "Value" "243" (id 1) (at 158.3436 83.82 90))
-    (property "Footprint" "Resistor_SMD:R_0603_1608Metric_Pad0.98x0.95mm_HandSolder" (id 2) (at 159.512 83.82 90)
+    (property "Footprint" "Resistor_SMD:R_0402_1005Metric" (id 2) (at 159.512 83.82 90)
       (effects (font (size 1.27 1.27)) hide)
     )

Commit message: prod. version blus mini a
Parts:
- C60: renamed from C85; MPN (none) -> C15195
- C97: renamed from C86; MPN (none) -> C15195
- R15: renamed from R41; MPN (none) -> C25133
- R44: renamed from R43; value 107 -> 100; MPN (none) -> C25076
- R45: renamed from R42; value 243 -> 220; MPN (none) -> C25091
- renumbered J9 to J2, J10 to J4
Connections:
- no-connect marks 1 -> 0
Changed lines of the file:
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@@
   (junction (at 97.79 88.9) (diameter 0) (color 0 0 0 0)
   )
-  (no_connect (at -11.43 134.62))
   (wire (pts (xy 161.29 97.79) (xy 161.29 99.06))
     (stroke (width 0) (type default) (color 0 0 0 0))
@@
   (symbol (lib_id "Device:C") (at 106.68 88.9 90) (mirror x) (unit 1)
     (in_bom yes) (on_board yes)
-    (property "Reference" "C85" (id 0) (at 104.14 89.535 0)
+    (property "Reference" "C60" (id 0) (at 104.14 89.535 0)
       (effects (font (size 1.27 1.27)) (justify left))
     )
@@
       (effects (font (size 1.524 1.524)))
     )
+    (property "Mfr.Nr." "" (id 4) (at 106.68 88.9 0)
+      (effects (font (size 1.27 1.27)) hide)
+    )
+    (property "MPN" "C15195" (id 5) (at 106.68 88.9 0)
+      (effects (font (size 1.27 1.27)) hide)
+    )
     (pin "1")
     (pin "2")
@@
   (symbol (lib_id "Device:R") (at 97.79 96.52 0) (unit 1)
     (in_bom yes) (on_board yes)
-    (property "Reference" "R41" (id 0) (at 92.5322 96.52 90))
+    (property "Reference" "R15" (id 0) (at 92.5322 96.52 90))
     (property "Value" "75" (id 1) (at 94.8436 96.52 90))
     (property "Footprint" "Resistor_SMD:R_0402_1005Metric" (id 2) (at 96.012 96.52 90)
@@
       (effects (font (size 1.27 1.27)) hide)
     )
+    (property "Mfr.Nr." "" (id 4) (at 97.79 96.52 0)
+      (effects (font (size 1.27 1.27)) hide)
+    )
+    (property "MPN" "C25133" (id 5) (at 97.79 96.52 0)
+      (effects (font (size 1.27 1.27)) hide)
+    )
     (pin "1")
     (pin "2")
@@
     (property "Datasheet" "" (id 3) (at 184.15 81.28 0)
       (effects (font (size 1.524 1.524)) hide)
+    )
+    (property "Mfr.Nr." "" (id 4) (at 184.15 91.44 0)
+      (effects (font (size 1.27 1.27)) hide)
     )
     (pin "1")
@@
   (symbol (lib_id "power:GND") (at 170.18 95.25 0) (unit 1)
     (in_bom yes) (on_board yes)
-    (property "Reference" "#PWR0105" (id 0) (at 170.18 101.6 0)
+    (property "Reference" "#PWR0192" (id 0) (at 170.18 101.6 0)
       (effects (font (size 1.27 1.27)) hide)
     )
     (property "Value" "GND" (id 1) (at 170.18 99.06 0))
     (property "Footprint" "" (id 2) (at 170.18 95.25 0)
-      (effects (font (size 1.524 1.524)))
+      (effects (font (size 1.27 1.27)) hide)
     )
     (property "Datasheet" "" (id 3) (at 170.18 95.25 0)
-      (effects (font (size 1.524 1.524)))
+      (effects (font (size 1.27 1.27)) hide)
     )
     (pin "1")
@@
   (symbol (lib_id "Device:C") (at 166.37 88.9 90) (mirror x) (unit 1)
     (in_bom yes) (on_board yes)
-    (property "Reference" "C86" (id 0) (at 163.83 89.535 0)
+    (property "Reference" "C97" (id 0) (at 163.83 89.535 0)
       (effects (font (size 1.27 1.27)) (justify left))
     )
@@
       (effects (font (size 1.524 1.524)))
     )
+    (property "Mfr.Nr." "" (id 4) (at 166.37 88.9 0)
+      (effects (font (size 1.27 1.27)) hide)
+    )
+    (property "MPN" "C15195" (id 5) (at 166.37 88.9 0)
+      (effects (font (size 1.27 1.27)) hide)
+    )
     (pin "1")
     (pin "2")
@@
   (symbol (lib_id "Device:R") (at 161.29 93.98 0) (unit 1)
     (in_bom yes) (on_board yes)
-    (property "Reference" "R43" (id 0) (at 156.0322 93.98 90))
-    (property "Value" "107" (id 1) (at 158.3436 93.98 90))
+    (property "Reference" "R44" (id 0) (at 156.0322 93.98 90))
+    (property "Value" "100" (id 1) (at 158.3436 93.98 90))
     (property "Footprint" "Resistor_SMD:R_0402_1005Metric" (id 2) (at 159.512 93.98 90)
       (effects (font (size 1.27 1.27)) hide)
@@
       (effects (font (size 1.27 1.27)) hide)
     )
+    (property "Mfr.Nr." "" (id 4) (at 161.29 93.98 0)
+      (effects (font (size 1.27 1.27)) hide)
+    )
+    (property "MPN" "C25076" (id 5) (at 161.29 93.98 0)
+      (effects (font (size 1.27 1.27)) hide)
+    )
     (pin "1")
     (pin "2")
@@
   (symbol (lib_id "Device:R") (at 161.29 83.82 0) (unit 1)
     (in_bom yes) (on_board yes)
-    (property "Reference" "R42" (id 0) (at 156.0322 83.82 90))
-    (property "Value" "243" (id 1) (at 158.3436 83.82 90))
+    (property "Reference" "R45" (id 0) (at 156.0322 83.82 90))
+    (property "Value" "220" (id 1) (at 158.3436 83.82 90))
     (property "Footprint" "Resistor_SMD:R_0402_1005Metric" (id 2) (at 159.512 83.82 90)
       (effects (font (size 1.27 1.27)) hide)
@@
       (effects (font (size 1.27 1.27)) hide)
     )
+    (property "Mfr.Nr." "" (id 4) (at 161.29 83.82 0)
+      (effects (font (size 1.27 1.27)) hide)
+    )
+    (property "MPN" "C25091" (id 5) (at 161.29 83.82 0)
+      (effects (font (size 1.27 1.27)) hide)
+    )
     (pin "1")
     (pin "2")
@@
   (symbol (lib_id "power:GND") (at 161.29 99.06 0) (unit 1)
     (in_bom yes) (on_board yes)
-    (property "Reference" "#PWR0104" (id 0) (at 161.29 105.41 0)
+    (property "Reference" "#PWR0193" (id 0) (at 161.29 105.41 0)
       (effects (font (size 1.27 1.27)) hide)
     )
     (property "Value" "GND" (id 1) (at 161.29 102.87 0))
     (property "Footprint" "" (id 2) (at 161.29 99.06 0)
-      (effects (font (size 1.524 1.524)))
+      (effects (font (size 1.27 1.27)) hide)
     )
     (property "Datasheet" "" (id 3) (at 161.29 99.06 0)
-      (effects (font (size 1.524 1.524)))
+      (effects (font (size 1.27 1.27)) hide)
     )
     (pin "1")
@@
   (symbol (lib_id "Connector:Conn_Coaxial") (at 88.9 88.9 0) (mirror y) (unit 1)
     (in_bom yes) (on_board yes)
-    (property "Reference" "J9" (id 0) (at 86.36 89.535 0)
+    (property "Reference" "J2" (id 0) (at 86.36 89.535 0)
       (effects (font (size 1.27 1.27)) (justify left))
     )
@@
       (effects (font (size 1.27 1.27)) hide)
     )
+    (property "Mfr.Nr." "" (id 4) (at 88.9 88.9 0)
+      (effects (font (size 1.27 1.27)) hide)
+    )
     (pin "1")
     (pin "2")
@@
   (symbol (lib_id "Connector:Conn_Coaxial") (at 203.2 88.9 0) (unit 1)
     (in_bom yes) (on_board yes)
-    (property "Reference" "J10" (id 0) (at 205.74 89.535 0)
+    (property "Reference" "J4" (id 0) (at 205.74 89.535 0)
       (effects (font (size 1.27 1.27)) (justify left))
     )
@@
       (effects (font (size 1.27 1.27)) hide)
     )
+    (property "Mfr.Nr." "" (id 4) (at 203.2 88.9 0)
+      (effects (font (size 1.27 1.27)) hide)
+    )
     (pin "1")
     (pin "2")
@@
   (symbol (lib_id "power:GND") (at 88.9 102.87 0) (unit 1)
     (in_bom yes) (on_board yes)
-    (property "Reference" "#PWR0103" (id 0) (at 88.9 109.22 0)
+    (property "Reference" "#PWR0189" (id 0) (at 88.9 109.22 0)
       (effects (font (size 1.27 1.27)) hide)
     )
     (property "Value" "GND" (id 1) (at 88.9 106.68 0))
     (property "Footprint" "" (id 2) (at 88.9 102.87 0)
-      (effects (font (size 1.524 1.524)))
+      (effects (font (size 1.27 1.27)) hide)
     )
     (property "Datasheet" "" (id 3) (at 88.9 102.87 0)
-      (effects (font (size 1.524 1.524)))
-    )
-    (pin "1")
+      (effects (font (size 1.27 1.27)) hide)
+    )
+    (pin "1")

Commit message: feat!: wip, version b
Parts:
- J2, J4: footprint connectors_audio:cui_rcj_02x -> Connector_Audio_Custom:cui_rcj_02x; Mfr.Nr. (none) -> DK
- T1: footprint da100j:SOIC-6 -> Transformer_Audio:SOIC-6; symbol transformer_audio:DA100J -> Transformer_Audio:DA100J; Mfr.Nr. (none) -> M
Changed lines of the file:
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@@
     (pin "2")
   )
-  (symbol (lib_id "transformer_audio:DA100J") (at 184.15 91.44 0) (unit 1)
+  (symbol (lib_id "Transformer_Audio:DA100J") (at 184.15 91.44 0) (unit 1)
     (in_bom yes) (on_board yes)
     (property "Reference" "T1" (id 0) (at 184.15 81.6102 0)
@@
       (effects (font (size 1.524 1.524)))
     )
-    (property "Footprint" "da100j:SOIC-6" (id 2) (at 184.15 81.28 0)
+    (property "Footprint" "Transformer_Audio:SOIC-6" (id 2) (at 184.15 81.28 0)
       (effects (font (size 1.524 1.524)) hide)
     )
@@
       (effects (font (size 1.524 1.524)) hide)
     )
-    (property "Mfr.Nr." "" (id 4) (at 184.15 91.44 0)
+    (property "Mfr.Nr." "M" (id 4) (at 184.15 91.44 0)
       (effects (font (size 1.27 1.27)) hide)
     )
@@
       (effects (font (size 1.27 1.27)) (justify left))
     )
-    (property "Footprint" "connectors_audio:cui_rcj_02x" (id 2) (at 88.9 88.9 0)
+    (property "Footprint" "Connector_Audio_Custom:cui_rcj_02x" (id 2) (at 88.9 88.9 0)
       (effects (font (size 1.27 1.27)) hide)
     )
@@
       (effects (font (size 1.27 1.27)) hide)
     )
-    (property "Mfr.Nr." "" (id 4) (at 88.9 88.9 0)
+    (property "Mfr.Nr." "DK" (id 4) (at 88.9 88.9 0)
       (effects (font (size 1.27 1.27)) hide)
     )
@@
       (effects (font (size 1.27 1.27)) (justify left))
     )
-    (property "Footprint" "connectors_audio:cui_rcj_02x" (id 2) (at 203.2 88.9 0)
+    (property "Footprint" "Connector_Audio_Custom:cui_rcj_02x" (id 2) (at 203.2 88.9 0)
       (effects (font (size 1.27 1.27)) hide)
     )
@@
       (effects (font (size 1.27 1.27)) hide)
     )
-    (property "Mfr.Nr." "" (id 4) (at 203.2 88.9 0)
+    (property "Mfr.Nr." "DK" (id 4) (at 203.2 88.9 0)
       (effects (font (size 1.27 1.27)) hide)
     )
