File: Hardware/clock.kicad_sch (KiCad schematic)
At the start: 4 parts, among them U12 74AVC9112, X1 ASV-24.576MHz-EJ-T

Commit message: feat!: wip, version b
Parts:
- U12: symbol buffers:74AVC9112 -> Buffers:74AVC9112; Mfr.Nr. (none) -> DK
- X1: Mfr.Nr. (none) -> DK
Other:
- company: TUD -> (none)
- title: freeDSP-AiO -> (none)
Changed lines of the file:
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@@
   (paper "A4")
   (title_block
-    (title "freeDSP-AiO")
-    (date "2018-08-09")
-    (rev "V1.0")
-    (company "TUD")
-    (comment 1 "Friedrich, Hoffmann, Kaiser, Schindler")
-    (comment 2 "Hauptseminar Kommunikationsnetze")
+    (date "2023-02-18")
   )
   (junction (at 116.84 49.53) (diameter 0) (color 0 0 0 0)
@@
       (effects (font (size 1.524 1.524)))
     )
-    (property "Mfr.Nr." "" (id 4) (at 132.08 81.28 0)
+    (property "Mfr.Nr." "DK" (id 4) (at 132.08 81.28 0)
       (effects (font (size 1.27 1.27)) hide)
     )
@@
     (pin "2")
   )
-  (symbol (lib_id "buffers:74AVC9112") (at 167.64 74.93 0) (unit 1)
+  (symbol (lib_id "Buffers:74AVC9112") (at 167.64 74.93 0) (unit 1)
     (in_bom yes) (on_board yes) (fields_autoplaced)
     (property "Reference" "U12" (id 0) (at 170.9294 71.0143 0)
@@
       (effects (font (size 1.27 1.27)) hide)
     )
-    (property "Mfr.Nr." "" (id 4) (at 167.64 74.93 0)
-      (effects (font (size 1.27 1.27)) hide)
-    )
+    (property "Mfr.Nr." "DK" (id 4) (at 167.64 74.93 0)
+      (effects (font (size 1.27 1.27)) hide)
+    )
