File: Hardware/mcu.kicad_sch (KiCad schematic)
At the start: 16 parts, among them J12 Conn_ST_STDC14, J8 USB_B, U6 USBLC6-2SC6, U9 STM32F401RBTx

Commit message: prod. version blus mini a
Parts:
- removed J12: Conn_ST_STDC14, Connector_PinHeader_1.27mm:PinHeader_2x07_P1.27mm_Vertical_SMD, symbol Connector:Conn_ST_STDC14
- added J3: REDFIT_SWD_6, connectors_debug:WR-WST REDFIT IDC 6 DBG, symbol connectors_debug:REDFIT_SWD_6
- added TP1: RX, TestPoint:TestPoint_THTPad_D2.0mm_Drill1.0mm, symbol Connector:TestPoint
- added TP2: TX, TestPoint:TestPoint_THTPad_D2.0mm_Drill1.0mm, symbol Connector:TestPoint
- C63: renamed from C35; MPN (none) -> C307331; Mfr.Nr. GRM31CR71H475KA12L -> (none)
- C70: renamed from C36; MPN (none) -> C307331; Mfr.Nr. GRM31CR71H475KA12L -> (none)
- C75: renamed from C1; MPN (none) -> C1779; Mfr.Nr. GRM31CR71H475KA12L -> (none)
- C76: renamed from C38; MPN (none) -> C307331; Mfr.Nr. GRM31CR71H475KA12L -> (none)
- C81: renamed from C39; MPN (none) -> C307331; Mfr.Nr. GRM31CR71H475KA12L -> (none)
- C86: renamed from C37; MPN (none) -> C307331; Mfr.Nr. GRM31CR71H475KA12L -> (none)
- R23: renamed from R29; MPN (none) -> C25105
- R24: renamed from R27; MPN (none) -> C25105
- R25: renamed from R31; value 4.3k -> 4.7k; MPN (none) -> C25900
- R26: renamed from R32; MPN (none) -> C25744
- R32: renamed from R30; value 4.3k -> 4.7k; MPN (none) -> C25900
- R35: renamed from R28; value 4.3k -> 4.7k; MPN (none) -> C25900
- U10: renamed from U9; JLCPCB Rotation Offset (none) -> -90; MPN (none) -> C75278
- U8: renamed from U6; JLCPCB Rotation Offset (none) -> 180
- renumbered J8 to J1
Connections:
- net GND: now also J3.5 (GND)
- net NRST: now also J3.3 (nRST)
- net SWO: now also J3.6 (SWO)
- net TCK: now also J3.4 (SWCLK)
- net TMS: now also J3.2 (SWDIO)
- net USART2_RX: now also TP1.1
- net USART2_TX: now also TP2.1
- net +3.3VA renamed +3.3V
- net +3.3V: now also J3.1 (VCC)
- no-connect marks 37 -> 34

Commit message: feat!: wip, version b
Parts:
- added SW1: BOOT, Button_Switch_SMD:SW_SPST_PTS810, symbol Switch:SW_SPST
- added SW2: NRST, Button_Switch_SMD:SW_SPST_PTS810, symbol Switch:SW_SPST
- J1: Mfr.Nr. (none) -> M
- J3: footprint connectors_debug:WR-WST REDFIT IDC 6 DBG -> Connector_Debug:WR-WST REDFIT IDC 6 DBG; symbol connectors_debug:REDFIT_SWD_6 -> Connectors_Debug:REDFIT_SWD_6
- U8: Mfr.Nr. (none) -> DK
Connections:
- net +3.3V: now also SW1.2 (B)
- net BOOT0: now also SW1.1 (A)
- net GND: now also SW2.1 (A)
- net I2S3_MCK: now also U10.14 (PA0)
- net NRST: now also SW2.2 (B)
- net ADC1_IN9: now reaches U10.27 (PB1)
- net DSP_STATUS: now reaches U10.28 (PB2)
- net NSPK_SD: now reaches U10.35 (PB14)
- no-connect marks 34 -> 30

Commit message: fix: issues with rev a
Parts:
- U10: MPN C75278 -> C74524
Other:
- note added: "Pin-compatible parts STM32F401Rx STM32F411Rx STM32F412Rx STM32F413Rx STM32F423Rx"
Changed lines of the file:
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@@
   (junction (at 142.24 44.45) (diameter 0) (color 0 0 0 0)
   )
+  (junction (at 125.73 109.22) (diameter 0) (color 0 0 0 0)
+  )
   (junction (at 203.2 80.01) (diameter 0) (color 0 0 0 0)
   )
   (junction (at 39.37 64.77) (diameter 0) (color 0 0 0 0)
-  )
-  (junction (at 124.46 109.22) (diameter 0) (color 0 0 0 0)
   )
   (junction (at 214.63 48.26) (diameter 0) (color 0 0 0 0)
@@
   (no_connect (at 160.02 93.98))
   (no_connect (at 160.02 53.34))
+  (no_connect (at 127 114.3))
   (no_connect (at 127 81.28))
   (no_connect (at 127 86.36))
@@
   (no_connect (at 127 106.68))
   (no_connect (at 127 111.76))
-  (no_connect (at 127 114.3))
   (no_connect (at 127 119.38))
   (no_connect (at 127 124.46))
@@
     (stroke (width 0) (type default) (color 0 0 0 0))
   )
+  (wire (pts (xy 111.76 106.68) (xy 125.73 106.68))
+    (stroke (width 0) (type default) (color 0 0 0 0))
+  )
   (wire (pts (xy 238.76 80.01) (xy 238.76 81.28))
     (stroke (width 0) (type default) (color 0 0 0 0))
@@
     (stroke (width 0) (type default) (color 0 0 0 0))
   )
-  (wire (pts (xy 124.46 105.41) (xy 124.46 109.22))
-    (stroke (width 0) (type default) (color 0 0 0 0))
-  )
   (wire (pts (xy 160.02 78.74) (xy 173.99 78.74))
     (stroke (width 0) (type default) (color 0 0 0 0))
@@
     (stroke (width 0) (type default) (color 0 0 0 0))
   )
-  (wire (pts (xy 109.22 105.41) (xy 124.46 105.41))
-    (stroke (width 0) (type default) (color 0 0 0 0))
-  )
   (wire (pts (xy 181.61 55.88) (xy 181.61 58.42))
     (stroke (width 0) (type default) (color 0 0 0 0))
@@
     (stroke (width 0) (type default) (color 0 0 0 0))
   )
+  (wire (pts (xy 124.46 78.74) (xy 127 78.74))
+    (stroke (width 0) (type default) (color 0 0 0 0))
+  )
   (wire (pts (xy 127 60.96) (xy 110.49 60.96))
     (stroke (width 0) (type default) (color 0 0 0 0))
@@
     (stroke (width 0) (type default) (color 0 0 0 0))
   )
-  (wire (pts (xy 124.46 78.74) (xy 127 78.74))
+  (wire (pts (xy 125.73 106.68) (xy 125.73 109.22))
     (stroke (width 0) (type default) (color 0 0 0 0))
   )
@@
     (stroke (width 0) (type default) (color 0 0 0 0))
   )
-  (wire (pts (xy 124.46 109.22) (xy 127 109.22))
-    (stroke (width 0) (type default) (color 0 0 0 0))
-  )
   (wire (pts (xy 229.87 90.17) (xy 238.76 90.17))
     (stroke (width 0) (type default) (color 0 0 0 0))
@@
     (stroke (width 0) (type default) (color 0 0 0 0))
   )
-  (wire (pts (xy 160.02 101.6) (xy 185.42 101.6))
+  (wire (pts (xy 160.02 101.6) (xy 184.15 101.6))
     (stroke (width 0) (type default) (color 0 0 0 0))
   )
@@
     (stroke (width 0) (type default) (color 0 0 0 0))
   )
+  (wire (pts (xy 125.73 109.22) (xy 127 109.22))
+    (stroke (width 0) (type default) (color 0 0 0 0))
+  )
   (wire (pts (xy 77.47 95.25) (xy 86.36 95.25))
     (stroke (width 0) (type default) (color 0 0 0 0))
@@
     (stroke (width 0) (type default) (color 0 0 0 0))
   )
-  (wire (pts (xy 121.92 109.22) (xy 124.46 109.22))
+  (wire (pts (xy 124.46 109.22) (xy 125.73 109.22))
     (stroke (width 0) (type default) (color 0 0 0 0))
   )
@@
     (stroke (width 0) (type default) (color 0 0 0 0))
   )
-  (label "TIM2_ETR" (at 109.22 105.41 0)
+  (text "Pin-compatible parts\nSTM32F401Rx\nSTM32F411Rx\nSTM32F412Rx\nSTM32F413Rx\nSTM32F423Rx"
+    (at 118.11 43.18 0)
+    (effects (font (size 1.524 1.524)) (justify left bottom))
+  )
+  (label "TIM2_ETR" (at 111.76 106.68 0)
     (effects (font (size 1.524 1.524)) (justify left bottom))
   )
@@
     (effects (font (size 1.524 1.524)) (justify right bottom))
   )
-  (label "SWO" (at 185.42 101.6 180)
+  (label "SWO" (at 184.15 101.6 180)
     (effects (font (size 1.524 1.524)) (justify right bottom))
   )
@@
     (effects (font (size 1.524 1.524)) (justify left))
   )
-  (hierarchical_label "I2S3_MCK" (shape output) (at 121.92 109.22 180)
+  (hierarchical_label "I2S3_MCK" (shape output) (at 124.46 109.22 180)
     (effects (font (size 1.524 1.524)) (justify right))
   )
@@
       (effects (font (size 1.27 1.27)) hide)
     )
-    (property "MPN" "C75278" (id 5) (at 144.78 88.9 0)
-      (effects (font (size 1.27 1.27)) hide)
-    )
+    (property "MPN" "C74524" (id 5) (at 144.78 88.9 0)
+      (effects (font (size 1.27 1.27)) hide)
+    )
