File: Hardware/amplifiers.kicad_sch (KiCad schematic)
At the start: 10 parts, among them J4 Screw_Terminal_01x02, J5 Screw_Terminal_01x02, J6 Screw_Terminal_01x02, J7 Screw_Terminal_01x02

Commit message: prod. version blus mini a
Parts:
- removed R8: 10k, Resistor_SMD:R_0402_1005Metric, symbol Device:R
- removed R9: 20k, Resistor_SMD:R_0402_1005Metric, symbol Device:R
- added R5: 10k, Resistor_SMD:R_0402_1005Metric, symbol Device:R
- R6: renamed from R15; MPN (none) -> C25744
- R7: renamed from R14; MPN (none) -> C25744
- R8: renamed from R12; MPN (none) -> C25117
- R9: renamed from R11; MPN (none) -> C25117
- renumbered J4 to J5, J5 to J6, J6 to J7, J7 to J8
Connections:
- net IRQZ: now also R5.1
- new net +3.3V: R5.2
- no-connect marks 4 -> 0
Other:
- sheet I2S-AMP-2CH-A ports: added none; removed BYP_EN, MCLK
- sheet I2S-AMP-2CH-B ports: added none; removed BYP_EN, MCLK
- sheet I2S-AMP-2CH-C ports: added none; removed BYP_EN, MCLK
- sheet I2S-AMP-2CH-D ports: added none; removed BYP_EN, MCLK

Commit message: feat!: wip, version b
Parts:
- J5, J6, J7, J8: footprint terminal_connectors:wuerth_691216410002 -> Connector_Terminal:wuerth_691216410002; Mfr.Nr. (none) -> DK
Changed lines of the file:
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@@
+    (stroke (width 0) (type default) (color 0 0 0 0))
+  )
+  (wire (pts (xy 57.15 41.91) (xy 68.58 41.91))
+    (stroke (width 0) (type default) (color 0 0 0 0))
+  )
+  (wire (pts (xy 140.97 165.1) (xy 142.24 165.1))
+    (stroke (width 0) (type default) (color 0 0 0 0))
+  )
+  (wire (pts (xy 105.41 182.88) (xy 87.63 182.88))
+    (stroke (width 0) (type default) (color 0 0 0 0))
+  )
+  (wire (pts (xy 87.63 43.18) (xy 105.41 43.18))
+    (stroke (width 0) (type default) (color 0 0 0 0))
+  )
+  (wire (pts (xy 140.97 92.71) (xy 151.13 92.71))
+    (stroke (width 0) (type default) (color 0 0 0 0))
+  )
+  (wire (pts (xy 87.63 74.93) (xy 105.41 74.93))
+    (stroke (width 0) (type default) (color 0 0 0 0))
+  )
+  (wire (pts (xy 87.63 31.75) (xy 105.41 31.75))
+    (stroke (width 0) (type default) (color 0 0 0 0))
+  )
+  (wire (pts (xy 87.63 158.75) (xy 105.41 158.75))
+    (stroke (width 0) (type default) (color 0 0 0 0))
+  )
+  (wire (pts (xy 140.97 138.43) (xy 151.13 138.43))
     (stroke (width 0) (type default) (color 0 0 0 0))
   )
@@
     (stroke (width 0) (type default) (color 0 0 0 0))
   )
-  (wire (pts (xy 140.97 165.1) (xy 142.24 165.1))
-    (stroke (width 0) (type default) (color 0 0 0 0))
-  )
-  (wire (pts (xy 105.41 182.88) (xy 87.63 182.88))
-    (stroke (width 0) (type default) (color 0 0 0 0))
-  )
-  (wire (pts (xy 87.63 43.18) (xy 105.41 43.18))
-    (stroke (width 0) (type default) (color 0 0 0 0))
-  )
-  (wire (pts (xy 140.97 92.71) (xy 151.13 92.71))
-    (stroke (width 0) (type default) (color 0 0 0 0))
-  )
-  (wire (pts (xy 68.58 34.29) (xy 57.15 34.29))
-    (stroke (width 0) (type default) (color 0 0 0 0))
-  )
-  (wire (pts (xy 87.63 74.93) (xy 105.41 74.93))
-    (stroke (width 0) (type default) (color 0 0 0 0))
-  )
-  (wire (pts (xy 87.63 31.75) (xy 105.41 31.75))
-    (stroke (width 0) (type default) (color 0 0 0 0))
-  )
-  (wire (pts (xy 87.63 158.75) (xy 105.41 158.75))
-    (stroke (width 0) (type default) (color 0 0 0 0))
-  )
-  (wire (pts (xy 140.97 138.43) (xy 151.13 138.43))
-    (stroke (width 0) (type default) (color 0 0 0 0))
-  )
-  (wire (pts (xy 57.15 26.67) (xy 68.58 26.67))
-    (stroke (width 0) (type default) (color 0 0 0 0))
-  )
   (wire (pts (xy 87.63 69.85) (xy 105.41 69.85))
     (stroke (width 0) (type default) (color 0 0 0 0))
@@
     (stroke (width 0) (type default) (color 0 0 0 0))
   )
-  (wire (pts (xy 68.58 39.37) (xy 57.15 39.37))
-    (stroke (width 0) (type default) (color 0 0 0 0))
-  )
-  (wire (pts (xy 68.58 29.21) (xy 57.15 29.21))
-    (stroke (width 0) (type default) (color 0 0 0 0))
-  )
   (wire (pts (xy 199.39 67.31) (xy 201.93 67.31))
     (stroke (width 0) (type default) (color 0 0 0 0))
   )
-  (wire (pts (xy 57.15 31.75) (xy 68.58 31.75))
+  (wire (pts (xy 57.15 39.37) (xy 68.58 39.37))
     (stroke (width 0) (type default) (color 0 0 0 0))
   )
@@
     (effects (font (size 1.524 1.524)) (justify right bottom))
   )
-  (label "LRCKA" (at 68.58 26.67 180)
+  (label "LRCKA" (at 68.58 36.83 180)
     (effects (font (size 1.524 1.524)) (justify right bottom))
   )
@@
     (effects (font (size 1.524 1.524)) (justify right bottom))
   )
+  (label "SCLKA" (at 87.63 172.72 0)
+    (effects (font (size 1.524 1.524)) (justify left bottom))
+  )
   (label "SDA" (at 87.63 29.21 0)
     (effects (font (size 1.524 1.524)) (justify left bottom))
   )
-  (label "LRCKB" (at 68.58 29.21 180)
-    (effects (font (size 1.524 1.524)) (justify right bottom))
+  (label "SDINA" (at 87.63 132.08 0)
+    (effects (font (size 1.524 1.524)) (justify left bottom))
   )
   (label "SDINA" (at 87.63 45.72 0)
@@
     (effects (font (size 1.524 1.524)) (justify left bottom))
   )
-  (label "LRCKB" (at 87.63 170.18 0)
-    (effects (font (size 1.524 1.524)) (justify left bottom))
-  )
-  (label "SCLKB" (at 68.58 34.29 180)
-    (effects (font (size 1.524 1.524)) (justify right bottom))
-  )
-  (label "SDINB" (at 87.63 175.26 0)
+  (label "SDINA" (at 87.63 175.26 0)
     (effects (font (size 1.524 1.524)) (justify left bottom))
   )
@@
     (effects (font (size 1.524 1.524)) (justify right bottom))
   )
-  (label "SCLKB" (at 87.63 172.72 0)
+  (label "SCLKA" (at 87.63 129.54 0)
     (effects (font (size 1.524 1.524)) (justify left bottom))
   )
@@
     (effects (font (size 1.524 1.524)) (justify left bottom))
   )
-  (label "SDINB" (at 87.63 132.08 0)
-    (effects (font (size 1.524 1.524)) (justify left bottom))
-  )
   (label "NSPK_SD" (at 87.63 96.52 0)
     (effects (font (size 1.524 1.524)) (justify left bottom))
   )
-  (label "SCLKB" (at 87.63 129.54 0)
-    (effects (font (size 1.524 1.524)) (justify left bottom))
-  )
   (label "NSPK_SD" (at 87.63 182.88 0)
     (effects (font (size 1.524 1.524)) (justify left bottom))
@@
     (effects (font (size 1.524 1.524)) (justify left bottom))
   )
-  (label "SDINA" (at 68.58 36.83 180)
-    (effects (font (size 1.524 1.524)) (justify right bottom))
-  )
-  (label "SDINB" (at 68.58 39.37 180)
+  (label "SDINA" (at 68.58 41.91 180)
     (effects (font (size 1.524 1.524)) (justify right bottom))
   )
@@
     (effects (font (size 1.524 1.524)) (justify right bottom))
   )
-  (label "LRCKB" (at 87.63 127 0)
-    (effects (font (size 1.524 1.524)) (justify left bottom))
-  )
   (label "SCLKA" (at 87.63 43.18 0)
     (effects (font (size 1.524 1.524)) (justify left bottom))
@@
     (effects (font (size 1.524 1.524)) (justify right bottom))
   )
-  (label "SCLKA" (at 68.58 31.75 180)
+  (label "SCLKA" (at 68.58 39.37 180)
     (effects (font (size 1.524 1.524)) (justify right bottom))
   )
@@
     (effects (font (size 1.524 1.524)) (justify left bottom))
   )
+  (label "LRCKA" (at 87.63 170.18 0)
+    (effects (font (size 1.524 1.524)) (justify left bottom))
+  )
   (label "NSPK_SD" (at 87.63 53.34 0)
     (effects (font (size 1.524 1.524)) (justify left bottom))
@@
   (label "IRQZ" (at 151.13 49.53 180)
     (effects (font (size 1.524 1.524)) (justify right bottom))
+  )
+  (label "LRCKA" (at 87.63 127 0)
+    (effects (font (size 1.524 1.524)) (justify left bottom))
   )
   (label "ADDRB" (at 87.63 74.93 0)
@@
     (effects (font (size 1.524 1.524)) (justify right))
   )
-  (hierarchical_label "LRCKB" (shape input) (at 57.15 29.21 180)
-    (effects (font (size 1.524 1.524)) (justify right))
-  )
-  (hierarchical_label "LRCKA" (shape input) (at 57.15 26.67 180)
+  (hierarchical_label "LRCKA" (shape input) (at 57.15 36.83 180)
     (effects (font (size 1.524 1.524)) (justify right))
   )
@@
     (effects (font (size 1.524 1.524)) (justify right))
   )
-  (hierarchical_label "SDINA" (shape input) (at 57.15 36.83 180)
+  (hierarchical_label "SDINA" (shape input) (at 57.15 41.91 180)
     (effects (font (size 1.524 1.524)) (justify right))
   )
@@
     (effects (font (size 1.524 1.524)) (justify right))
   )
-  (hierarchical_label "SCLKB" (shape input) (at 57.15 34.29 180)
-    (effects (font (size 1.524 1.524)) (justify right))
-  )
-  (hierarchical_label "SDINB" (shape input) (at 57.15 39.37 180)
-    (effects (font (size 1.524 1.524)) (justify right))
-  )
-  (hierarchical_label "SCLKA" (shape input) (at 57.15 31.75 180)
+  (hierarchical_label "SCLKA" (shape input) (at 57.15 39.37 180)
     (effects (font (size 1.524 1.524)) (justify right))
   )
@@
       (effects (font (size 1.27 1.27)) (justify left))
     )
-    (property "Footprint" "terminal_connectors:wuerth_691216410002" (id 2) (at 147.32 124.46 0)
+    (property "Footprint" "Connector_Terminal:wuerth_691216410002" (id 2) (at 147.32 124.46 0)
       (effects (font (size 1.27 1.27)) hide)
     )
@@
       (effects (font (size 1.27 1.27)) hide)
     )
-    (property "Mfr.Nr." "" (id 4) (at 147.32 124.46 0)
+    (property "Mfr.Nr." "DK" (id 4) (at 147.32 124.46 0)
       (effects (font (size 1.27 1.27)) hide)
     )
@@
       (effects (font (size 1.27 1.27)) (justify left))
     )
-    (property "Footprint" "terminal_connectors:wuerth_691216410002" (id 2) (at 147.32 167.64 0)
+    (property "Footprint" "Connector_Terminal:wuerth_691216410002" (id 2) (at 147.32 167.64 0)
       (effects (font (size 1.27 1.27)) hide)
     )
@@
       (effects (font (size 1.27 1.27)) hide)
     )
-    (property "Mfr.Nr." "" (id 4) (at 147.32 167.64 0)
+    (property "Mfr.Nr." "DK" (id 4) (at 147.32 167.64 0)
       (effects (font (size 1.27 1.27)) hide)
     )
@@
       (effects (font (size 1.27 1.27)) (justify left))
     )
-    (property "Footprint" "terminal_connectors:wuerth_691216410002" (id 2) (at 147.32 38.1 0)
+    (property "Footprint" "Connector_Terminal:wuerth_691216410002" (id 2) (at 147.32 38.1 0)
       (effects (font (size 1.27 1.27)) hide)
     )
@@
       (effects (font (size 1.27 1.27)) hide)
     )
-    (property "Mfr.Nr." "" (id 4) (at 147.32 38.1 0)
+    (property "Mfr.Nr." "DK" (id 4) (at 147.32 38.1 0)
       (effects (font (size 1.27 1.27)) hide)
     )
@@
       (effects (font (size 1.27 1.27)) (justify left))
     )
-    (property "Footprint" "terminal_connectors:wuerth_691216410002" (id 2) (at 147.32 81.28 0)
+    (property "Footprint" "Connector_Terminal:wuerth_691216410002" (id 2) (at 147.32 81.28 0)
       (effects (font (size 1.27 1.27)) hide)
     )
@@
       (effects (font (size 1.27 1.27)) hide)
     )
-    (property "Mfr.Nr." "" (id 4) (at 147.32 81.28 0)
-      (effects (font (size 1.27 1.27)) hide)
-    )
+    (property "Mfr.Nr." "DK" (id 4) (at 147.32 81.28 0)
+      (effects (font (size 1.27 1.27)) hide)
+    )

Commit message: chore: cleanup
Other:
- sheet I2S-AMP-2CH-A renamed TAS2780-A
- sheet I2S-AMP-2CH-B renamed TAS2780-B
- sheet I2S-AMP-2CH-C renamed TAS2780-C
- sheet I2S-AMP-2CH-D renamed TAS2780-D
- sheet TAS2780-A: file I2S-AMP-2CH.kicad_sch -> tas2780.kicad_sch
- sheet TAS2780-B: file I2S-AMP-2CH.kicad_sch -> tas2780.kicad_sch
- sheet TAS2780-C: file I2S-AMP-2CH.kicad_sch -> tas2780.kicad_sch
- sheet TAS2780-D: file I2S-AMP-2CH.kicad_sch -> tas2780.kicad_sch
Changed lines of the file:
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@@
     (stroke (width 0) (type solid) (color 0 0 0 0))
     (fill (color 0 0 0 0.0000))
-    (property "Sheet name" "I2S-AMP-2CH-D" (id 0) (at 105.41 151.5614 0)
+    (property "Sheet name" "TAS2780-D" (id 0) (at 105.41 151.5614 0)
       (effects (font (size 1.524 1.524)) (justify left bottom))
     )
-    (property "Sheet file" "I2S-AMP-2CH.kicad_sch" (id 1) (at 105.41 188.6462 0)
+    (property "Sheet file" "tas2780.kicad_sch" (id 1) (at 105.41 188.6462 0)
       (effects (font (size 1.524 1.524)) (justify left top))
     )
@@
     (stroke (width 0) (type solid) (color 0 0 0 0))
     (fill (color 0 0 0 0.0000))
-    (property "Sheet name" "I2S-AMP-2CH-A" (id 0) (at 105.41 22.0214 0)
+    (property "Sheet name" "TAS2780-A" (id 0) (at 105.41 22.0214 0)
       (effects (font (size 1.524 1.524)) (justify left bottom))
     )
-    (property "Sheet file" "I2S-AMP-2CH.kicad_sch" (id 1) (at 105.41 59.1062 0)
+    (property "Sheet file" "tas2780.kicad_sch" (id 1) (at 105.41 59.1062 0)
       (effects (font (size 1.524 1.524)) (justify left top))
     )
@@
     (stroke (width 0) (type solid) (color 0 0 0 0))
     (fill (color 0 0 0 0.0000))
-    (property "Sheet name" "I2S-AMP-2CH-C" (id 0) (at 105.41 108.3814 0)
+    (property "Sheet name" "TAS2780-C" (id 0) (at 105.41 108.3814 0)
       (effects (font (size 1.524 1.524)) (justify left bottom))
     )
-    (property "Sheet file" "I2S-AMP-2CH.kicad_sch" (id 1) (at 105.41 145.4662 0)
+    (property "Sheet file" "tas2780.kicad_sch" (id 1) (at 105.41 145.4662 0)
       (effects (font (size 1.524 1.524)) (justify left top))
     )
@@
     (stroke (width 0) (type solid) (color 0 0 0 0))
     (fill (color 0 0 0 0.0000))
-    (property "Sheet name" "I2S-AMP-2CH-B" (id 0) (at 105.41 65.2014 0)
+    (property "Sheet name" "TAS2780-B" (id 0) (at 105.41 65.2014 0)
       (effects (font (size 1.524 1.524)) (justify left bottom))
     )
-    (property "Sheet file" "I2S-AMP-2CH.kicad_sch" (id 1) (at 105.41 102.2862 0)
+    (property "Sheet file" "tas2780.kicad_sch" (id 1) (at 105.41 102.2862 0)
       (effects (font (size 1.524 1.524)) (justify left top))
     )
