File: blus-mini/kicad/amplifiers.kicad_sch (KiCad schematic)
At the start: 9 parts, among them J5 Screw_Terminal_01x02, J6 Screw_Terminal_01x02, J7 Screw_Terminal_01x02, J8 Screw_Terminal_01x02

Commit message: chore: add title blocks, extend readme minor changes
Other:
- company: (none) -> elagil
- title: (none) -> blus mini
Changed lines of the file:
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@@
 (kicad_sch (version 20211123) (generator eeschema)
   (paper "A4")
+  (title_block
+    (title "blus mini")
+    (date "2023-05-08")
+    (rev "b")
+    (company "elagil")
+  )
   (wire (pts (xy 181.61 49.53) (xy 191.77 49.53))
     (stroke (width 0) (type default) (color 0 0 0 0))
