File: blus-mini/kicad/clock.kicad_sch (KiCad schematic)
At the start: 4 parts, among them U12 74AVC9112, X1 ASV-24.576MHz-EJ-T

Commit message: chore: add title blocks, extend readme minor changes
Other:
- company: (none) -> elagil
- title: (none) -> blus mini
Changed lines of the file:
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@@
   (paper "A4")
   (title_block
-    (date "2023-02-18")
+    (title "blus mini")
+    (date "2023-05-08")
+    (rev "b")
+    (company "elagil")
   )
   (junction (at 116.84 49.53) (diameter 0) (color 0 0 0 0)
