File: blus-mini/kicad/dsp-amplifier-x4.kicad_sch (KiCad schematic)
At the start: 60 parts, among them J10 Conn_01x16_Female, J11 Raspberry_Pi_2_3, J9 Screw_Terminal_01x02, Q1 SS8550, U10 ADAU1452, U13 TSOP583xx

Commit message: chore: add title blocks, extend readme minor changes
Connections:
- removed net PI_SCL: J10.15 (Pin_15), J11.5 (SCL/GPIO3), R27.1
- removed net PI_SDA: J10.14 (Pin_14), J11.3 (SDA/GPIO2), R29.1
- new net SCL: J10.14 (Pin_14), R27.1
- new net SDA: J10.15 (Pin_15), R29.1
- no-connect marks 38 -> 40
Other:
- company: (none) -> elagil
- title: DSP-AMP -> blus mini
- moved on the sheet: R15, R16, R22, R23, R24, R25

Commit message: chore: update submodules, minor part changes
Parts:
- added RV2: R_Potentiometer, Potentiometer_SMD:Potentiometer_Vishay_TS53YL_Vertical, symbol Device:R_Potentiometer
Connections:
- net +3.3V: now also RV2.1
- net GND: now also RV2.3
- new net VPOT1: RV2.2
Other:
- sheet MCU ports: added IR_RX; removed none
