File: blus-mini/kicad/mcu.kicad_sch (KiCad schematic)
At the start: 20 parts, among them J1 USB_B, J3 REDFIT_SWD_6, SW1 BOOT, SW2 NRST, U8 USBLC6-2SC6, U9 STM32F401RBTx

Commit message: chore: add title blocks, extend readme minor changes
Parts:
- SW1, SW2: footprint Button_Switch_SMD:SW_SPST_PTS810 -> Button_Switch_SMD:SW_SPST_TL3342; MPN (none) -> C318884
Other:
- company: (none) -> elagil
- title: (none) -> blus mini
Changed lines of the file:
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@@
 (kicad_sch (version 20211123) (generator eeschema)
   (paper "A4")
+  (title_block
+    (title "blus mini")
+    (date "2023-05-08")
+    (rev "b")
+    (company "elagil")
+  )
   (junction (at 220.98 80.01) (diameter 0) (color 0 0 0 0)
   )
@@
       (effects (font (size 1.27 1.27)) (justify right))
     )
-    (property "Footprint" "Button_Switch_SMD:SW_SPST_PTS810" (id 2) (at 214.63 55.88 0)
+    (property "Footprint" "Button_Switch_SMD:SW_SPST_TL3342" (id 2) (at 214.63 55.88 0)
       (effects (font (size 1.27 1.27)) hide)
     )
     (property "Datasheet" "~" (id 3) (at 214.63 55.88 0)
+      (effects (font (size 1.27 1.27)) hide)
+    )
+    (property "MPN" "C318884" (id 4) (at 214.63 55.88 0)
       (effects (font (size 1.27 1.27)) hide)
     )
@@
       (effects (font (size 1.27 1.27)) (justify right))
     )
-    (property "Footprint" "Button_Switch_SMD:SW_SPST_PTS810" (id 2) (at 203.2 40.64 0)
+    (property "Footprint" "Button_Switch_SMD:SW_SPST_TL3342" (id 2) (at 203.2 40.64 0)
       (effects (font (size 1.27 1.27)) hide)
     )
@@
       (effects (font (size 1.27 1.27)) hide)
     )
+    (property "MPN" "C318884" (id 4) (at 203.2 40.64 0)
+      (effects (font (size 1.27 1.27)) hide)
+    )

Commit message: chore: update submodules, minor part changes
Parts:
- removed J3: REDFIT_SWD_6, Connector_Debug:WR-WST REDFIT IDC 6 DBG, symbol Connectors_Debug:REDFIT_SWD_6
- removed TP1: RX, TestPoint:TestPoint_THTPad_D2.0mm_Drill1.0mm, symbol Connector:TestPoint
- removed TP2: TX, TestPoint:TestPoint_THTPad_D2.0mm_Drill1.0mm, symbol Connector:TestPoint
- added J12: REDFIT_SWD_10, Connector_Debug:WR-WST REDFIT IDC 6 10 DBG, symbol Connectors_Debug:REDFIT_SWD_10
Connections:
- net +3.3V: now also J12.1 (VREF)
- net GND: now also J12.5 (GND)
- net NRST: now also J12.3 (nRST)
- net SWO: now also J12.6 (SWO)
- net TCK: now also J12.4 (SWCLK)
- net TMS: now also J12.2 (SWDIO)
- net USART2_RX: now also J12.10 (TX)
- net USART2_TX: now also J12.9 (RX)
- net IR_RX: now reaches U9.15 (PA1)
- no-connect marks 30 -> 29
Other:
- moved on the sheet: C63, C69, C76, C81, C86, R32, R35, SW1, SW2
