File: blus-mini/kicad/power.kicad_sch (KiCad schematic)
At the start: 16 parts, among them U5 AMS1117-3.3, U6 AMS1117-1.8, U7 TPS54302

Commit message: chore: add title blocks, extend readme minor changes
Other:
- company: (none) -> elagil
- title: (none) -> blus mini
Changed lines of the file:
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@@
 (kicad_sch (version 20211123) (generator eeschema)
   (paper "A4")
+  (title_block
+    (title "blus mini")
+    (date "2023-05-08")
+    (rev "b")
+    (company "elagil")
+  )
   (junction (at 74.93 49.53) (diameter 0) (color 0 0 0 0)
   )
