File: blus-mini/kicad/spdif.kicad_sch (KiCad schematic)
At the start: 8 parts, among them J2 Conn_Coaxial, J4 Conn_Coaxial, T1 DA100J

Commit message: chore: add title blocks, extend readme minor changes
Other:
- company: (none) -> elagil
- title: SPDIF -> blus mini
Changed lines of the file:
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@@
   (paper "A4")
   (title_block
-    (title "SPDIF")
-    (date "2021-03-30")
-    (rev "V0.1")
+    (title "blus mini")
+    (date "2023-05-08")
+    (rev "b")
+    (company "elagil")
   )
   (junction (at 161.29 88.9) (diameter 0) (color 0 0 0 0)
