File: blus-mini/kicad/tas2780.kicad_sch (KiCad schematic)
At the start: 15 parts, among them U4 TAS2780

Commit message: chore: add title blocks, extend readme minor changes
Other:
- company: (none) -> elagil
- title: AMP -> blus mini
Changed lines of the file:
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@@
   (paper "A4")
   (title_block
-    (title "AMP")
-    (date "2021-03-30")
-    (rev "V0.1")
+    (title "blus mini")
+    (date "2023-05-08")
+    (rev "b")
+    (company "elagil")
   )
   (junction (at 91.44 34.29) (diameter 0) (color 0 0 0 0)
