File: blus-mini-mk2/kicad/amplifiers.kicad_sch (KiCad schematic)
At the start: 9 parts, among them J5 Screw_Terminal_01x02, J6 Screw_Terminal_01x02, J7 Screw_Terminal_01x02, J8 Screw_Terminal_01x02

Commit message: feat: production version, blus mini mk2 a
Parts:
- renumbered J7 to J10, J8 to J11, J5 to J8, J6 to J9, R5 to R38, R9 to R39, R8 to R40, R7 to R41, R6 to R42
Other:
- sheet TAS2780-A ports: added TDM_FS, TDM_SCK, TDM_SDI, ~{SPK_SD}; removed LRCK, NSPK_SD, SCLK, SDIN
- sheet TAS2780-B ports: added TDM_FS, TDM_SCK, TDM_SDI, ~{SPK_SD}; removed LRCK, NSPK_SD, SCLK, SDIN
- sheet TAS2780-C ports: added TDM_FS, TDM_SCK, TDM_SDI, ~{SPK_SD}; removed LRCK, NSPK_SD, SCLK, SDIN
- sheet TAS2780-D ports: added TDM_FS, TDM_SCK, TDM_SDI, ~{SPK_SD}; removed LRCK, NSPK_SD, SCLK, SDIN
