File: blus-mini-mk2/kicad/blus-mini-mk2.kicad_sch (KiCad schematic)
At the start: 25 parts, among them J10 Conn_01x16_Female, J11 Raspberry_Pi_2_3, J9 Screw_Terminal_01x02, U13 TSOP583xx

Commit message: feat: wip, added most components
Parts:
- removed J10: Conn_01x16_Female, Connector_Debug:WR-WST REDFIT IDC 16, symbol Connector:Conn_01x16_Female
- removed R15, R22: 33, Resistor_SMD:R_0402_1005Metric, symbol Device:R
Connections:
- net AMP1_LRCLK renamed USB_CLK
- net Clock/CLK0 renamed Clock/CLK_24.576
- net EXT_BCLKO renamed EXT_SCK
- net EXT_LRCLKO renamed EXT_FS
- net EXT_MDO renamed EXT_SD
- net MCU/I2S3_SCK renamed MCU/SAI4_SCK_A
- net MCU/I2S3_SD renamed MCU/SAI4_SD_A
- net MCU/I2S3_WS renamed MCU/SAI4_FS_A
- net MCU_CLOCK renamed AUDIO_CLK
- net PI_BCLK renamed PI_SCK
- net PI_SCK: now also J11.12 (GPIO18/PWM0)
- net PI_LRCLK renamed PI_FS
- net PI_FS: now also J11.35 (GPIO19/MISO1)
- net PI_SDATA_I renamed PI_SDI
- net PI_SDATA_O renamed PI_SD
- net USB_BCLK renamed Amplifiers/SCLKA
- net USB_LRCLK renamed Amplifiers/LRCKA
- net USB_SDATA renamed Amplifiers/SDINA
- net _AMP1_LRCLK renamed Clock/CLK_24.000
- net _EXT_BCLKO renamed MCU/SAI1_SCK_A
- net _EXT_LRCLKO renamed MCU/SAI1_FS_A
- net _EXT_MDO renamed MCU/SAI1_SD_A
- net _PI_BCLK renamed MCU/SAI4_SCK_B
- net MCU/SAI4_SCK_B: no longer J11.12 (GPIO18/PWM0)
- net _PI_LRCLK renamed MCU/SAI4_FS_B
- net MCU/SAI4_FS_B: no longer J11.35 (GPIO19/MISO1)
- net _PI_SDATA_O renamed MCU/SAI4_SD_B
- net MCU/SAI4_SD_B: no longer J11.40 (GPIO21/SCLK1)
- new net PI_SDO: J11.40 (GPIO21/SCLK1)
- no-connect marks 20 -> 19
Other:
- sheet Clock ports: added CLK_24.000, CLK_24.576; removed CLK0
- sheet MCU ports: added SAI1_FS_A, SAI1_SCK_A, SAI1_SD_A, SAI1_SD_B, SAI4_FS_A, SAI4_FS_B, SAI4_SCK_A, SAI4_SCK_B, SAI4_SD_A, SAI4_SD_B, SPDIF_IN0, SPDIF_IN1, USB_CLK; removed DSP_STATUS, I2S3_MCK, I2S3_SCK, I2S3_SD, I2S3_WS, USB_SOF
- sheet Power ports: added VOUT_1V8; removed none
- moved on the sheet: R16, R24, R25, R27, R29, R38, R41, R42, R43

Commit message: feat: production version, blus mini mk2 a
Parts:
- removed R24: 33, Resistor_SMD:R_0402_1005Metric, symbol Device:R
- removed oshw1: Logo_Open_Hardware_Large, Symbol:OSHW-Symbol_6.7x6mm_SilkScreen, symbol Graphic:Logo_Open_Hardware_Large
- added J3: Conn_02x08_Odd_Even, Connector_IDC:IDC-Header_2x08_P2.54mm_Horizontal, symbol Connector_Generic:Conn_02x08_Odd_Even
- added JP1: SolderJumper_3_Bridged12, Jumper:SolderJumper-3_P1.3mm_Bridged12_RoundedPad1.0x1.5mm, symbol Jumper:SolderJumper_3_Bridged12
- added R13, R14: 33, Resistor_SMD:R_0402_1005Metric, symbol Device:R
- H1: renamed from H2; now not fitted; now left out of the parts list
- H2: renamed from H1; now not fitted; now left out of the parts list
- H3, H4: now not fitted; now left out of the parts list
- renumbered J9 to J1, J11 to J2, R38 to R1, R41 to R10, R25 to R11, R16 to R12, R23 to R2, R27 to R3, R29 to R4, R28 to R5, R30 to R6, R33 to R7, R43 to R8, R42 to R9, U13 to U1
Connections:
- net AVDD is gone; now on net +3.3V: RV1.1
- net PI_SD is gone; now on net PI_SDO: R10.2
- net +3.3V: now also U1.3 (Vs)
- net +5V: now also J3.1 (Pin_1)
- net EXT_FS: now also J3.9 (Pin_9)
- net EXT_SCK: now also J3.7 (Pin_7)
- net GND: now also J3.10 (Pin_10), J3.12 (Pin_12), J3.14 (Pin_14), J3.16 (Pin_16), J3.2 (Pin_2), J3.4 (Pin_4), J3.6 (Pin_6), J3.8 (Pin_8)
- net MCU/SAI1_SD_A: now also JP1.2 (C)
- net SCL: now also J3.13 (Pin_13)
- net SDA: now also J3.11 (Pin_11)
- net at J2.17 (3V3): now also J2.1 (3V3)
- net Amplifiers/LRCKA renamed Amplifiers/TDM_FS
- net Amplifiers/SCLKA renamed Amplifiers/TDM_SCK
- net Amplifiers/SDINA renamed Amplifiers/TDM_SDI
- net DSP_NRESET: no longer names the net of J2.11 (GPIO17)
- net DSP_SELFBOOT: no longer names the net of J2.15 (GPIO22)
- removed net PI_3V3: J2.1 (3V3), U1.3 (Vs)
- net PI_SCLK0 renamed PI_TDM_SCK0
- new net: JP1.3 (B), R14.2
- new net EXT_MCLK: J3.15 (Pin_15), R13.1
- new net EXT_SDI: J3.3 (Pin_3), JP1.1 (A)
- new net EXT_SDO: J3.5 (Pin_5), R14.1
- new net MCU/SAI1_MCLK_A: R13.2
- no-connect marks 19 -> 24
Other:
- sheet Amplifiers ports: added IRQZ, TDM_FS, TDM_SCK, TDM_SDI, ~{SPK_SD}; removed LRCKA, NSPK_SD, SCLKA, SDINA
- sheet MCU ports: added ADC1_INP3, SAI1_MCLK_A, SAI4_MCLK_A, SAI4_MCLK_B, SPI2_MISO, SPI2_MOSI, SPI2_NSS, SPI2_SCK, SPK_IRQZ, ~{SPK_SD}; removed ADC1_IN9, NSPK_SD
- moved on the sheet: J1, R1, R10, R11, R12, R2, R3, R4, R5, R6, R7, R8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
