File: blus-mini-mk2/kicad/clock.kicad_sch (KiCad schematic)
At the start: 3 parts, among them X1 ASV-24.576MHz-EJ-T

Commit message: feat: wip, added most components
Parts:
- removed X1: ASV-24.576MHz-EJ-T, Oscillator:Oscillator_SMD_Abracon_ASV-4Pin_7.0x5.1mm, symbol Oscillator:ASV-xxxMHz
- added X1: ASE-24.576 MHz, Oscillator:Oscillator_SMD_Abracon_ASE-4Pin_3.2x2.5mm, symbol Oscillator:ASE-xxxMHz
- added X2: ASE-24 MHz, Oscillator:Oscillator_SMD_Abracon_ASE-4Pin_3.2x2.5mm, symbol Oscillator:ASE-xxxMHz
Connections:
- net +3.3V: now also X1.1 (EN), X1.4 (Vdd), X2.1 (EN), X2.4 (Vdd)
- net GND: now also X1.2 (GND), X2.2 (GND)
- new net CLK_24.000: X2.3 (OUT)
- new net CLK_24.576: X1.3 (OUT)

Commit message: feat: production version, blus mini mk2 a
Parts:
- added C3: 100n, Capacitor_SMD:C_0402_1005Metric, symbol Device:C
- added C4: 10n, Capacitor_SMD:C_0402_1005Metric, symbol Device:C
- X2: MPN (none) -> C507379
- renumbered C96 to C1, C94 to C2
Connections:
- net +3.3V: now also C3.1, C4.1
- net GND: now also C3.2, C4.2
Other:
- moved on the sheet: C1, C2
