File: blus-mini-mk2/kicad/mcu.kicad_sch (KiCad schematic)
At the start: 21 parts, among them J1 USB_B, J12 REDFIT_SWD_10, SW1 BOOT, SW2 NRST, U6 STM32H723VGTx, U8 USBLC6-2SC6, U9 STM32F401RBTx

Commit message: feat: wip, added most components
Parts:
- removed C75: 4.7u, Capacitor_SMD:C_0805_2012Metric, symbol Device:C
- removed R19: 4.7k, Resistor_SMD:R_0402_1005Metric, symbol Device:R
- removed R20: 10k, Resistor_SMD:R_0402_1005Metric, symbol Device:R
- removed U9: STM32F401RBTx, Package_QFP:LQFP-64_10x10mm_P0.5mm, symbol MCU_ST_STM32F4:STM32F401RBTx
- added C64, C65, C66, C67, C68, C71: 100n, Capacitor_SMD:C_0402_1005Metric, symbol Device:C
- added C70: 4.7u, Capacitor_SMD:C_0805_2012Metric, symbol Device:C
- added R15: 10k, Resistor_SMD:R_0402_1005Metric, symbol Device:R
- added R22: 12k, Resistor_SMD:R_0402_1005Metric, symbol Device:R
- added U11: USB3300-EZK, Package_DFN_QFN:QFN-32-1EP_5x5mm_P0.5mm_EP3.45x3.45mm, symbol Interface_USB:USB3300-EZK
Connections:
- net +3.3V: now also U6.20 (VREF+), C64.1, C65.1, C66.1, C67.1, U11.16 (VDD3.3), U11.25 (VDD3.3), U11.30 (VDD3.3), U11.31 (REG_EN), U11.6 (VDD3.3)
- net GND: now also C64.2, C65.2, C66.2, C67.2, C68.2, C70.2, C71.2, R22.1, U11.1 (GND), U11.2 (GND), U11.33 (GND), U11.9 (RESET)
- net SAI4_FS_B: now also U6.43 (PE13); no longer U6.15 (PC0)
- net SAI4_SCK_B: now also U6.24 (PA2); no longer U6.42 (PE12)
- net SAI4_SD_A: now also U6.16 (PC1); no longer U6.36 (PB2)
- net USB_DM: now also U11.8 (DM); no longer U6.70 (PA11)
- net USB_DP: now also U11.7 (DP); no longer U6.71 (PA12)
- net VBUS: now also R15.2
- net ULPI_DIR: now reaches U6.17 (PC2_C)
- net ULPI_DIR: now also U11.12 (DIR)
- net ULPI_NXT: now reaches U6.18 (PC3_C)
- net ULPI_NXT: now also U11.11 (NXT)
- net ULPI_D0: now reaches U6.25 (PA3)
- net ULPI_D0: now also U11.24 (DATA0)
- net ULPI_CK: now reaches U6.29 (PA5)
- net ULPI_CK: now also U11.14 (CLKOUT)
- net ULPI_D1: now reaches U6.34 (PB0)
- net ULPI_D1: now also U11.23 (DATA1)
- net ULPI_D2: now reaches U6.35 (PB1)
- net ULPI_D2: now also U11.22 (DATA2)
- net TIM1_ETR: now reaches U6.37 (PE7)
- net TIM1_ETR: now also U6.67 (PA8)
- net ULPI_D3: now reaches U6.46 (PB10)
- net ULPI_D3: now also U11.21 (DATA3)
- net ULPI_D4: now reaches U6.47 (PB11)
- net ULPI_D4: now also U11.20 (DATA4)
- net ULPI_D5: now reaches U6.51 (PB12)
- net ULPI_D5: now also U11.19 (DATA5)
- net ULPI_D6: now reaches U6.52 (PB13)
- net ULPI_D6: now also U11.18 (DATA6)
- net SPDIF_IN1: now reaches U6.55 (PD8)
- net ULPI_D7: now reaches U6.91 (PB5)
- net ULPI_D7: now also U11.17 (DATA7)
- net USB_VBUS: no longer names the net of U6.68 (PA9)
- new net: R22.2, U11.32 (RBIAS)
- new net: C68.1, U11.15 (VDD1.8), U11.26 (VDD1.8)
- new net: C70.1, C71.1, U11.29 (VDDA1.8)
- new net: R15.1, U11.4 (VBUS)
- new net ULPI_STP: U11.13 (STP), U6.15 (PC0)
- new net USB_CLK: U11.28 (XI)
- no-connect marks 30 -> 5
Other:
- note added: "Required for feedback mechanism"
- note removed: "Pin-compatible parts STM32F401Rx STM32F411Rx STM32F412Rx STM32F413Rx STM32F423Rx"
- moved on the sheet: C60, C61, C63, C69, C76, C81, C86, J1, J12, R17, R18, R32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
Changed lines of the file:
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@@
-(kicad_sch (version 20230121) (generator eeschema)
-  (paper "A4")
-  (title_block
-    (title "blus mini mk2")
-    (date "2024-04-05")
-    (rev "a")
-    (company "elagil")
-  )
+(kicad_sch
+	(version 20231120)
+	(generator "eeschema")
+	(generator_version "8.0")
+	(paper "A4")
+	(title_block
+		(title "blus mini mk2")
+		(date "2024-04-05")
+		(rev "a")
+		(company "elagil")
+	)

Commit message: feat: production version, blus mini mk2 a
Parts:
- added C46, C50, C57: 4.7u, Capacitor_SMD:C_0805_2012Metric, symbol Device:C
- added C63, C64, C65: 100n, Capacitor_SMD:C_0402_1005Metric, symbol Device:C
- added D1: Blue, LED_SMD:LED_0603_1608Metric, symbol Device:LED
- added D2: Green, LED_SMD:LED_0603_1608Metric, symbol Device:LED
- added D3: Yellow, LED_SMD:LED_0603_1608Metric, symbol Device:LED
- added D4: Red, LED_SMD:LED_0603_1608Metric, symbol Device:LED
- added R26, R27, R28, R29: 330, Resistor_SMD:R_0402_1005Metric, symbol Device:R
- J6: renamed from J12; now not fitted
- J7: renamed from J1; MPN (none) -> C592900
- R30: renamed from R22; MPN (none) -> C25752
- U6: renamed from U8; JLCPCB Rotation Offset 180 -> 90; MPN (none) -> C7519
- U7: renamed from U11; JLCPCB Rotation Offset (none) -> 180; MPN (none) -> C108383
- U8: renamed from U6; MPN (none) -> C730142
- renumbered C71 to C47, C70 to C48, C68 to C49, C64 to C51, C65 to C52, C66 to C53, C67 to C54, C61 to C55, C60 to C56, C63 to C58, C69 to C59, C86 to C60, C76 to C61, C81 to C62, R18 to R23, R17 to R24, R15 to R25, R35 to R31
Connections:
- net +3.3V: now also C57.1, C63.1, C64.1, C65.1
- net GND: now also C46.2, C50.2, C57.2, C63.2, C64.2, C65.2, D1.1 (K), D2.1 (K), D3.1 (K), D4.1 (K)
- net HSE: now also U8.12 (PH0); no longer U8.97 (PE0)
- net SAI4_SCK_B: now also U8.42 (PE12); no longer U8.24 (PA2)
- net SAI4_SD_B: now also U8.41 (PE11); no longer U8.22 (PA0)
- net USART2_RX: now also U8.87 (PD6)
- net USART2_TX: now also U8.86 (PD5)
- net VBUS: now also C46.1
- net TDI: now reaches J6.8 (TDI)
- net TDI: now also U8.77 (PA15(JTDI))
- net _USB_DN: now reaches J7.2 (D-), U6.1 (I/O1)
- net _USB_DP: now reaches J7.3 (D+), U6.3 (I/O2)
- net at C49.1, U7.15 (VDD1.8), U7.26 (VDD1.8): now also C50.1
- net SAI1_MCLK_A: now reaches U8.1 (PE2)
- net SAI4_MCLK_B: now reaches U8.23 (PA1)
- net ADC1_INP3: now reaches U8.30 (PA6)
- net SPI2_MISO: now reaches U8.53 (PB14)
- net SPI2_MOSI: now reaches U8.54 (PB15)
- net IR_RX: now reaches U8.56 (PD9)
- net LED1: now reaches U8.63 (PC6)
- net LED1: now also R26.2
- net LED2: now reaches U8.64 (PC7)
- net LED2: now also R27.2
- net LED3: now reaches U8.65 (PC8)
- net LED3: now also R28.2
- net LED4: now reaches U8.66 (PC9)
- net LED4: now also R29.2
- net SPI2_SCK: now reaches U8.68 (PA9)
- net ~{SPK_SD}: now reaches U8.7 (PC13)
- net SPI2_NSS: now reaches U8.70 (PA11)
- net SPK_IRQZ: now reaches U8.8 (PC14)
- net I2C1_SCL: now reaches U8.92 (PB6)
- net I2C1_SDA: now reaches U8.93 (PB7)
- net TIM1_ETR renamed SAI4_MCLK_A
- net SAI4_MCLK_A: now also U8.97 (PE0); no longer U8.67 (PA8)
- net USB_DM renamed USB_DN
- new net: D4.2 (A), R29.1
- new net: D3.2 (A), R28.1
- new net: D1.2 (A), R26.1
- new net: D2.2 (A), R27.1
- new net USB_SOF: U8.67 (PA8)
- no-connect marks 5 -> 37
Other:
- moved on the sheet: C47, C48, C49, C51, C52, C53, C54, C58, C59, C60, C61, C62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
Changed lines of the file:
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@@
 	(title_block
 		(title "blus mini mk2")
-		(date "2024-04-05")
+		(date "2024-06-04")
 		(rev "a")
 		(company "elagil")
