File: blus-mini-mk2/kicad/power.kicad_sch (KiCad schematic)
At the start: 15 parts, among them U5 AMS1117-3.3, U7 TPS54302

Commit message: feat: wip, added most components
Parts:
- added U10: AMS1117-1.8, Package_TO_SOT_SMD:SOT-223-3_TabPin2, symbol Regulator_Linear:AMS1117-1.8
Connections:
- net GND: now also U10.1 (GND)
- net VOUT_5V0: now also U10.3 (VI)
- new net VOUT_1V8: U10.2 (VO)

Commit message: feat: production version, blus mini mk2 a
Parts:
- L1: MPN (none) -> C167220
- U10: renamed from U5; JLCPCB Rotation Offset 180 -> (none)
- U11: renamed from U10; MPN (none) -> C6185
- U9: renamed from U7; JLCPCB Rotation Offset 180 -> -90; MPN (none) -> C311983
- renumbered C54 to C66, C53 to C67, C55 to C68, C59 to C69, C58 to C70, C57 to C71, C56 to C72, R12 to R33, R11 to R34, R14 to R35, R10 to R36, R13 to R37
