File: blus-mini-mk2/kicad/spdif.kicad_sch (KiCad schematic)
At the start: 8 parts, among them J2 Conn_Coaxial, J4 Conn_Coaxial, T1 DA100J

Commit message: feat: wip, added most components
Parts:
- added R53: 220, Resistor_SMD:R_0402_1005Metric, symbol Device:R
- added R54: 100, Resistor_SMD:R_0402_1005Metric, symbol Device:R
- added U9: 74LVC1GU04DRL, Package_TO_SOT_SMD:SOT-553, symbol 74xGxx:74LVC1GU04DRL
- C62: value 10n -> 4.7n
Connections:
- net GND: now also U9.3 (GND)
- net SPDIF_IN: now also U9.4; no longer C62.2
- new net: C62.2, R53.1
- new net: R53.2, R54.1, U9.2
- new net: R54.2, U9.5 (VCC)
Other:
- moved on the sheet: C62, C97, J2, J4, R21, R44, R45, T1

Commit message: feat: production version, blus mini mk2 a
Parts:
- added C86: 100n, Capacitor_SMD:C_0402_1005Metric, symbol Device:C
- C44: renamed from C62; MPN C15195 -> (none)
- U5: renamed from U9; MPN (none) -> C2877548
- renumbered C97 to C45, J2 to J4, J4 to J5, R54 to R18, R53 to R19, R44 to R20, R45 to R22
Connections:
- net GND: now also C86.2
- net SPDIF_IN: now also R18.2
- net +3.3V: now reaches U5.5 (VCC)
- net +3.3V: now also C86.1; no longer R18.2
