File: blus-mini-mk2/kicad/tas2780.kicad_sch (KiCad schematic)
At the start: 15 parts, among them U4 TAS2780

Commit message: feat: production version, blus mini mk2 a
Parts:
- U2: renamed from U4; MPN (none) -> C5214951
- renumbered C52 to C10, C39 to C11, C44 to C12, C51 to C13, C24 to C14, C8 to C15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
Connections:
- net LRCK renamed TDM_FS
- net NSPK_SD renamed ~{SPK_SD}
- net SCLK renamed TDM_SCK
- net SDIN renamed TDM_SDI
